File: PRODIGY-MOTHERBOARD/heater.kicad_sch (KiCad schematic)
At the start: 4 parts, among them Q3 NJFET

Commit message: project restructure done. Hierarchical sheet done. Outputs/breakouts sheet done
Parts:
- removed D?: LED, LED_THT:LED_D5.0mm, symbol Device:LED
- removed Q3: NJFET, Package_TO_SOT_SMD:TO-252-3_TabPin2, symbol Simulation_SPICE:NJFET
- removed R15: R_Photo, OptoDevice:R_LDR_5.1x4.3mm_P3.4mm_Vertical, symbol Device:R_Photo
- removed TH1: Thermistor, Package_TO_SOT_THT:TO-92_Inline_W4.0mm_Horizontal_FlatSideUp, symbol Device:Thermistor
Changed lines of the file:
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@@
-(kicad_sch (version 20230121) (generator eeschema)
-  (paper "A4")
-  (symbol (lib_id "Device:Thermistor") (at 165.1 82.55 0) (unit 1)
-    (in_bom yes) (on_board yes) (dnp no) (fields_autoplaced)
-    (property "Reference" "TH1" (at 168.91 81.915 0)
-      (effects (font (size 1.27 1.27)) (justify left))
-    )
-    (property "Value" "Thermistor" (at 168.91 84.455 0)
-      (effects (font (size 1.27 1.27)) (justify left))
-    )
-    (property "Footprint" "Package_TO_SOT_THT:TO-92_Inline_W4.0mm_Horizontal_FlatSideUp" (at 165.1 82.55 0)
-      (effects (font (size 1.27 1.27)) hide)
-    )
-    (property "Datasheet" "~" (at 165.1 82.55 0)
-      (effects (font (size 1.27 1.27)) hide)
-    )
-    (pin "1")
-    (pin "2")
-    (instances
-      (project "PRODIGY-MOTHERBOARD"
-        (path "/f1c25860-8989-4190-bd24-2491d23ca7d9/57a67dfa-34a0-418f-88a6-5d1f09f28bd2"
-          (reference "TH1") (unit 1)
-        )
-      )
-    )
-  )
-  (symbol (lib_id "Simulation_SPICE:NJFET") (at 128.27 78.74 0) (unit 1)
-    (in_bom yes) (on_board yes) (dnp no) (fields_autoplaced)
-    (property "Reference" "Q3" (at 133.35 78.105 0)
-      (effects (font (size 1.27 1.27)) (justify left))
-    )
-    (property "Value" "NJFET" (at 133.35 80.645 0)
-      (effects (font (size 1.27 1.27)) (justify left))
-    )
-    (property "Footprint" "Package_TO_SOT_SMD:TO-252-3_TabPin2" (at 133.35 76.2 0)
-      (effects (font (size 1.27 1.27)) hide)
-    )
-    (property "Datasheet" "~" (at 128.27 78.74 0)
-      (effects (font (size 1.27 1.27)) hide)
-    )
-    (property "Sim.Device" "NJFET" (at 128.27 78.74 0)
-      (effects (font (size 1.27 1.27)) hide)
-    )
-    (property "Sim.Type" "SHICHMANHODGES" (at 128.27 78.74 0)
-      (effects (font (size 1.27 1.27)) hide)
-    )
-    (property "Sim.Pins" "1=D 2=G 3=S" (at 128.27 78.74 0)
-      (effects (font (size 1.27 1.27)) hide)
-    )
-    (pin "1")
-    (pin "2")
-    (pin "3")
-    (instances
-      (project "PRODIGY-MOTHERBOARD"
-        (path "/f1c25860-8989-4190-bd24-2491d23ca7d9/57a67dfa-34a0-418f-88a6-5d1f09f28bd2"
-          (reference "Q3") (unit 1)
-        )
-      )
-    )
-  )
-  (symbol (lib_id "Device:LED") (at 132.08 105.41 0) (unit 1)
-    (in_bom yes) (on_board yes) (dnp no) (fields_autoplaced)
-    (property "Reference" "D?" (at 130.4925 100.33 0)
-      (effects (font (size 1.27 1.27)))
-    )
-    (property "Value" "LED" (at 130.4925 102.87 0)
-      (effects (font (size 1.27 1.27)))
-    )
-    (property "Footprint" "LED_THT:LED_D5.0mm" (at 132.08 105.41 0)
-      (effects (font (size 1.27 1.27)) hide)
-    )
-    (property "Datasheet" "~" (at 132.08 105.41 0)
-      (effects (font (size 1.27 1.27)) hide)
-    )
-    (property "JLCPCB" "" (at 132.08 105.41 0)
-      (effects (font (size 1.27 1.27)) hide)
-    )
-    (pin "1")
-    (pin "2")
-    (instances
-      (project "PRODIGY-MOTHERBOARD"
-        (path "/f1c25860-8989-4190-bd24-2491d23ca7d9/b1537168-6bed-494f-94fc-02099d073fc2"
-          (reference "D?") (unit 1)
-        )
-        (path "/f1c25860-8989-4190-bd24-2491d23ca7d9/57a67dfa-34a0-418f-88a6-5d1f09f28bd2"
-          (reference "D21") (unit 1)
-        )
-      )
-    )
-  )
-  (symbol (lib_id "Device:R_Photo") (at 196.85 83.82 0) (unit 1)
-    (in_bom yes) (on_board yes) (dnp no) (fields_autoplaced)
-    (property "Reference" "R15" (at 199.39 83.185 0)
-      (effects (font (size 1.27 1.27)) (justify left))
-    )
-    (property "Value" "R_Photo" (at 199.39 85.725 0)
-      (effects (font (size 1.27 1.27)) (justify left))
-    )
-    (property "Footprint" "OptoDevice:R_LDR_5.1x4.3mm_P3.4mm_Vertical" (at 198.12 90.17 90)
-      (effects (font (size 1.27 1.27)) (justify left) hide)
-    )
-    (property "Datasheet" "~" (at 196.85 85.09 0)
-      (effects (font (size 1.27 1.27)) hide)
-    )
-    (pin "1")
-    (pin "2")
-    (instances
-      (project "PRODIGY-MOTHERBOARD"
-        (path "/f1c25860-8989-4190-bd24-2491d23ca7d9/57a67dfa-34a0-418f-88a6-5d1f09f28bd2"
-          (reference "R15") (unit 1)
-        )
-      )
-    )
-  )
+(kicad_sch
+	(version 20231120)
+	(generator "eeschema")
+	(generator_version "8.0")
+	(paper "A4")
 )
