File: PRODIGY-MOTHERBOARD/oled.kicad_sch (KiCad schematic)
At the start: 0 parts

Commit message: Finished I2C device and bus schematics. Added logic level translation.
Parts:
- added C31: 10uF, symbol Device:C
- added J25: OLED, symbol Connector_Generic:Conn_01x04
Connections:
- new net +5V: C31.1, J25.3 (Pin_3)
- new net GND: C31.2, J25.4 (Pin_4)
- new net I2C_SCK_OLED: J25.2 (Pin_2)
- new net I2C_SDA_OLED: J25.1 (Pin_1)
