File: PRODIGY-MOTHERBOARD/PRODIGY-MOTHERBOARD.kicad_pcb (KiCad board)
At the start: 2 copper layers, 170 x 125 mm, 87 parts, among them J1 GPIO, J10 USB_A, J11 Micro_SD_Card_Det2, J12 KEYPAD_MATRIX, J13 Conn_01x10, J14 Barrel_Jack_MountingPin, J15 AudioJack3, J2 PWM_OUT, J3 A_IN, J4 MOTOR, J5 SPI_OUT, J6 I2C, J7 CAN, J8 SERIAL, J9 Bus_M.2_Socket_A, P1 USB_C_Plug, P2 USB_C_Plug, Q1 NJFET, Q2 PMOS, Q3 Q_Photo_NPN, SW1 SW_SPST, SW2 SW_SPST, SW3 SW_SPST, SW4 SW_SPST, SW5 SW_SPST, U1 CP2102N-Axx-xQFN24, U10 LM386, U11 PN5321A3HN_C1xx, U13 LM386, U14 ST1S14PHR, U15 Si4460, U2 ESP32-WROOM-32, U3 CR2013-MI2120, U4 LM358, U5 ST1S14PHR, U6 HDC1080, U7 LIS2DH, U8 SN65HVD232, U9 DRV8870DDA

Commit message: project restructure done. Hierarchical sheet done. Outputs/breakouts sheet done
Parts:
- removed the D1 at (180.8, 79.8)
- removed the D10 at (166.5, 88.7)
- removed the D11 at (166.5, 97.3)
- removed the D12 at (166.5, 105.8)
- removed the D13 at (166.5, 114.4)
- removed the D14 at (166.5, 123.0)
- removed the D15 at (166.5, 131.6)
- removed the D16 at (166.5, 140.1)
- removed the D17 at (203.3, 79.8)
- removed the D2 at (188.3, 79.8)
- removed the D3 at (195.8, 79.8)
- removed the D4 at (218.2, 79.8)
- removed the D5 at (225.7, 79.8)
- removed the D6 at (233.2, 79.8)
- removed the D7 at (210.1, 79.8)
- removed the D8 at (240.0, 79.8)
- removed the D9 at (166.5, 79.7)
- removed G***: LOGO, LOGO
- removed the J12 at (127.2, 136.0)
- removed the J4 at (131.0, 148.6)
- removed the Q1 at (154.1, 37.1)
- removed U14: ST1S14PHR, Package_SO:TI_SO-PowerPAD-8
- added C10: 100nF, Capacitor_SMD:C_0603_1608Metric, F.Cu at (93.4, 126.6)
- added C11: 10nF, Capacitor_SMD:C_0603_1608Metric, F.Cu at (93.4, 131.7)
- added C12: 10nF, Capacitor_SMD:C_0603_1608Metric, F.Cu at (93.4, 129.2)
- added C13: 1nF, Capacitor_SMD:C_0603_1608Metric, F.Cu at (93.4, 136.7)
- added C14: 4.7nF, Capacitor_SMD:C_0603_1608Metric, F.Cu at (93.4, 134.2)
- added C15: 47pF, Capacitor_SMD:C_0603_1608Metric, F.Cu at (97.4, 124.1)
- added C16: 39pF, Capacitor_SMD:C_0603_1608Metric, F.Cu at (93.4, 139.2)
- added C17: 100nF, Capacitor_SMD:C_0603_1608Metric, F.Cu at (97.4, 129.2)
- added C18: 100nF, Capacitor_SMD:C_0603_1608Metric, F.Cu at (97.4, 126.6)
- added C19: 47uF, Capacitor_SMD:C_1210_3225Metric, F.Cu at (88.6, 129.2)
- added C20: 47uF, Capacitor_SMD:C_1210_3225Metric, F.Cu at (88.6, 125.0)
- added C21: 47uF, Capacitor_SMD:C_1210_3225Metric, F.Cu at (88.6, 137.8)
- added C22: 47uF, Capacitor_SMD:C_1210_3225Metric, F.Cu at (88.6, 133.5)
- added C9: 100nF, Capacitor_SMD:C_0603_1608Metric, F.Cu at (93.4, 124.1)
- added D1: D_IR_EMITTER, LED_THT:LED_D5.0mm_Horizontal_O1.27mm_Z3.0mm_Clear, F.Cu at (41.6, 119.7)
- added D1: D_Schottky, Diode_SMD:D_SMB, F.Cu at (117.3, 125.7)
- added D10: WS2812B, LED_SMD:LED_WS2812B_PLCC4_5.0x5.0mm_P3.2mm, F.Cu at (19.0, 134.4)
- added D10: WS2812B, LED_SMD:LED_WS2812B_PLCC4_5.0x5.0mm_P3.2mm, F.Cu at (158.5, 135.4)
- added D11: WS2812B, LED_SMD:LED_WS2812B_PLCC4_5.0x5.0mm_P3.2mm, F.Cu at (158.5, 142.0)
- added D11: WS2812B, LED_SMD:LED_WS2812B_PLCC4_5.0x5.0mm_P3.2mm, F.Cu at (19.0, 141.0)
- added D12: LED_ABGR, LED_THT:LED_D5.0mm-4_RGB, F.Cu at (33.5, 121.7)
- added D12: WS2812B, LED_SMD:LED_WS2812B_PLCC4_5.0x5.0mm_P3.2mm, F.Cu at (166.9, 115.5)
- added D13: LED_ABGR, LED_THT:LED_D5.0mm-4_RGB, F.Cu at (33.5, 129.2)
- added D13: WS2812B, LED_SMD:LED_WS2812B_PLCC4_5.0x5.0mm_P3.2mm, F.Cu at (166.9, 122.2)
- added D14: WS2812B, LED_SMD:LED_WS2812B_PLCC4_5.0x5.0mm_P3.2mm, F.Cu at (166.9, 128.8)
- added D14: WS2812B, LED_SMD:LED_WS2812B_PLCC4_5.0x5.0mm_P3.2mm, F.Cu at (19.0, 147.7)
- added D15: LED, LED_THT:LED_D5.0mm, F.Cu at (173.6, 116.0)
- added D15: WS2812B, LED_SMD:LED_WS2812B_PLCC4_5.0x5.0mm_P3.2mm, F.Cu at (27.4, 121.2)
- added D16: WS2812B, LED_SMD:LED_WS2812B_PLCC4_5.0x5.0mm_P3.2mm, F.Cu at (27.4, 127.8)
- added D16: LED, LED_THT:LED_D5.0mm, F.Cu at (181.1, 116.0)
- added D17: LED, LED_THT:LED_D5.0mm, F.Cu at (188.6, 116.0)
- added D17: WS2812B, LED_SMD:LED_WS2812B_PLCC4_5.0x5.0mm_P3.2mm, F.Cu at (27.4, 134.4)
- added D2: LED, LED_THT:LED_D5.0mm, F.Cu at (17.2, 114.1)
- added D2: D_Schottky, Diode_SMD:D_SMB, F.Cu at (117.3, 136.8)
- added D21: LED, LED_THT:LED_D5.0mm, F.Cu at (139.7, 54.8)
- added D21: LED_ABGR, LED_THT:LED_D5.0mm-4_RGB, F.Cu at (173.0, 131.1)
- added D23: LED, LED_THT:LED_D5.0mm, F.Cu at (188.6, 123.6)
- added D3: LED, LED_THT:LED_D5.0mm, F.Cu at (24.7, 114.1)
- added D3: D_Schottky, Diode_SMD:D_SMB, F.Cu at (117.3, 131.2)
- added D4: LED, LED_THT:LED_D5.0mm, F.Cu at (32.2, 114.1)
- added D4: D_Schottky, Diode_SMD:D_SMB, F.Cu at (139.5, 84.0)
- added D5: D_Schottky, Diode_SMD:D_SMB, F.Cu at (102.5, 56.9)
- added D5: WS2812B, LED_SMD:LED_WS2812B_PLCC4_5.0x5.0mm_P3.2mm, F.Cu at (19.0, 121.2)
- added D6: D_IR_EMITTER, LED_THT:LED_D5.0mm_Horizontal_O1.27mm_Z3.0mm_Clear, F.Cu at (181.1, 129.1)
- added D6: LED, LED_THT:LED_D5.0mm, F.Cu at (39.7, 114.1)
- added D7: WS2812B, LED_SMD:LED_WS2812B_PLCC4_5.0x5.0mm_P3.2mm, F.Cu at (158.5, 115.5)
- added D7: LED, LED_THT:LED_D5.0mm, F.Cu at (47.2, 114.1)
- added D8: LED, LED_THT:LED_D5.0mm, F.Cu at (54.7, 114.1)
- added D8: WS2812B, LED_SMD:LED_WS2812B_PLCC4_5.0x5.0mm_P3.2mm, F.Cu at (158.5, 122.2)
- added D9: WS2812B, LED_SMD:LED_WS2812B_PLCC4_5.0x5.0mm_P3.2mm, F.Cu at (19.0, 127.8)
- added D9: WS2812B, LED_SMD:LED_WS2812B_PLCC4_5.0x5.0mm_P3.2mm, F.Cu at (158.5, 128.8)
- added J12: USB_A, Connector_USB:USB_A_TE_292303-7_Horizontal, F.Cu at (126.2, 51.8)
- added J12: MOTOR, Connector_JST:JST_XH_S6B-XH-A_1x06_P2.50mm_Horizontal, F.Cu at (89.2, 83.5)
- added J16: AudioJack3, Connector_Audio:Jack_3.5mm_Lumberg_1503_07_Horizontal, F.Cu at (137.4, 25.5)
- added J19: KEYPAD_MATRIX, Connector_PinHeader_2.54mm:PinHeader_1x08_P2.54mm_Vertical_SMD_Pin1Left, F.Cu at (121.0, 29.7)
- added J20: Ultrasonic, Connector_JST:JST_XH_S4B-XH-A_1x04_P2.50mm_Horizontal, F.Cu at (241.5, 69.0)
- added J21: GPIO, Connector_JST:JST_XH_S3B-XH-A_1x03_P2.50mm_Horizontal, F.Cu at (205.5, 69.0)
- added J22: GPIO, Connector_JST:JST_XH_S3B-XH-A_1x03_P2.50mm_Horizontal, F.Cu at (217.4, 69.0)
- added J23: GPIO, Connector_JST:JST_XH_S3B-XH-A_1x03_P2.50mm_Horizontal, F.Cu at (229.4, 69.0)
- added J24: 12V OUT, TerminalBlock_Phoenix:TerminalBlock_Phoenix_MKDS-1,5-2-5.08_1x02_P5.08mm_Horizontal, F.Cu at (274.5, 74.5)
- added J4: SERVO, Connector_JST:JST_XH_S3B-XH-A_1x03_P2.50mm_Horizontal, F.Cu at (169.7, 69.0)
- added J4: PWM_OUT, Connector_JST:JST_XH_S3B-XH-A_1x03_P2.50mm_Horizontal, F.Cu at (101.2, 70.0)
- added Q1: Q_Photo_NPN, LED_THT:LED_D5.0mm_Horizontal_O1.27mm_Z3.0mm_IRBlack, F.Cu at (49.1, 119.7)
- added Q1: Q_Photo_NPN, LED_THT:LED_D5.0mm_Horizontal_O1.27mm_Z3.0mm_IRBlack, F.Cu at (188.6, 129.1)
- added R10: 1k 1%, Resistor_SMD:R_0603_1608Metric, F.Cu at (105.5, 129.2)
- added R11: 10k 1%, Resistor_SMD:R_0603_1608Metric, F.Cu at (101.5, 131.7)
- added R12: 1k 1%, Resistor_SMD:R_0603_1608Metric, F.Cu at (101.5, 134.2)
- added R13: 680 1%, Resistor_SMD:R_0603_1608Metric, F.Cu at (105.5, 124.1)
- added R14: 220 1%, Resistor_SMD:R_0603_1608Metric, F.Cu at (105.5, 126.6)
- added R15: R_Photo, OptoDevice:R_LDR_5.1x4.3mm_P3.4mm_Vertical, F.Cu at (141.9, 112.6)
- added R2: 330k, Resistor_SMD:R_0603_1608Metric, F.Cu at (97.4, 139.2)
- added R3: 68k, Resistor_SMD:R_0603_1608Metric, F.Cu at (101.5, 124.1)
- added R4: 330k, Resistor_SMD:R_0603_1608Metric, F.Cu at (97.4, 134.2)
- added R5: 68k, Resistor_SMD:R_0603_1608Metric, F.Cu at (97.4, 136.7)
- added R6: 29.4k, Resistor_SMD:R_0603_1608Metric, F.Cu at (101.5, 129.2)
- added R7: 50k, Resistor_SMD:R_0603_1608Metric, F.Cu at (101.5, 126.6)
- added R8: 10k 1%, Resistor_SMD:R_0603_1608Metric, F.Cu at (101.5, 136.7)
- added R9: 2.2k 1%, Resistor_SMD:R_0603_1608Metric, F.Cu at (101.5, 139.2)
- added U12: PCF8574TS, Package_SO:SSOP-20_4.4x6.5mm_P0.65mm, F.Cu at (129.2, 22.8)
- added U16: LM386, Package_SO:SOP-8_3.9x4.9mm_P1.27mm, F.Cu at (127.8, 113.1)
- AE1, P1, P2: moved to F.Cu
- C1, C5, C6, C7, C8: value C -> 4.7uF; footprint Capacitor_SMD:C_1210_3225Metric -> Capacitor_SMD:C_1206_3216Metric; moved to F.Cu
- C2: value C -> 22nF; footprint Capacitor_SMD:C_1210_3225Metric -> Capacitor_SMD:C_0603_1608Metric; moved to F.Cu
- C3: value C -> 100uF; footprint Capacitor_SMD:C_1210_3225Metric -> Capacitor_SMD:CP_Elec_6.3x7.7; moved to F.Cu
- C4: value C -> 47uF; moved to F.Cu
- D18, D19, D20: value D_Schottky -> LED; footprint Diode_SMD:D_SMB -> LED_THT:LED_D5.0mm; moved to F.Cu
- D22: value D_IR_EMITTER -> LED_ABGR; footprint LED_THT:LED_D5.0mm_Horizontal_O1.27mm_Z3.0mm_Clear -> LED_THT:LED_D5.0mm-4_RGB; moved to F.Cu
- F1: value Fuse -> 2A; moved to F.Cu
- J1: value GPIO -> USB_A; footprint Connector_JST:JST_XH_S3B-XH-A_1x03_P2.50mm_Horizontal -> Connector_USB:USB_A_TE_292303-7_Horizontal; moved to F.Cu
- J10: value USB_A -> CAN; footprint Connector_USB:USB_A_TE_292303-7_Horizontal -> Connector_JST:JST_XH_S4B-XH-A_1x04_P2.50mm_Horizontal; moved to F.Cu
- J11: value Micro_SD_Card_Det2 -> SERIAL; footprint Connector_Card:microSD_HC_Hirose_DM3AT-SF-PEJM5 -> Connector_JST:JST_XH_S4B-XH-A_1x04_P2.50mm_Horizontal; moved to F.Cu
- J13: value Conn_01x10 -> MOTOR; footprint Potentiometer_THT:Potentiometer_Piher_PT-15-V02_Vertical -> Connector_JST:JST_XH_S6B-XH-A_1x06_P2.50mm_Horizontal
- J14: value Barrel_Jack_MountingPin -> Micro_SD_Card_Det2; footprint Connector_BarrelJack:BarrelJack_CUI_PJ-063AH_Horizontal -> Connector_Card:microSD_HC_Hirose_DM3AT-SF-PEJM5; moved to F.Cu
- J15: value AudioJack3 -> Barrel_Jack_MountingPin; footprint Connector_Audio:Jack_3.5mm_Lumberg_1503_07_Horizontal -> Connector_BarrelJack:BarrelJack_CUI_PJ-063AH_Horizontal; moved to F.Cu
- J2: value PWM_OUT -> SERVO; moved to F.Cu
- J3: value A_IN -> SERVO; moved to F.Cu
- J5: value SPI_OUT -> GPIO; footprint Connector_JST:JST_XH_S6B-XH-A_1x06_P2.50mm_Horizontal -> Connector_JST:JST_XH_S3B-XH-A_1x03_P2.50mm_Horizontal; moved to F.Cu
- J6: value I2C -> A_IN; footprint Connector_JST:JST_XH_S4B-XH-A_1x04_P2.50mm_Horizontal -> Connector_JST:JST_XH_S3B-XH-A_1x03_P2.50mm_Horizontal; moved to F.Cu
- J7: value CAN -> A_OUT; footprint Connector_JST:JST_XH_S4B-XH-A_1x04_P2.50mm_Horizontal -> Connector_JST:JST_XH_S3B-XH-A_1x03_P2.50mm_Horizontal; moved to F.Cu
- J8: value SERIAL -> SPI_OUT; footprint Connector_JST:JST_XH_S4B-XH-A_1x04_P2.50mm_Horizontal -> Connector_JST:JST_XH_S6B-XH-A_1x06_P2.50mm_Horizontal; moved to F.Cu
- J9: value Bus_M.2_Socket_A -> I2C; footprint m.2_edge_connector_key_a:121992304 -> Connector_JST:JST_XH_S4B-XH-A_1x04_P2.50mm_Horizontal; moved to F.Cu
- L1, L2: value L -> 6.8; moved to F.Cu
- Q2: value PMOS -> NJFET; footprint Package_TO_SOT_SMD:SOT-23 -> Package_TO_SOT_SMD:TO-252-3_TabPin2; moved to F.Cu
- Q3: value Q_Photo_NPN -> NJFET; footprint LED_THT:LED_D5.0mm_Horizontal_O1.27mm_Z3.0mm_IRBlack -> Package_TO_SOT_SMD:TO-252-3_TabPin2; moved to F.Cu
- R1: value R_Photo -> DNP; footprint OptoDevice:R_LDR_5.1x4.3mm_P3.4mm_Vertical -> Resistor_SMD:R_0603_1608Metric
- U1: value CP2102N-Axx-xQFN24 -> PN5321A3HN_C1xx; footprint Package_DFN_QFN:QFN-24-1EP_4x4mm_P0.5mm_EP2.6x2.6mm -> Package_DFN_QFN:HVQFN-40-1EP_6x6mm_P0.5mm_EP4.1x4.1mm; moved to F.Cu
- U10: value LM386 -> DRV8870DDA; footprint Package_SO:SOP-8_3.9x4.9mm_P1.27mm -> Package_SO:Texas_HTSOP-8-1EP_3.9x4.9mm_P1.27mm_EP2.95x4.9mm_Mask2.4x3.1mm_ThermalVias; moved to F.Cu
- U11: value PN5321A3HN_C1xx -> CR2013-MI2120; footprint Package_DFN_QFN:HVQFN-40-1EP_6x6mm_P0.5mm_EP4.1x4.1mm -> Display:CR2013-MI2120; moved to F.Cu
- U13: value LM386 -> PCF8574TS; footprint Package_SO:SOP-8_3.9x4.9mm_P1.27mm -> Package_SO:SSOP-20_4.4x6.5mm_P0.65mm; moved to F.Cu
- U15: value Si4460 -> CC56-12YWA; footprint Package_DFN_QFN:QFN-20-1EP_4x4mm_P0.5mm_EP2.5x2.5mm -> Display_7Segment:CC56-12YWA; moved to F.Cu
- U2: value ESP32-WROOM-32 -> LIS2DH; footprint RF_Module:ESP32-WROOM-32 -> Package_LGA:LGA-14_2x2mm_P0.35mm_LayoutBorder3x4y; moved to F.Cu
- U3: value CR2013-MI2120 -> TPS22810DRV; footprint Display:CR2013-MI2120 -> Package_SON:WSON-6-1EP_2x2mm_P0.65mm_EP1x1.6mm
- U4: value LM358 -> TPS54331DR; footprint Package_SO:SOIC-8_3.9x4.9mm_P1.27mm -> Package_SO:TI_SO-PowerPAD-8_ThermalVias; moved to F.Cu
- U5: value ST1S14PHR -> TPS54331DR; footprint Package_SO:TI_SO-PowerPAD-8 -> Package_SO:TI_SO-PowerPAD-8_ThermalVias; moved to F.Cu
- U6: value HDC1080 -> Si4460; footprint Package_SON:Texas_PWSON-N6 -> Package_DFN_QFN:QFN-20-1EP_4x4mm_P0.5mm_EP2.5x2.5mm; moved to F.Cu
- U7: value LIS2DH -> LM386; footprint Package_LGA:LGA-14_2x2mm_P0.35mm_LayoutBorder3x4y -> Package_SO:SOP-8_3.9x4.9mm_P1.27mm; moved to F.Cu
- U8: value SN65HVD232 -> HDC1080; footprint Package_SO:SOIC-8_3.9x4.9mm_P1.27mm -> Package_SON:Texas_PWSON-N6; moved to F.Cu
- U9: value DRV8870DDA -> SN65HVD232; footprint Package_SO:Texas_HTSOP-8-1EP_3.9x4.9mm_P1.27mm_EP2.95x4.9mm_Mask2.4x3.1mm_ThermalVias -> Package_SO:SOIC-8_3.9x4.9mm_P1.27mm; moved to F.Cu
- moved U13 233.9 mm to (18.9, 60.6), turned to 0 degrees
- moved U10 205.1 mm to (29.8, 156.3), turned to 0 degrees
- moved U11 199.0 mm to (17.3, 77.3), turned to 0 degrees
- moved AE1 149.3 mm to (147.4, 33.6)
- moved R1 142.3 mm to (105.5, 131.7)
- moved J2 141.6 mm to (89.2, 70.0), turned to 0 degrees
- moved H4 137.4 mm to (134.5, 77.5)
- moved Q2 136.3 mm to (185.6, 143.9)
- moved U3 135.2 mm to (109.1, 157.3)
- moved J15 129.4 mm to (107.9, 142.5)
- moved H3 115.2 mm to (134.5, 70.3)
- moved D19 115.0 mm to (173.6, 123.6), turned to 0 degrees
- moved J6 113.3 mm to (113.2, 70.0), turned to 0 degrees
- moved U4 112.4 mm to (118.7, 150.5), turned to 0 degrees
- moved SW3 109.8 mm to (131.9, 141.8), turned to 0 degrees
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Connections:
- C1 pad 1: unconnected-(C1-Pad1) -> +5V
- C1 pad 2: unconnected-(C1-Pad2) -> GND
- C2 pad 1: unconnected-(C2-Pad1) -> Net-(U3-CT)
- C2 pad 2: unconnected-(C2-Pad2) -> GND
- C3 pad 1: unconnected-(C3-Pad1) -> /POWER/VIN
- C3 pad 2: unconnected-(C3-Pad2) -> GND
- C4 pad 1: unconnected-(C4-Pad1) -> /POWER/USB_HOST_PWR
- C4 pad 2: unconnected-(C4-Pad2) -> GND
- C5 pad 1: unconnected-(C5-Pad1) -> /POWER/VIN
- C5 pad 2: unconnected-(C5-Pad2) -> GND
- C6 pad 1: unconnected-(C6-Pad1) -> +5V
- C6 pad 2: unconnected-(C6-Pad2) -> GND
- C7 pad 1: unconnected-(C7-Pad1) -> /POWER/VIN
- C7 pad 2: unconnected-(C7-Pad2) -> GND
- C8 pad 1: unconnected-(C8-Pad1) -> +5V
- C8 pad 2: unconnected-(C8-Pad2) -> GND
- F1 pad 1: unconnected-(F1-Pad1) -> Net-(F1-Pad1)
- F1 pad 2: unconnected-(F1-Pad2) -> Net-(D1-A)
- J1 pad 1: unconnected-(J1-Pin_1-Pad1) -> /OUTPUTS/BREAKOUT_USB_VBUS
- J1 pad 2: unconnected-(J1-Pin_2-Pad2) -> /OUTPUTS/BREAKOUT_USB_D-
- J1 pad 3: unconnected-(J1-Pin_3-Pad3) -> /OUTPUTS/BREAKOUT_USB_D+
- J10 pad 1: unconnected-(J10-VBUS-Pad1) -> /OUTPUTS/BREAKOUT_CAN_TX
- J10 pad 2: unconnected-(J10-D--Pad2) -> /OUTPUTS/BREAKOUT_CAN_RX
- J10 pad 3: unconnected-(J10-D+-Pad3) -> VCC
- J10 pad 4: unconnected-(J10-GND-Pad4) -> GND
- J11 pad 1: unconnected-(J11-DAT2-Pad1) -> /OUTPUTS/BREAKOUT_SERIAL_TX
- J11 pad 2: unconnected-(J11-DAT3/CD-Pad2) -> /OUTPUTS/BREAKOUT_SERIAL_RX
- J11 pad 3: unconnected-(J11-CMD-Pad3) -> VCC
- J11 pad 4: unconnected-(J11-VDD-Pad4) -> GND
- J13 pad 1: unconnected-(J13-Pin_1-Pad1) -> /OUTPUTS/BREAKOUT_MOTOR_PWM1_2
- J13 pad 2: unconnected-(J13-Pin_2-Pad2) -> /OUTPUTS/BREAKOUT_MOTOR_PWM2_2
- J13 pad 3: unconnected-(J13-Pin_3-Pad3) -> /OUTPUTS/BREAKOUT_MOTOR_C1_2
- J2 pad 1: unconnected-(J2-Pin_1-Pad1) -> /OUTPUTS/BREAKOUT_SERVO_0
- J2 pad 2: unconnected-(J2-Pin_2-Pad2) -> VCC
- J2 pad 3: unconnected-(J2-Pin_3-Pad3) -> GND
- J3 pad 1: unconnected-(J3-Pin_1-Pad1) -> /OUTPUTS/BREAKOUT_SERVO_1
- J3 pad 2: unconnected-(J3-Pin_2-Pad2) -> VCC
- J3 pad 3: unconnected-(J3-Pin_3-Pad3) -> GND
- J5 pad 1: unconnected-(J5-Pin_1-Pad1) -> /OUTPUTS/BREAKOUT_D_GPIO_0
- J5 pad 2: unconnected-(J5-Pin_2-Pad2) -> VCC
- J5 pad 3: unconnected-(J5-Pin_3-Pad3) -> GND
- J6 pad 1: unconnected-(J6-Pin_1-Pad1) -> /OUTPUTS/BREAKOUT_A_IN_0
- J6 pad 2: unconnected-(J6-Pin_2-Pad2) -> VCC
- J6 pad 3: unconnected-(J6-Pin_3-Pad3) -> GND
- J7 pad 1: unconnected-(J7-Pin_1-Pad1) -> /OUTPUTS/BREAKOUT_A_OUT_0
- J7 pad 2: unconnected-(J7-Pin_2-Pad2) -> VCC
- J7 pad 3: unconnected-(J7-Pin_3-Pad3) -> GND
- J8 pad 1: unconnected-(J8-Pin_1-Pad1) -> /OUTPUTS/BREAKOUT_SPI_CS
- J8 pad 2: unconnected-(J8-Pin_2-Pad2) -> /OUTPUTS/BREAKOUT_SPI_SCK
- J8 pad 3: unconnected-(J8-Pin_3-Pad3) -> /OUTPUTS/BREAKOUT_SPI_MSIO
- J8 pad 4: unconnected-(J8-Pin_4-Pad4) -> /OUTPUTS/BREAKOUT_SPI_MOSI
- J9 pad 1: Net-(J9-GND-Pad1) -> /OUTPUTS/BREAKOUT_I2C_SDA
- J9 pad 2: Net-(J9-3.3V-Pad2) -> /OUTPUTS/BREAKOUT_I2C_SCL
- J9 pad 3: unconnected-(J9-USB_D+-Pad3) -> VCC
- J9 pad 4: Net-(J9-3.3V-Pad2) -> GND
- L1 pad 1: unconnected-(L1-Pad1) -> Net-(D2-K)
- L1 pad 2: unconnected-(L1-Pad2) -> /POWER/+3V3
- L2 pad 1: unconnected-(L2-Pad1) -> Net-(D3-K)
- L2 pad 2: unconnected-(L2-Pad2) -> +5V
- R1 pad 1: unconnected-(R1-Pad1) -> Net-(U3-QOD)
- R1 pad 2: unconnected-(R1-Pad2) -> /POWER/USB_HOST_PWR
- U1 pad 11: unconnected-(U1-~{WAKEUP}/GPIO.3-Pad11) -> Net-(U1-AVSS-Pad11)
- U1 pad 2: Net-(U1-GND-Pad2) -> unconnected-(U1-LOADMOD-Pad2)
- U1 pad 25: Net-(U1-GND-Pad2) -> unconnected-(U1-P70_IRQ-Pad25)
- U10 pad 1: unconnected-(U10-GAIN-Pad1) -> Net-(U10-GND-Pad1)
- U11 pad 11: Net-(U11-AVSS-Pad11) -> unconnected-(U11-SD_MOSI-Pad11)
- U2 pad 1: Net-(U2-GND-Pad1) -> unconnected-(U2-SCL/SPC-Pad1)
- U2 pad 10: unconnected-(U2-IO25-Pad10) -> Net-(U2-GND-Pad10)
- U2 pad 11: unconnected-(U2-IO26-Pad11) -> Net-(U2-GND-Pad10)
- U2 pad 12: unconnected-(U2-IO27-Pad12) -> Net-(U2-GND-Pad10)
- U2 pad 13: unconnected-(U2-IO14-Pad13) -> Net-(U2-GND-Pad10)
- U2 pad 14: unconnected-(U2-IO12-Pad14) -> Net-(U2-GND-Pad10)
- U2 pad 9: unconnected-(U2-IO33-Pad9) -> Net-(U2-GND-Pad10)
- U3 pad 1: unconnected-(U3-VCC-Pad1) -> /POWER/USB_HOST_PWR
- U3 pad 2: unconnected-(U3-GND-Pad2) -> Net-(U3-QOD)
- U3 pad 3: unconnected-(U3-~{CS}-Pad3) -> Net-(U3-CT)
- U3 pad 4: unconnected-(U3-RESET-Pad4) -> GND
- U3 pad 5: unconnected-(U3-D/~{C}-Pad5) -> /POWER/EN_USB_HOST_PWR
- U3 pad 6: unconnected-(U3-MOSI-Pad6) -> +5V
- U3 pad 7: unconnected-(U3-SCK-Pad7) -> GND
- U4 pad 1: unconnected-(U4-Pad1) -> Net-(U4-BOOT)
- U4 pad 2: unconnected-(U4A---Pad2) -> +5V
- U4 pad 3: unconnected-(U4A-+-Pad3) -> Net-(D2-K)
- U4 pad 4: unconnected-(U4C-V--Pad4) -> GND
- U4 pad 5: unconnected-(U4B-+-Pad5) -> Net-(U4-VSENSE)
- U4 pad 6: unconnected-(U4B---Pad6) -> Net-(U4-COMP)
- U4 pad 7: unconnected-(U4-Pad7) -> Net-(U4-EN)
- U4 pad 8: unconnected-(U4C-V+-Pad8) -> Net-(U4-SS)
- U5 pad 1: unconnected-(U5-BOOT-Pad1) -> Net-(U5-BOOT)
- U5 pad 2: unconnected-(U5-PG-Pad2) -> /POWER/VIN
- U5 pad 3: unconnected-(U5-~{EN1}-Pad3) -> Net-(D3-K)
- U5 pad 4: unconnected-(U5-FB-Pad4) -> GND
- U5 pad 5: unconnected-(U5-EN2-Pad5) -> Net-(U5-VSENSE)
- U5 pad 6: unconnected-(U5-GND-Pad6) -> Net-(U5-COMP)
- U5 pad 7: unconnected-(U5-VIN-Pad7) -> Net-(U5-EN)
- U5 pad 8: unconnected-(U5-SW-Pad8) -> Net-(U5-SS)
- U5 pad 9: unconnected-(U5-PADGND-Pad9) -> GND
- U9 pad 1: Net-(U9-GND-Pad1) -> unconnected-(U9-D-Pad1)
Routing:
- net (no net): track 464.8 -> 0.00 mm
- removed copper zone on B.Cu, net (none)
Other:
- board outline removed
- board text removed: "+ A - ANALOG"
- board text removed: "+ G A B V - MOTOR"
- board text removed: "+MOMICKCS- SPI"
- board text removed: "+RXTX- CAN"
- board text removed: "+RXTX- SERIAL"
- board text removed: "+S- DIO"
- board text removed: "+S- PWM"
- board text removed: "+SDASCL- I2C"
- board text removed: "0"
- board text removed: "1"
- board text removed: "12V VBUS 3.3V HTR TYPE LED1 LED2 LED3 RGB"
- board text removed: "2"
- board text removed: "3"
- board text removed: "4"
- board text removed: "5"
- board text removed: "6"
- board text removed: "7"
- board text removed: "AUDIO"
- board text removed: "ESP32 USB"
- board text removed: "MCU USB"
- board text removed: "PHOTO-R"
- board text removed: "PWR"
- board text removed: "RESET"
- board text removed: "USB HOST"
- board text removed: "uSD CARD"

Commit message: Finished I2C device and bus schematics. Added logic level translation.
Parts:
- removed U13: PCF8574TS, Package_SO:SSOP-20_4.4x6.5mm_P0.65mm
- added C23: 10uF, Capacitor_SMD:C_0805_2012Metric, F.Cu at (201.1, 94.8)
- added C24: 100nF, Capacitor_SMD:C_0603_1608Metric, F.Cu at (200.9, 89.6)
- added Q3: BC850, Package_TO_SOT_SMD:SOT-23, F.Cu at (207.8, 97.1)
- added R16: 33k, Resistor_SMD:R_0603_1608Metric, F.Cu at (200.9, 92.1)
- added R17: 10k, Resistor_SMD:R_0603_1608Metric, F.Cu at (207.3, 110.8)
- added RN1: 4.7k, Resistor_SMD:R_Array_Concave_4x0603, F.Cu at (212.3, 97.1)
- added RV2: 10k, Potentiometer_SMD:Potentiometer_Bourns_3224J_Horizontal, F.Cu at (221.4, 104.8)
- added U17: TXS0108EPW, Package_SO:TSSOP-20_4.4x6.5mm_P0.65mm, F.Cu at (210.1, 105.5)
- added U18: PCA9306DC, Package_SO:VSSOP-8_2.3x2mm_P0.5mm, F.Cu at (217.6, 122.8)
- added U19: PCF8574, Package_SO:SSOP-20_4.4x6.5mm_P0.65mm, F.Cu at (218.9, 114.9)
- added U2: LIS2DH, Package_LGA:LGA-14_2x2mm_P0.35mm_LayoutBorder3x4y, F.Cu at (207.1, 115.9)
- D1: value D_IR_EMITTER -> D_Schottky; footprint LED_THT:LED_D5.0mm_Horizontal_O1.27mm_Z3.0mm_Clear -> Diode_SMD:D_SMB
- D12, D13: value LED_ABGR -> WS2812B; footprint LED_THT:LED_D5.0mm-4_RGB -> LED_SMD:LED_WS2812B_PLCC4_5.0x5.0mm_P3.2mm
- D15, D16, D17: value WS2812B -> LED; footprint LED_SMD:LED_WS2812B_PLCC4_5.0x5.0mm_P3.2mm -> LED_THT:LED_D5.0mm
- D2, D3, D4: value LED -> D_Schottky; footprint LED_THT:LED_D5.0mm -> Diode_SMD:D_SMB
- D21: value LED -> LED_ABGR; footprint LED_THT:LED_D5.0mm -> LED_THT:LED_D5.0mm-4_RGB
- D5: value WS2812B -> D_Schottky; footprint LED_SMD:LED_WS2812B_PLCC4_5.0x5.0mm_P3.2mm -> Diode_SMD:D_SMB
- D6: value LED -> D_IR_EMITTER; footprint LED_THT:LED_D5.0mm -> LED_THT:LED_D5.0mm_Horizontal_O1.27mm_Z3.0mm_Clear
- D7, D8: value LED -> WS2812B; footprint LED_THT:LED_D5.0mm -> LED_SMD:LED_WS2812B_PLCC4_5.0x5.0mm_P3.2mm
- J12: value USB_A -> MOTOR; footprint Connector_USB:USB_A_TE_292303-7_Horizontal -> Connector_JST:JST_XH_S6B-XH-A_1x06_P2.50mm_Horizontal
- J4: value PWM_OUT -> SERVO
- Q3: value NJFET -> BC850; footprint Package_TO_SOT_SMD:TO-252-3_TabPin2 -> Package_TO_SOT_SMD:SOT-23
- moved U15 173.2 mm to (65.0, 131.5), turned to 0 degrees
- moved J13 67.9 mm to (195.6, 38.0)
- moved J20 67.9 mm to (181.1, 38.0)
- moved J23 67.9 mm to (169.0, 38.0)
- moved J22 67.9 mm to (157.1, 38.0)
- moved J24 67.9 mm to (214.1, 43.5)
- moved D21 14.0 mm to (153.7, 55.5)
Connections:
- C4 pad 1: /POWER/USB_HOST_PWR -> /OUTPUTS/BREAKOUT_USB_VBUS
- D1 pad 1: unconnected-(D1-K-Pad1) -> /POWER/VIN
- D1 pad 2: unconnected-(D1-A-Pad2) -> Net-(D1-A)
- D12 pad 1: unconnected-(D12-A-Pad1) -> unconnected-(D12-VDD-Pad1)
- D12 pad 2: unconnected-(D12-BK-Pad2) -> unconnected-(D12-DOUT-Pad2)
- D12 pad 3: unconnected-(D12-GK-Pad3) -> unconnected-(D12-VSS-Pad3)
- D12 pad 4: unconnected-(D12-RK-Pad4) -> unconnected-(D12-DIN-Pad4)
- D13 pad 1: unconnected-(D13-A-Pad1) -> unconnected-(D13-VDD-Pad1)
- D13 pad 2: unconnected-(D13-BK-Pad2) -> unconnected-(D13-DOUT-Pad2)
- D13 pad 3: unconnected-(D13-GK-Pad3) -> unconnected-(D13-VSS-Pad3)
- D13 pad 4: unconnected-(D13-RK-Pad4) -> unconnected-(D13-DIN-Pad4)
- D15 pad 1: unconnected-(D15-VDD-Pad1) -> unconnected-(D15-K-Pad1)
- D15 pad 2: unconnected-(D15-DOUT-Pad2) -> unconnected-(D15-A-Pad2)
- D16 pad 1: unconnected-(D16-VDD-Pad1) -> unconnected-(D16-K-Pad1)
- D16 pad 2: unconnected-(D16-DOUT-Pad2) -> unconnected-(D16-A-Pad2)
- D17 pad 1: unconnected-(D17-VDD-Pad1) -> unconnected-(D17-K-Pad1)
- D17 pad 2: unconnected-(D17-DOUT-Pad2) -> unconnected-(D17-A-Pad2)
- D2 pad 1: unconnected-(D2-K-Pad1) -> Net-(D2-K)
- D2 pad 2: unconnected-(D2-A-Pad2) -> GND
- D21 pad 1: unconnected-(D21-K-Pad1) -> unconnected-(D21-A-Pad1)
- D21 pad 2: unconnected-(D21-A-Pad2) -> unconnected-(D21-BK-Pad2)
- D3 pad 1: unconnected-(D3-K-Pad1) -> Net-(D3-K)
- D3 pad 2: unconnected-(D3-A-Pad2) -> GND
- D5 pad 1: unconnected-(D5-VDD-Pad1) -> unconnected-(D5-K-Pad1)
- D5 pad 2: unconnected-(D5-DOUT-Pad2) -> unconnected-(D5-A-Pad2)
- D7 pad 1: unconnected-(D7-K-Pad1) -> unconnected-(D7-VDD-Pad1)
- D7 pad 2: unconnected-(D7-A-Pad2) -> unconnected-(D7-DOUT-Pad2)
- D8 pad 1: unconnected-(D8-K-Pad1) -> unconnected-(D8-VDD-Pad1)
- D8 pad 2: unconnected-(D8-A-Pad2) -> unconnected-(D8-DOUT-Pad2)
- DS1 pad 1: unconnected-(DS1-VSS-Pad1) -> GND
- DS1 pad 11: unconnected-(DS1-D4-Pad11) -> Net-(DS1-D4)
- DS1 pad 12: unconnected-(DS1-D5-Pad12) -> Net-(DS1-D5)
- DS1 pad 13: unconnected-(DS1-D6-Pad13) -> Net-(DS1-D6)
- DS1 pad 14: unconnected-(DS1-D7-Pad14) -> Net-(DS1-D7)
- DS1 pad 15: unconnected-(DS1-LED(+)-Pad15) -> +5V
- DS1 pad 16: unconnected-(DS1-LED(-)-Pad16) -> Net-(DS1-LED(-))
- DS1 pad 2: unconnected-(DS1-VDD-Pad2) -> +5V
- DS1 pad 3: unconnected-(DS1-VO-Pad3) -> Net-(DS1-VO)
- DS1 pad 4: unconnected-(DS1-RS-Pad4) -> Net-(DS1-RS)
- DS1 pad 5: unconnected-(DS1-R/W-Pad5) -> Net-(DS1-R/W)
- DS1 pad 6: unconnected-(DS1-E-Pad6) -> Net-(DS1-E)
- J10 pad 3: VCC -> /OUTPUTS/BREAKOUT_VCC
- J11 pad 3: VCC -> /OUTPUTS/BREAKOUT_VCC
- J12 pad 1: unconnected-(J12-VBUS-Pad1) -> /OUTPUTS/BREAKOUT_MOTOR_PWM1_1
- J12 pad 2: unconnected-(J12-D--Pad2) -> /OUTPUTS/BREAKOUT_MOTOR_PWM2_1
- J12 pad 3: unconnected-(J12-D+-Pad3) -> /OUTPUTS/BREAKOUT_MOTOR_C1_1
- J12 pad 4: unconnected-(J12-GND-Pad4) -> /OUTPUTS/BREAKOUT_MOTOR_C2_1
- J12 pad 5: unconnected-(J12-Shield-Pad5) -> /POWER/VIN
- J2 pad 2: VCC -> /OUTPUTS/BREAKOUT_VCC
- J20 pad 3: VCC -> /OUTPUTS/BREAKOUT_VCC
- J21 pad 2: VCC -> /OUTPUTS/BREAKOUT_VCC
- J22 pad 2: VCC -> /OUTPUTS/BREAKOUT_VCC
- J23 pad 2: VCC -> /OUTPUTS/BREAKOUT_VCC
- J3 pad 2: VCC -> /OUTPUTS/BREAKOUT_VCC
- J4 pad 2: VCC -> /OUTPUTS/BREAKOUT_VCC
- J4 pad 1: unconnected-(J4-Pin_1-Pad1) -> /OUTPUTS/BREAKOUT_SERVO_2
- J4 pad 2: unconnected-(J4-Pin_2-Pad2) -> /OUTPUTS/BREAKOUT_VCC
- J4 pad 3: unconnected-(J4-Pin_3-Pad3) -> GND
- J5 pad 2: VCC -> /OUTPUTS/BREAKOUT_VCC
- J6 pad 2: VCC -> /OUTPUTS/BREAKOUT_VCC
- J7 pad 2: VCC -> /OUTPUTS/BREAKOUT_VCC
- J8 pad 5: VCC -> /OUTPUTS/BREAKOUT_VCC
- J9 pad 1: /OUTPUTS/BREAKOUT_I2C_SDA -> /I2C/I2C_SDA_BREAKOUT
- J9 pad 2: /OUTPUTS/BREAKOUT_I2C_SCL -> /I2C/I2C_SCL_BREAKOUT
- J9 pad 3: VCC -> /OUTPUTS/BREAKOUT_VCC
- Q3 pad 1: unconnected-(Q3-D-Pad1) -> Net-(Q3-B)
- Q3 pad 2: unconnected-(Q3-G-Pad2) -> GND
- Q3 pad 3: unconnected-(Q3-S-Pad3) -> Net-(DS1-LED(-))
- R1 pad 2: /POWER/USB_HOST_PWR -> /OUTPUTS/BREAKOUT_USB_VBUS
- U15 pad 1: unconnected-(U15-e-Pad1) -> Net-(U14-SEG_E)
- U15 pad 10: unconnected-(U15-f-Pad10) -> Net-(U14-SEG_F)
- U15 pad 11: unconnected-(U15-a-Pad11) -> Net-(U14-SEG_A)
- U15 pad 12: unconnected-(U15-CC1-Pad12) -> Net-(U14-DIG_0)
- U15 pad 2: unconnected-(U15-d-Pad2) -> Net-(U14-SEG_D)
- U15 pad 3: unconnected-(U15-DPX-Pad3) -> Net-(U14-SEG_DP)
- U15 pad 4: unconnected-(U15-c-Pad4) -> Net-(U14-SEG_C)
- U15 pad 5: unconnected-(U15-g-Pad5) -> Net-(U14-SEG_G)
- U15 pad 6: unconnected-(U15-CC4-Pad6) -> Net-(U14-DIG_3)
- U15 pad 7: unconnected-(U15-b-Pad7) -> Net-(U14-SEG_B)
- U15 pad 8: unconnected-(U15-CC3-Pad8) -> Net-(U14-DIG_2)
- U15 pad 9: unconnected-(U15-CC2-Pad9) -> Net-(U14-DIG_1)
- U3 pad 1: /POWER/USB_HOST_PWR -> /OUTPUTS/BREAKOUT_USB_VBUS

Commit message: SPI SD CARD circuit added.
Parts:
- removed J14: Micro_SD_Card_Det2, Connector_Card:microSD_HC_Hirose_DM3AT-SF-PEJM5
- removed U2 (x2): LIS2DH, Package_LGA:LGA-14_2x2mm_P0.35mm_LayoutBorder3x4y
- added C32: 1uF, Capacitor_SMD:C_0603_1608Metric, F.Cu at (244.8, 103.2)
- added C33: 100nF, Capacitor_SMD:C_0603_1608Metric, F.Cu at (244.8, 105.7)
- added C34: 100nF C0G, Capacitor_SMD:C_1206_3216Metric, F.Cu at (239.5, 111.2)
- added C35: 47uF, Capacitor_SMD:C_1210_3225Metric, F.Cu at (239.5, 118.3)
- added C36: 10uF, Capacitor_SMD:C_1206_3216Metric, F.Cu at (239.5, 114.5)
- added C38: 10uF, Capacitor_SMD:C_1206_3216Metric, F.Cu at (243.2, 77.3)
- added C39: 100nF, Capacitor_SMD:C_0805_2012Metric, F.Cu at (242.6, 90.0)
- added D24: SD05_SOD323, Diode_SMD:D_SOD-323, F.Cu at (244.5, 111.0)
- added D25: SD05_SOD323, Diode_SMD:D_SOD-323, F.Cu at (244.5, 113.9)
- added Q4: DMP2045U-7, Package_TO_SOT_SMD:SOT-23, F.Cu at (242.8, 86.3)
- added R22: 1k, Resistor_SMD:R_0805_2012Metric, F.Cu at (234.5, 103.4)
- added R23: 1k, Resistor_SMD:R_0805_2012Metric, F.Cu at (234.5, 106.3)
- added R24: 68k, Resistor_SMD:R_0805_2012Metric, F.Cu at (234.5, 109.3)
- added R25: 100, Resistor_SMD:R_0805_2012Metric, F.Cu at (234.5, 112.2)
- added R26: 220k, Resistor_SMD:R_0805_2012Metric, F.Cu at (234.5, 115.2)
- added R27: 220k, Resistor_SMD:R_0805_2012Metric, F.Cu at (234.5, 118.2)
- added R28: 220k, Resistor_SMD:R_0805_2012Metric, F.Cu at (234.5, 121.1)
- added R29: 1k, Resistor_SMD:R_0805_2012Metric, F.Cu at (234.5, 124.0)
- added R30: 10k, Resistor_SMD:R_0603_1608Metric, F.Cu at (242.3, 69.3)
- added R37: 10k, Resistor_SMD:R_0603_1608Metric, F.Cu at (242.3, 71.8)
- added R38: 100, Resistor_SMD:R_0603_1608Metric, F.Cu at (242.3, 74.3)
- added RN2: 10k, Resistor_SMD:R_Array_Convex_5x0603, F.Cu at (52.4, 138.4)
- added RN3: 4.7k, Resistor_SMD:R_Array_Convex_4x0603, F.Cu at (40.9, 147.0)
- added RN5: 10k, Resistor_SMD:R_Array_Convex_5x0603, F.Cu at (250.1, 70.5)
- added RV3: 2k, Potentiometer_SMD:Potentiometer_Bourns_3314J_Vertical, F.Cu at (239.7, 105.7)
- added TP1: A1, TestPoint:TestPoint_Pad_D3.0mm, F.Cu at (244.4, 123.0)
- added U13: SN74LVC1T45DBV, Package_TO_SOT_SMD:SOT-23-6, F.Cu at (51.4, 147.1)
- added U20: LIS2DH12TR, Package_LGA:LGA-12_2x2mm_P0.5mm, F.Cu at (45.0, 146.7)
- added U21: DRV8870DDA, Package_SO:Texas_HTSOP-8-1EP_3.9x4.9mm_P1.27mm_EP2.95x4.9mm_Mask2.4x3.1mm_ThermalVias, F.Cu at (43.6, 139.4)
- added U22: IP4252CZ16, Package_SON:Nexperia_HUSON-16_USON-16-1EP_1.35x3.3mm_P0.4mm_EP0.4x2.8mm, F.Cu at (234.8, 65.3)
- added U23: MCP6021RT-E/OT, Package_TO_SOT_SMD:SOT-23-5, F.Cu at (239.3, 122.8)
- BZ1: footprint Buzzer_Beeper:MagneticBuzzer_ProSignal_ABI-010-RC -> Buzzer_Beeper:Buzzer_Mallory_AST1240MLQ
- J6: value A_IN -> DM3BT-DSF-PEJS/C; footprint Connector_JST:JST_XH_S3B-XH-A_1x03_P2.50mm_Horizontal -> Connector_Card:microSD_HC_Hirose_DM3BT-DSF-PEJS
- RN1: footprint Resistor_SMD:R_Array_Concave_4x0603 -> Resistor_SMD:R_Array_Convex_4x0603
- U12: value PCF8574TS -> PCF8574
- moved J6 119.1 mm to (232.0, 77.4)
- moved BZ1 46.0 mm to (161.5, 89.0)
Connections:
- net /OUTPUTS/BREAKOUT_SPI_MOSI renamed /SPI/MOSI
- net /OUTPUTS/BREAKOUT_SPI_MSIO renamed /SPI/MISO
- net /OUTPUTS/BREAKOUT_SPI_SCK renamed /SPI/CLK
- J19 pad 1: unconnected-(J19-Pin_1-Pad1) -> Net-(J19-Pin_1)
- J19 pad 2: unconnected-(J19-Pin_2-Pad2) -> Net-(J19-Pin_2)
- J19 pad 3: unconnected-(J19-Pin_3-Pad3) -> Net-(J19-Pin_3)
- J19 pad 4: unconnected-(J19-Pin_4-Pad4) -> Net-(J19-Pin_4)
- J19 pad 5: unconnected-(J19-Pin_5-Pad5) -> Net-(J19-Pin_5)
- J19 pad 6: unconnected-(J19-Pin_6-Pad6) -> Net-(J19-Pin_6)
- J19 pad 7: unconnected-(J19-Pin_7-Pad7) -> Net-(J19-Pin_7)
- J19 pad 8: unconnected-(J19-Pin_8-Pad8) -> Net-(J19-Pin_8)
- J6 pad 1: /OUTPUTS/BREAKOUT_A_IN_0 -> unconnected-(J6-DAT2-Pad1)
- J6 pad 2: /OUTPUTS/BREAKOUT_VCC -> /SPI/micro_SD/SD_CS-CS
- J6 pad 3: GND -> /SPI/micro_SD/SD_DI-MOSI
- J8 pad 1: /OUTPUTS/BREAKOUT_SPI_CS -> /SPI/CS_BREAKOUT
- RN1 pad 2: /I2C/I2C_SCL_BREAKOUT -> Net-(JP5-B)
- RN1 pad 3: /I2C/I2C_SDA_BREAKOUT -> Net-(JP3-B)
- RN1 pad 5: Net-(JP2-B) -> Net-(Q3-B)
- RN1 pad 6: Net-(JP3-B) -> (no net)
- RN1 pad 7: Net-(Q3-B) -> (no net)
- U12 pad 1: unconnected-(U12-~{INT}-Pad1) -> Net-(JP5-B)
- U12 pad 10: unconnected-(U12-P0-Pad10) -> Net-(DS1-D5)
- U12 pad 11: unconnected-(U12-P1-Pad11) -> Net-(DS1-D6)
- U12 pad 12: unconnected-(U12-P2-Pad12) -> Net-(DS1-D7)
- U12 pad 14: unconnected-(U12-P3-Pad14) -> /I2C/I2C_SCL_BREAKOUT
- U12 pad 15: unconnected-(U12-VSS-Pad15) -> /I2C/I2C_SDA_BREAKOUT
- U12 pad 16: unconnected-(U12-P4-Pad16) -> +5V
- U12 pad 17: unconnected-(U12-P5-Pad17) -> (no net)
- U12 pad 18: unconnected-(U12-NC-Pad18) -> (no net)
- U12 pad 19: unconnected-(U12-P6-Pad19) -> (no net)
- U12 pad 2: unconnected-(U12-SCL-Pad2) -> Net-(JP3-B)
- U12 pad 20: unconnected-(U12-P7-Pad20) -> (no net)
- U12 pad 3: unconnected-(U12-NC-Pad3) -> Net-(JP1-B)
- U12 pad 4: unconnected-(U12-SDA-Pad4) -> Net-(DS1-RS)
- U12 pad 5: unconnected-(U12-VDD-Pad5) -> Net-(DS1-R/W)
- U12 pad 6: unconnected-(U12-A0-Pad6) -> Net-(DS1-E)
- U12 pad 7: unconnected-(U12-A1-Pad7) -> Net-(Q3-B)
- U12 pad 8: unconnected-(U12-NC-Pad8) -> GND
- U12 pad 9: unconnected-(U12-A2-Pad9) -> Net-(DS1-D4)
- U17 pad 12: unconnected-(U17-B8-Pad12) -> /SPI/CS_AUDIO
- U17 pad 13: unconnected-(U17-B7-Pad13) -> /SPI/CS_TFT
- U17 pad 14: unconnected-(U17-B6-Pad14) -> /SPI/CS_NFC
- U17 pad 15: unconnected-(U17-B5-Pad15) -> /SPI/CS_BREAKOUT
- U17 pad 16: /SPI/7segment driver/SPI_CS_SEVENSEG -> /SPI/CS_SEVENSEG
- U17 pad 4: /SPI/SPI_SCK -> /SPI/SPI_CLK
- U17 pad 6: /SPI/SPI_CS_SDCARD -> /SPI/SPI_CS_BREAKOUT_IN
- U18 pad 4: /I2C/I2C_SDA -> /I2C/I2C_SCL
- U18 pad 8: unconnected-(U18-EN-Pad8) -> Net-(U18-EN)
- U19 pad 1: Net-(JP1-B) -> Net-(JP6-B)
- U19 pad 10: Net-(DS1-D5) -> Net-(J19-Pin_6)
- U19 pad 11: Net-(DS1-D6) -> Net-(J19-Pin_7)
- U19 pad 12: Net-(DS1-D7) -> Net-(J19-Pin_8)
- U19 pad 13: unconnected-(U19-~{INT}-Pad13) -> /I2C/I2C Devices/INTERRUPT_KEYPAD
- U19 pad 2: Net-(JP2-B) -> Net-(JP4-B)
- U19 pad 3: Net-(JP3-B) -> Net-(JP2-B)
- U19 pad 4: Net-(DS1-RS) -> Net-(J19-Pin_1)
- U19 pad 5: Net-(DS1-R/W) -> Net-(J19-Pin_2)
- U19 pad 6: Net-(DS1-E) -> Net-(J19-Pin_3)
- U19 pad 7: Net-(Q3-B) -> Net-(J19-Pin_4)
- U19 pad 9: Net-(DS1-D4) -> Net-(J19-Pin_5)
- U8 pad 1: unconnected-(U8-SDA-Pad1) -> /I2C/I2C_SCL
- U8 pad 2: unconnected-(U8-GND-Pad2) -> GND
- U8 pad 5: unconnected-(U8-VCC-Pad5) -> +3.3V
- U8 pad 6: unconnected-(U8-SCL-Pad6) -> /I2C/I2C_SCL
