File: PRODIGY-MOTHERBOARD/PRODIGY-MOTHERBOARD.kicad_pcb (KiCad board)
At the start: 2 copper layers, 204 parts, among them J10 GPIO, J11 SPI_OUT, J12 I2C, J13 CAN, J14 SERIAL, J15 12V OUT, J16 SERVO, J17 SERVO, J18 SERVO, J19 Ultrasonic, J20 MOTOR, J21 MOTOR, J22 DM3BT-DSF-PEJS/C, J23 Barrel_Jack_MountingPin, J26 KEYPAD_MATRIX, J28 AudioJack4, J4 USB_A, J5 A_OUT, J6 Neopixel, J7 GPIO, J8 GPIO, J9 GPIO, P1 USB_C_Plug, Q1 DMP2045U-7, Q2 BC850, Q3 BC850, Q4 BS870, Q5 BC850, Q6 ALS-PDIC15-21B/TR8, U10 TJA1051T-E, U11 DRV8870DDA, U12 DRV8870DDA, U13 PCA9306DC, U14 SN74LVC1T45DBV, U15 TXS0108EPW, U16 CR2013-MI2120, U17 PCF8574, U18 PCF8574, U19 HDC1080, U2 CC56-12YWA, U20 LIS2DH12TR, U21 MCP6021RT-E/OT, U22 SN74LVC1T45DBV, U23 TSDP341xx, U3 PN5321A3HN_C1xx, U4 IP4252CZ16, U5 TPS22810DRV, U6 TPS54331DR, U7 TPS54331DR, U8 Si4460, U9 LM386

Commit message: Added pins to MCU. Added Decoder for SPI SS-Multiplexing.
Parts:
- added D33: SD05_SOD323, Diode_SMD:D_SOD-323, F.Cu at (179.6, 78.9)
- added D34: SD05_SOD323, Diode_SMD:D_SOD-323, F.Cu at (179.6, 81.9)
- added D35: SD05_SOD323, Diode_SMD:D_SOD-323, F.Cu at (179.6, 84.8)
- added R80: 1k, Resistor_SMD:R_0603_1608Metric, F.Cu at (185.7, 88.0)
- added U24: CS43L21, Package_DFN_QFN:QFN-32-1EP_5x5mm_P0.5mm_EP3.45x3.45mm, F.Cu at (187.3, 81.1)
- MK1: value Microphone_Condenser -> Mic; footprint Buzzer_Beeper:MagneticBuzzer_Kingstate_KCG0601 -> Sensor_Audio:POM-2244P-C3310-2-R
Connections:
- Q5 pad 1: /digital/DIGITAL_BUZZER_IN -> Net-(Q5-B)
- RV4 pad 1: unconnected-(RV4-VIN-Pad1) -> +3V3
- RV4 pad 2: unconnected-(RV4-RVX-Pad2) -> /analog/ANALOG_JOYSTICK_X_OUT
- RV4 pad 3: unconnected-(RV4-GND-Pad3) -> GND
- RV4 pad 4: unconnected-(RV4-VIN-Pad4) -> +3V3
- RV4 pad 5: unconnected-(RV4-RVY-Pad5) -> /analog/ANALOG_JOYSTICK_Y_OUT
- RV4 pad 6: unconnected-(RV4-GND-Pad6) -> GND
- U16 pad 1: unconnected-(U16-VCC-Pad1) -> +3V3
- U16 pad 2: unconnected-(U16-GND-Pad2) -> GND
- U16 pad 3: unconnected-(U16-~{CS}-Pad3) -> /SPI/SPI_CS_TFT
- U16 pad 5: unconnected-(U16-D/~{C}-Pad5) -> /SPI/SPI_MODE_TFT
- U16 pad 6: unconnected-(U16-MOSI-Pad6) -> /SPI/SPI_MOSI
- U16 pad 7: unconnected-(U16-SCK-Pad7) -> /SPI/SPI_CLK
- U16 pad 9: unconnected-(U16-MISO-Pad9) -> /SPI/SPI_MISO

Commit message: Added proper debounce filter elements to buttons.
Parts:
- removed D18: WS2812B, LED_SMD:LED_WS2812B_PLCC4_5.0x5.0mm_P3.2mm
- removed J11: SPI_OUT, Connector_JST:JST_XH_S6B-XH-A_1x06_P2.50mm_Horizontal
- removed J28: AudioJack4, Connector_Audio:Jack_3.5mm_KoreanHropartsElec_PJ-320D-4A_Horizontal
- removed J4: USB_A, Connector_USB:USB_A_TE_292303-7_Horizontal
- removed J8: GPIO, Connector_JST:JST_XH_S3B-XH-A_1x03_P2.50mm_Horizontal
- removed P1: USB_C_Plug, Connector_USB:USB_C_Receptacle_GCT_USB4105-xx-A_16P_TopMnt_Horizontal
- removed R80: 1k, Resistor_SMD:R_0603_1608Metric
- added C39: 47uF, Capacitor_SMD:C_1210_3225Metric, F.Cu at (219.2, 71.3)
- added C40: 100nF, Capacitor_SMD:C_0603_1608Metric, F.Cu at (208.7, 62.1)
- added C41: 4.7uF, Capacitor_SMD:C_1206_3216Metric, F.Cu at (213.5, 70.8)
- added C42: 4.7uF, Capacitor_SMD:C_1206_3216Metric, F.Cu at (213.5, 74.2)
- added C43: 100nF, Capacitor_SMD:C_0603_1608Metric, F.Cu at (208.7, 64.7)
- added C46: 10nF, Capacitor_SMD:C_0603_1608Metric, F.Cu at (208.7, 67.2)
- added C47: 1nF, Capacitor_SMD:C_0603_1608Metric, F.Cu at (208.7, 69.7)
- added C48: 47pF, Capacitor_SMD:C_0603_1608Metric, F.Cu at (208.7, 72.2)
- added C49: 100nF, Capacitor_SMD:C_0603_1608Metric, F.Cu at (208.7, 86.6)
- added C55: 47uF, Capacitor_SMD:CP_Elec_6.3x5.8, F.Cu at (251.4, 79.0)
- added C65: 1uF, Capacitor_SMD:C_0603_1608Metric, F.Cu at (241.6, 62.1)
- added C66: 100nF, Capacitor_SMD:C_0603_1608Metric, F.Cu at (241.6, 64.7)
- added C67: 47uF, Capacitor_SMD:C_1210_3225Metric, F.Cu at (236.8, 69.7)
- added C68: 100nF C0G, Capacitor_SMD:C_1206_3216Metric, F.Cu at (236.8, 62.6)
- added C69: 10uF, Capacitor_SMD:C_1206_3216Metric, F.Cu at (236.8, 65.9)
- added C79: 4.7uF, Capacitor_SMD:C_0603_1608Metric, F.Cu at (219.7, 29.8)
- added C80: 4.7uF, Capacitor_SMD:C_0603_1608Metric, F.Cu at (219.7, 32.3)
- added C81: 4.7uF, Capacitor_SMD:C_0603_1608Metric, F.Cu at (219.7, 34.9)
- added D27: WS2812B, LED_SMD:LED_WS2812B_PLCC4_5.0x5.0mm_P3.2mm, F.Cu at (225.9, 31.9)
- added D29: WS2812B, LED_SMD:LED_WS2812B_PLCC4_5.0x5.0mm_P3.2mm, F.Cu at (225.9, 38.5)
- added D37: LED, LED_THT:LED_D5.0mm, F.Cu at (209.1, 24.8)
- added D38: LED, LED_THT:LED_D5.0mm, F.Cu at (216.6, 24.8)
- added D39: LED, LED_THT:LED_D5.0mm, F.Cu at (224.1, 24.8)
- added D40: LED, LED_THT:LED_D5.0mm, F.Cu at (231.6, 24.8)
- added D41: LED, LED_THT:LED_D5.0mm, F.Cu at (239.1, 24.8)
- added D42: D_IR_EMITTER, LED_THT:LED_D5.0mm_Horizontal_O1.27mm_Z3.0mm_Clear, F.Cu at (232.6, 30.4)
- added D43: SD05_SOD323, Diode_SMD:D_SOD-323, F.Cu at (271.2, 22.5)
- added D44: SD05_SOD323, Diode_SMD:D_SOD-323, F.Cu at (271.2, 25.4)
- added D45: SD05_SOD323, Diode_SMD:D_SOD-323, F.Cu at (271.2, 28.4)
- added D46: SD05_SOD323, Diode_SMD:D_SOD-323, F.Cu at (271.2, 31.4)
- added D47: SD05_SOD323, Diode_SMD:D_SOD-323, F.Cu at (271.2, 34.3)
- added D48: SD05_SOD323, Diode_SMD:D_SOD-323, F.Cu at (271.2, 37.2)
- added D49: SD05_SOD323, Diode_SMD:D_SOD-323, F.Cu at (271.2, 40.2)
- added J27: KEYPAD_MATRIX, Connector_PinHeader_2.54mm:PinHeader_1x08_P2.54mm_Vertical_SMD_Pin1Left, F.Cu at (227.9, 72.1)
- added L4: 6.8, Inductor_SMD:L_Chilisin_BMRB00060624, F.Cu at (215.7, 65.0)
- added L5: L_Iron_Coupled_1324, Inductor_SMD:L_CommonModeChoke_TDK_ACM7060, F.Cu at (212.0, 81.6)
- added R30: 2, Resistor_SMD:R_2512_6332Metric, F.Cu at (250.5, 85.5)
- added R31: 5.1k, Resistor_SMD:R_0603_1608Metric, F.Cu at (260.6, 76.1)
- added R32: 5.1k, Resistor_SMD:R_0603_1608Metric, F.Cu at (260.6, 78.6)
- added R33: 10k, Resistor_SMD:R_0603_1608Metric, F.Cu at (260.6, 81.2)
- added R34: 10k, Resistor_SMD:R_0603_1608Metric, F.Cu at (260.6, 83.7)
- added R69: 100, Resistor_SMD:R_0603_1608Metric, F.Cu at (219.7, 37.4)
- added R70: 10k, Resistor_SMD:R_0603_1608Metric, F.Cu at (219.7, 39.9)
- added R71: 39, Resistor_SMD:R_0603_1608Metric, F.Cu at (219.7, 42.4)
- added R72: 100, Resistor_SMD:R_0603_1608Metric, F.Cu at (219.7, 44.9)
- added SW1: SW_Push, Button_Switch_SMD:SW_Push_1P1T_NO_CK_KMR2, F.Cu at (237.2, 76.2)
- added SW2: SW_Push, Button_Switch_SMD:SW_Push_1P1T_NO_CK_KMR2, F.Cu at (265.9, 77.2)
- added SW3: SW_Push, Button_Switch_SMD:SW_Push_1P1T_NO_6x6mm_H9.5mm, F.Cu at (225.5, 132.5)
- added SW4: SW_Push, Button_Switch_SMD:SW_Push_1P1T_NO_6x6mm_H9.5mm, F.Cu at (234.5, 124.0)
- added SW5: SW_Push, Button_Switch_SMD:SW_Push_1P1T_NO_6x6mm_H9.5mm, F.Cu at (234.5, 140.0)
- added SW7: SW_Push, Button_Switch_SMD:SW_Push_1P1T_NO_6x6mm_H9.5mm, F.Cu at (243.5, 133.0)
- added U1: CC56-12YWA, Display_7Segment:CC56-12YWA, F.Cu at (249.1, 40.6)
- C25: value 100nF -> 10uF; footprint Capacitor_SMD:C_0603_1608Metric -> Capacitor_SMD:C_1206_3216Metric
- C26: value 10nF -> 100nF; footprint Capacitor_SMD:C_0603_1608Metric -> Capacitor_SMD:C_0805_2012Metric
- C27: value 10nF -> 100nF
- C28: value 1nF -> 4.7uF; footprint Capacitor_SMD:C_0603_1608Metric -> Capacitor_SMD:C_1206_3216Metric
- C29: value 4.7nF -> 4.7uF; footprint Capacitor_SMD:C_0603_1608Metric -> Capacitor_SMD:C_1206_3216Metric
- C30: value 47pF -> 100nF
- C31: value 39pF -> 47uF; footprint Capacitor_SMD:C_0603_1608Metric -> Capacitor_SMD:C_1210_3225Metric
- C32: value 100nF -> 47uF; footprint Capacitor_SMD:C_0603_1608Metric -> Capacitor_SMD:C_1210_3225Metric
- C33: value 100nF -> 100uF; footprint Capacitor_SMD:C_0603_1608Metric -> Capacitor_SMD:CP_Elec_6.3x7.7
- C34: value 47uF -> 10nF; footprint Capacitor_SMD:C_1210_3225Metric -> Capacitor_SMD:C_0603_1608Metric
- C35: value 47uF -> 4.7nF; footprint Capacitor_SMD:C_1210_3225Metric -> Capacitor_SMD:C_0603_1608Metric
- C36: value 47uF -> 39pF; footprint Capacitor_SMD:C_1210_3225Metric -> Capacitor_SMD:C_0603_1608Metric
- C37: value 47uF -> 4.7uF; footprint Capacitor_SMD:C_1210_3225Metric -> Capacitor_SMD:C_1206_3216Metric
- C38: value 100nF -> 22nF
- C44, C45: footprint Capacitor_SMD:CP_Elec_6.3x5.8 -> Capacitor_SMD:C_1210_3225Metric
- D10, D11, D8: value SD05_SOD323 -> D_Schottky; footprint Diode_SMD:D_SOD-323 -> Diode_SMD:D_SMB
- D12, D13: value LED -> SD05_SOD323; footprint LED_THT:LED_D5.0mm -> Diode_SMD:D_SOD-323
- D14: value LED -> 1N4148W; footprint LED_THT:LED_D5.0mm -> Diode_SMD:D_SOD-123
- D15, D19, D20: value WS2812B -> SD05_SOD323; footprint LED_SMD:LED_WS2812B_PLCC4_5.0x5.0mm_P3.2mm -> Diode_SMD:D_SOD-323
- D16: value D_IR_EMITTER -> 1N4148W; footprint LED_THT:LED_D5.0mm_Horizontal_O1.27mm_Z3.0mm_Clear -> Diode_SMD:D_SOD-123
- D17, D25, D26: value WS2812B -> 1N4148W; footprint LED_SMD:LED_WS2812B_PLCC4_5.0x5.0mm_P3.2mm -> Diode_SMD:D_SOD-123
- D21, D22, D23, D28: value LED -> WS2812B; footprint LED_THT:LED_D5.0mm -> LED_SMD:LED_WS2812B_PLCC4_5.0x5.0mm_P3.2mm
- D30: value 1N4148W -> WS2812B; footprint Diode_SMD:D_SOD-123 -> LED_SMD:LED_WS2812B_PLCC4_5.0x5.0mm_P3.2mm
- D33, D34: value SD05_SOD323 -> LED; footprint Diode_SMD:D_SOD-323 -> LED_THT:LED_D5.0mm
- D35: value SD05_SOD323 -> 1N4148W; footprint Diode_SMD:D_SOD-323 -> Diode_SMD:D_SOD-123
- D4: value D_Schottky -> 1N4148W; footprint Diode_SMD:D_SMB -> Diode_SMD:D_SOD-123
- D5, D6: value D_Schottky -> SD05_SOD323; footprint Diode_SMD:D_SMB -> Diode_SMD:D_SOD-323
- J10: value GPIO -> I2C; footprint Connector_JST:JST_XH_S3B-XH-A_1x03_P2.50mm_Horizontal -> Connector_JST:JST_XH_S4B-XH-A_1x04_P2.50mm_Horizontal
- J12: value I2C -> Neopixel; footprint Connector_JST:JST_XH_S4B-XH-A_1x04_P2.50mm_Horizontal -> Connector_JST:JST_XH_S3B-XH-A_1x03_P2.50mm_Horizontal
- J13: value CAN -> GPIO; footprint Connector_JST:JST_XH_S4B-XH-A_1x04_P2.50mm_Horizontal -> Connector_JST:JST_XH_S3B-XH-A_1x03_P2.50mm_Horizontal
- J14: value SERIAL -> CAN
- J15: value 12V OUT -> MOTOR; footprint TerminalBlock_Phoenix:TerminalBlock_Phoenix_MKDS-1,5-2-5.08_1x02_P5.08mm_Horizontal -> Connector_JST:JST_XH_S6B-XH-A_1x06_P2.50mm_Horizontal
- J17: value SERVO -> GPIO
- J18: value SERVO -> SERIAL; footprint Connector_JST:JST_XH_S3B-XH-A_1x03_P2.50mm_Horizontal -> Connector_JST:JST_XH_S4B-XH-A_1x04_P2.50mm_Horizontal
- J19: value Ultrasonic -> 12V OUT; footprint Connector_JST:JST_XH_S4B-XH-A_1x04_P2.50mm_Horizontal -> TerminalBlock_Phoenix:TerminalBlock_Phoenix_MKDS-1,5-2-5.08_1x02_P5.08mm_Horizontal
- J20: value MOTOR -> USB_A; footprint Connector_JST:JST_XH_S6B-XH-A_1x06_P2.50mm_Horizontal -> Connector_USB:USB_A_TE_292303-7_Horizontal
- J21: value MOTOR -> DM3BT-DSF-PEJS/C; footprint Connector_JST:JST_XH_S6B-XH-A_1x06_P2.50mm_Horizontal -> Connector_Card:microSD_HC_Hirose_DM3BT-DSF-PEJS
- J22: value DM3BT-DSF-PEJS/C -> Barrel_Jack_MountingPin; footprint Connector_Card:microSD_HC_Hirose_DM3BT-DSF-PEJS -> Connector_BarrelJack:BarrelJack_CUI_PJ-063AH_Horizontal
- J23: value Barrel_Jack_MountingPin -> AudioJack4; footprint Connector_BarrelJack:BarrelJack_CUI_PJ-063AH_Horizontal -> Connector_Audio:Jack_3.5mm_KoreanHropartsElec_PJ-320D-4A_Horizontal
- J6: value Neopixel -> SPI_OUT; footprint Connector_JST:JST_XH_S3B-XH-A_1x03_P2.50mm_Horizontal -> Connector_JST:JST_XH_S6B-XH-A_1x06_P2.50mm_Horizontal
- L3: value L_Iron_Coupled_1324 -> 6.8; footprint Inductor_SMD:L_CommonModeChoke_TDK_ACM7060 -> Inductor_SMD:L_Chilisin_BMRB00060624
- R1: value 10k -> 5.1k
- R11, R13: value 330k -> 10k
- R12: value 68k -> 100
- R14: value 68k -> 330k
- R15: value 29.4k -> 10k 1%
- R16: value 50k -> 68k
- R17: value 10k 1% -> 1k 1%
- R18: value 2.2k 1% -> 680 1%
- R19: value 1k 1% -> 50k
- R2: value 100 -> 5.1k
- R20: value 10k 1% -> 220 1%
- R21: value 1k 1% -> DNP
- R22: value 680 1% -> 330k
- R23: value 220 1% -> 68k
- R24: value 59 -> 10k 1%; footprint Resistor_SMD:R_1206_3216Metric -> Resistor_SMD:R_0603_1608Metric
- R25: value 59 -> 2.2k 1%; footprint Resistor_SMD:R_1206_3216Metric -> Resistor_SMD:R_0603_1608Metric
- R26: value 2 -> 29.4k; footprint Resistor_SMD:R_2512_6332Metric -> Resistor_SMD:R_0603_1608Metric
- R27: value 2 -> 1k 1%; footprint Resistor_SMD:R_2512_6332Metric -> Resistor_SMD:R_0603_1608Metric
- R28: value 10k -> 59; footprint Resistor_SMD:R_0603_1608Metric -> Resistor_SMD:R_1206_3216Metric
- R29: value 100 -> 59; footprint Resistor_SMD:R_0603_1608Metric -> Resistor_SMD:R_1206_3216Metric
- R3, R4: value 5.1k -> 10k
- R41: value 220k -> 100
- R42: value 1k -> 220k
- R43: value 1k -> 68k; footprint Resistor_SMD:R_0603_1608Metric -> Resistor_SMD:R_0805_2012Metric
- R44, R45: value 1k -> 220k; footprint Resistor_SMD:R_0603_1608Metric -> Resistor_SMD:R_0805_2012Metric
- R46: value 100 -> 1k; footprint Resistor_SMD:R_0603_1608Metric -> Resistor_SMD:R_0805_2012Metric
- R47: value 39 -> 1k; footprint Resistor_SMD:R_0603_1608Metric -> Resistor_SMD:R_0805_2012Metric
- R48: footprint Resistor_SMD:R_0603_1608Metric -> Resistor_SMD:R_0805_2012Metric
- R49, R50, R53, R54, R55: value 1k -> 10k
- R52, R60: value 100 -> 10k
- R57: value 22 -> 1k; footprint Resistor_SMD:R_2512_6332Metric -> Resistor_SMD:R_0603_1608Metric
- R58, R59, R66: value 10k -> 1k
- R61, R67, R68: value 100 -> 1k
- R65: value 10k -> 22; footprint Resistor_SMD:R_0603_1608Metric -> Resistor_SMD:R_2512_6332Metric
- U10: value TJA1051T-E -> Si4460; footprint Package_SO:SOIC-8_3.9x4.9mm_P1.27mm -> Package_DFN_QFN:QFN-20-1EP_4x4mm_P0.5mm_EP2.5x2.5mm
- U11: value DRV8870DDA -> TJA1051T-E; footprint Package_SO:Texas_HTSOP-8-1EP_3.9x4.9mm_P1.27mm_EP2.95x4.9mm_Mask2.4x3.1mm_ThermalVias -> Package_SO:SOIC-8_3.9x4.9mm_P1.27mm
- U16: value CR2013-MI2120 -> 74HC138; footprint Display:CR2013-MI2120 -> Package_SO:SOIC-16_3.9x9.9mm_P1.27mm
- U17: value PCF8574 -> CR2013-MI2120; footprint Package_SO:SSOP-20_4.4x6.5mm_P0.65mm -> Display:CR2013-MI2120
- U18: value PCF8574 -> LIS2DH12TR; footprint Package_SO:SSOP-20_4.4x6.5mm_P0.65mm -> Package_LGA:LGA-12_2x2mm_P0.5mm
- U19: value HDC1080 -> PCF8574; footprint Package_SON:Texas_PWSON-N6 -> Package_SO:SSOP-20_4.4x6.5mm_P0.65mm
- U20: value LIS2DH12TR -> HDC1080; footprint Package_LGA:LGA-12_2x2mm_P0.5mm -> Package_SON:Texas_PWSON-N6
- U21: value MCP6021RT-E/OT -> PCF8574; footprint Package_TO_SOT_SMD:SOT-23-5 -> Package_SO:SSOP-20_4.4x6.5mm_P0.65mm
- U22: value SN74LVC1T45DBV -> MCP6021RT-E/OT; footprint Package_TO_SOT_SMD:SOT-23-6 -> Package_TO_SOT_SMD:SOT-23-5
- U23: value TSDP341xx -> SN74LVC1T45DBV; footprint OptoDevice:Vishay_MOLD-3Pin -> Package_TO_SOT_SMD:SOT-23-6
- U24: value CS43L21 -> TSDP341xx; footprint Package_DFN_QFN:QFN-32-1EP_5x5mm_P0.5mm_EP3.45x3.45mm -> OptoDevice:Vishay_MOLD-3Pin
- U5: value TPS22810DRV -> TPS54331DR; footprint Package_SON:WSON-6-1EP_2x2mm_P0.65mm_EP1x1.6mm -> Package_SO:TI_SO-PowerPAD-8_ThermalVias
- U6: value TPS54331DR -> TPS22810DRV; footprint Package_SO:TI_SO-PowerPAD-8_ThermalVias -> Package_SON:WSON-6-1EP_2x2mm_P0.65mm_EP1x1.6mm
- U8: value Si4460 -> LM386; footprint Package_DFN_QFN:QFN-20-1EP_4x4mm_P0.5mm_EP2.5x2.5mm -> Package_SO:SOP-8_3.9x4.9mm_P1.27mm
- U9: value LM386 -> CS43L21; footprint Package_SO:SOP-8_3.9x4.9mm_P1.27mm -> Package_DFN_QFN:QFN-32-1EP_5x5mm_P0.5mm_EP3.45x3.45mm
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Connections:
- net /MOTOR/MOTOR_IN1_2 renamed /MCU/MOTOR_PWM_OUT_1
- net /MOTOR/MOTOR_IN2_2 renamed /MCU/MOTOR_PWM_OUT_2
- net /OUTPUTS/BREAKOUT_MOTOR_C1_1 renamed /MCU/USB_HOST_OUT_P+
- net /OUTPUTS/BREAKOUT_SERVO_2 renamed /MCU/SERIAL_OUT_RX2
- net /SPI/SPI_CS_AUDIO renamed /MCU/SPI_CS_AUDIO
- net /SPI/SPI_CS_BREAKOUT_IN renamed /MCU/SPI_CS_BREAKOUT
- net /SPI/SPI_CS_NFC renamed /MCU/SPI_CS_NFC
- net /SPI/SPI_CS_SEVENSEG renamed /MCU/SPI_CS_SEVENSEG
- net /digital/DIGITAL_DETECT_B renamed /MCU/DIGITAL_RGB_B
- net /digital/DIGITAL_LED_5V renamed Net-(D13-A2)
- C25 pad 1: +5V -> /SPI/micro_SD/SD_VCC
- C26 pad 1: Net-(U6-SS) -> /SPI/micro_SD/SD_VCC
- C27 pad 1: Net-(U7-SS) -> Net-(U5-BOOT)
- C27 pad 2: GND -> Net-(D9-K)
- C28 pad 1: Net-(U6-COMP) -> +12V
- C28 pad 2: Net-(C28-Pad2) -> GND
- C29 pad 1: Net-(U7-COMP) -> +12V
- C29 pad 2: Net-(C29-Pad2) -> GND
- C30 pad 1: Net-(U6-COMP) -> +12V
- C31 pad 1: Net-(U7-COMP) -> +5V
- C32 pad 1: Net-(U6-BOOT) -> +5V
- C32 pad 2: Net-(D5-K) -> GND
- C33 pad 1: Net-(U7-BOOT) -> +12V
- C33 pad 2: Net-(D6-K) -> GND
- C34 pad 1: /POWER/+3V3 -> Net-(U5-SS)
- C35 pad 1: +5V -> Net-(U5-COMP)
- C35 pad 2: GND -> Net-(C35-Pad2)
- C36 pad 1: /POWER/+3V3 -> Net-(U5-COMP)
- C38 pad 1: +3.3V -> Net-(U6-CT)
- C44 pad 1: +12V -> +3V3
- C45 pad 1: +12V -> +3V3
- D10 pad 1: GND -> Net-(D10-K)
- D10 pad 2: /analog/ANALOG_POTENTIOMETER_OUT -> GND
- D11 pad 1: GND -> +5V
- D11 pad 2: +3V3 -> Net-(D11-A)
- D12 pad 1: Net-(D12-K) -> GND
- D12 pad 2: /digital/DIGITAL_LED_12V -> Net-(D12-A2)
- D13 pad 1: Net-(D13-K) -> GND
- D14 pad 1: Net-(D14-K) -> ESP_BUTTON_RESET
- D14 pad 2: /digital/DIGITAL_LED_3V3 -> Net-(D14-A)
- D15 pad 1: +5V -> GND
- D15 pad 2: Net-(D15-DOUT) -> Net-(D14-A)
- D17 pad 1: +5V -> /MCU/DIGITAL_BUTTON_IN_1
- D17 pad 2: Net-(D17-DOUT) -> Net-(D17-A)
- D19 pad 1: +5V -> GND
- D19 pad 2: Net-(D19-DOUT) -> Net-(D16-A)
- D20 pad 1: +5V -> GND
- D20 pad 2: Net-(D20-DOUT) -> Net-(D17-A)
- D21 pad 1: Net-(D21-K) -> +5V
- D21 pad 2: /digital/DIGITAL_LED_0 -> Net-(D21-DOUT)
- D22 pad 1: Net-(D22-K) -> +5V
- D22 pad 2: /digital/DIGITAL_LED_1 -> Net-(D22-DOUT)
- D23 pad 1: Net-(D23-K) -> +5V
- D23 pad 2: /digital/DIGITAL_LED_2 -> Net-(D23-DOUT)
- D24 pad 2: /digital/DIGITAL_NEOPIXEL_OUT -> Net-(D24-DOUT)
- D24 pad 4: Net-(D19-DOUT) -> Net-(D23-DOUT)
- D25 pad 1: +5V -> /MCU/DIGITAL_BUTTON_IN_2
- D25 pad 2: Net-(D25-DOUT) -> Net-(D25-A)
- D26 pad 1: +5V -> /MCU/DIGITAL_BUTTON_IN_3
- D26 pad 2: Net-(D15-DIN) -> Net-(D26-A)
- D28 pad 1: Net-(D28-K) -> +5V
- D28 pad 2: Net-(D28-A) -> Net-(D28-DOUT)
- D30 pad 1: +3V3 -> +5V
- D30 pad 2: Net-(BZ1-+) -> /OUTPUTS/BREAKOUT_NEOPIXEL_IN
- D31 pad 2: /analog/ANALOG_PHOTOTRANSISTOR_OUT -> Net-(D25-A)
- D32 pad 2: /analog/ANALOG_THERMISTOR_OUT -> Net-(D26-A)
- D33 pad 1: GND -> Net-(D33-K)
- D33 pad 2: /analog/ANALOG_JOYSTICK_X_OUT -> /MCU/DIGITAL_LED_OUT_0
- D34 pad 1: GND -> Net-(D34-K)
- D34 pad 2: /analog/ANALOG_JOYSTICK_Y_OUT -> /digital/DIGITAL_LED_12V
- D35 pad 1: GND -> +3V3
- D35 pad 2: Net-(D35-A2) -> Net-(BZ1-+)
- D4 pad 1: +12V -> MCU_BUTTON_RESET
- D5 pad 1: Net-(D5-K) -> GND
- D5 pad 2: GND -> Net-(D4-A)
- D6 pad 1: Net-(D6-K) -> GND
- D6 pad 2: GND -> /50Hz Filter/IN_P1+
- D7 pad 2: /50Hz Filter/IN_P1+ -> /50Hz Filter/IN_P1-
- D8 pad 1: GND -> +12V
- D8 pad 2: /50Hz Filter/IN_P1- -> Net-(D8-A)
- D9 pad 1: +5V -> Net-(D9-K)
- D9 pad 2: Net-(D9-A) -> GND
- F1 pad 2: Net-(D4-A) -> Net-(D8-A)
- J10 pad 1: /OUTPUTS/BREAKOUT_D_GPIO_3 -> /I2C/I2C_SDA_BREAKOUT
- J10 pad 2: /OUTPUTS/BREAKOUT_VCC -> /I2C/I2C_SCL_BREAKOUT
- J10 pad 3: GND -> /OUTPUTS/BREAKOUT_VCC
- J12 pad 1: /I2C/I2C_SDA_BREAKOUT -> /OUTPUTS/BREAKOUT_NEOPIXEL_IN
- J12 pad 2: /I2C/I2C_SCL_BREAKOUT -> /OUTPUTS/BREAKOUT_VCC
- J12 pad 3: /OUTPUTS/BREAKOUT_VCC -> GND
- J13 pad 1: /CAN/CAN_H -> /OUTPUTS/BREAKOUT_D_GPIO_2
- J13 pad 2: /CAN/CAN_L -> /OUTPUTS/BREAKOUT_VCC
- J13 pad 3: /OUTPUTS/BREAKOUT_VCC -> GND
- J14 pad 1: /OUTPUTS/BREAKOUT_SERIAL_TX -> /CAN/CAN_H
- J14 pad 2: /OUTPUTS/BREAKOUT_SERIAL_RX -> /CAN/CAN_L
- J15 pad 1: +12V -> /MOTOR/MOTOR_OUT1_BREAKOUT_1
- J15 pad 2: GND -> /MOTOR/MOTOR_OUT2_BREAKOUT_1
- J17 pad 1: /OUTPUTS/BREAKOUT_SERVO_1 -> /OUTPUTS/BREAKOUT_D_GPIO_3
- J18 pad 2: /OUTPUTS/BREAKOUT_VCC -> /MCU/SERIAL_OUT_TX2
- J18 pad 3: GND -> /OUTPUTS/BREAKOUT_VCC
- J19 pad 1: /OUTPUTS/BREAKOUT_ULTRASONIC_TRIG -> +12V
- J19 pad 2: /OUTPUTS/BREAKOUT_ULTRASONIC_ECHO -> GND
- J20 pad 1: /MOTOR/MOTOR_OUT1_BREAKOUT_1 -> /OUTPUTS/BREAKOUT_USB_VBUS
- J20 pad 2: /MOTOR/MOTOR_OUT1_BREAKOUT_2 -> /MCU/USB_HOST_OUT_P-
- J20 pad 4: /OUTPUTS/BREAKOUT_MOTOR_C2_1 -> GND
- J20 pad 5: +12V -> unconnected-(J20-Shield-Pad5)
- J21 pad 1: /MOTOR/MOTOR_OUT2_BREAKOUT_1 -> unconnected-(J21-DAT2-Pad1)
- J21 pad 2: /MOTOR/MOTOR_OUT2_BREAKOUT_2 -> /SPI/micro_SD/SD_CS-CS
- J21 pad 3: /OUTPUTS/BREAKOUT_MOTOR_C1_2 -> /SPI/micro_SD/SD_DI-MOSI
- J21 pad 4: /OUTPUTS/BREAKOUT_MOTOR_C2_2 -> /SPI/micro_SD/SD_VCC
- J21 pad 5: +12V -> /SPI/micro_SD/SD_CLK-SCK
- J22 pad 1: unconnected-(J22-DAT2-Pad1) -> GND
- J22 pad 2: /SPI/micro_SD/SD_CS-CS -> Net-(F1-Pad1)
- J6 pad 1: /OUTPUTS/BREAKOUT_NEOPIXEL_IN -> /SPI/CS_BREAKOUT
- J6 pad 2: /OUTPUTS/BREAKOUT_VCC -> /SPI/CLK
- J6 pad 3: GND -> /SPI/MISO
- J9 pad 1: /OUTPUTS/BREAKOUT_D_GPIO_2 -> /OUTPUTS/BREAKOUT_D_GPIO_1
- L3 pad 1: /CAN/CAN_H -> Net-(D9-K)
- L3 pad 2: /CAN/CAN_L -> +5V
- MK1 pad 2: Net-(D35-A2) -> Net-(D49-A2)
- Q3 pad 3: Net-(D16-K) -> Net-(BZ1-+)
- Q4 pad 3: Net-(D28-K) -> Net-(D39-K)
- Q5 pad 3: Net-(BZ1-+) -> Net-(D42-K)
- Q6 pad 2: /analog/ANALOG_PHOTOTRANSISTOR_OUT -> /MCU/ANALOG_PHOTOTRANSISTOR
- Q6 pad 4: /analog/ANALOG_PHOTOTRANSISTOR_OUT -> /MCU/ANALOG_PHOTOTRANSISTOR
- R1 pad 1: Net-(SW1A-D) -> GND
- R1 pad 2: +3V3 -> Net-(J1-CC2)
- R11 pad 1: +5V -> Net-(Q1-G)
- R11 pad 2: Net-(U6-EN) -> +3.3V
- R12 pad 1: Net-(U6-EN) -> Net-(Q1-G)
- R12 pad 2: GND -> /SPI/SPI_ENABLE_SD
- R13 pad 1: +12V -> /SPI/SPI_DETECT_SD
- R13 pad 2: Net-(U7-EN) -> +3.3V
- R14 pad 1: Net-(U7-EN) -> +12V
- R14 pad 2: GND -> Net-(U5-EN)
- R15 pad 1: Net-(C28-Pad2) -> +5V
- R15 pad 2: GND -> Net-(U5-VSENSE)
- R16 pad 1: Net-(C29-Pad2) -> Net-(U5-EN)
- R17 pad 1: /POWER/+3V3 -> Net-(U5-VSENSE)
- R17 pad 2: Net-(U6-VSENSE) -> Net-(R17-Pad2)
- R18 pad 1: Net-(U6-VSENSE) -> Net-(R17-Pad2)
- R19 pad 1: Net-(R18-Pad2) -> Net-(C35-Pad2)
- R2 pad 1: Net-(SW1A-D) -> GND
- R2 pad 2: MCU_BUTTON_RESET -> Net-(J1-CC1)
- R20 pad 1: +5V -> Net-(R18-Pad2)
- R20 pad 2: Net-(U7-VSENSE) -> GND
- R21 pad 1: Net-(U7-VSENSE) -> Net-(U6-QOD)
- R21 pad 2: Net-(R21-Pad2) -> /OUTPUTS/BREAKOUT_USB_VBUS
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
Commit message: Esp32 motherboard schematic done.
Parts:
- added J28: Conn_02x20_Odd_Even, Connector_PinHeader_2.54mm:PinHeader_2x20_P2.54mm_Horizontal, F.Cu at (257.5, 92.7)
Connections:
- net ESP_BUTTON_RESET renamed /esp32/ESP_BUTTON_RESET

Commit message: Finished v0.1 schematic.
Parts:
- removed AE2: Antenna, Connector_PinSocket_2.54mm:PinSocket_1x01_P2.54mm_Vertical
- removed C26: 100nF, Capacitor_SMD:C_0805_2012Metric
- removed C28, C29, C37, C41: 4.7uF, Capacitor_SMD:C_1206_3216Metric
- removed C30, C40, C49, C57: 100nF, Capacitor_SMD:C_0603_1608Metric
- removed C31, C32, C39, C44, C45, C59, C67: 47uF, Capacitor_SMD:C_1210_3225Metric
- removed C34, C46: 10nF, Capacitor_SMD:C_0603_1608Metric
- removed C35: 4.7nF, Capacitor_SMD:C_0603_1608Metric
- removed C36: 39pF, Capacitor_SMD:C_0603_1608Metric
- removed C38: 22nF, Capacitor_SMD:C_0603_1608Metric
- removed C47: 1nF, Capacitor_SMD:C_0603_1608Metric
- removed C48: 47pF, Capacitor_SMD:C_0603_1608Metric
- removed C55: 47uF, Capacitor_SMD:CP_Elec_6.3x5.8
- removed C56: 1uF, Capacitor_SMD:C_0603_1608Metric
- removed C58, C68: 100nF C0G, Capacitor_SMD:C_1206_3216Metric
- removed C60, C69: 10uF, Capacitor_SMD:C_1206_3216Metric
- removed C80, C81: 4.7uF, Capacitor_SMD:C_0603_1608Metric
- removed the H5 at (134.2, 126.4)
- removed J20: USB_A, Connector_USB:USB_A_TE_292303-7_Horizontal
- removed J22: Barrel_Jack_MountingPin, Connector_BarrelJack:BarrelJack_CUI_PJ-063AH_Horizontal
- removed J23: AudioJack4, Connector_Audio:Jack_3.5mm_KoreanHropartsElec_PJ-320D-4A_Horizontal
- removed J26, J27: KEYPAD_MATRIX, Connector_PinHeader_2.54mm:PinHeader_1x08_P2.54mm_Vertical_SMD_Pin1Left
- removed J28: Conn_02x20_Odd_Even, Connector_PinHeader_2.54mm:PinHeader_2x20_P2.54mm_Horizontal
- removed J7: GPIO, Connector_JST:JST_XH_S3B-XH-A_1x03_P2.50mm_Horizontal
- removed L1: 6.8, Inductor_SMD:L_Chilisin_BMRB00060624
- removed L5: L_Iron_Coupled_1324, Inductor_SMD:L_CommonModeChoke_TDK_ACM7060
- removed R26: 29.4k, Resistor_SMD:R_0603_1608Metric
- removed R27: 1k 1%, Resistor_SMD:R_0603_1608Metric
- removed R28, R29: 59, Resistor_SMD:R_1206_3216Metric
- removed R30: 2, Resistor_SMD:R_2512_6332Metric
- removed R31: 5.1k, Resistor_SMD:R_0603_1608Metric
- removed R33, R34, R70: 10k, Resistor_SMD:R_0603_1608Metric
- removed R35, R36: 1k, Resistor_SMD:R_0805_2012Metric
- removed R37: 68k, Resistor_SMD:R_0805_2012Metric
- removed R65: 22, Resistor_SMD:R_2512_6332Metric
- removed R66, R67, R68: 1k, Resistor_SMD:R_0603_1608Metric
- removed R69: 100, Resistor_SMD:R_0603_1608Metric
- removed R71: 39, Resistor_SMD:R_0603_1608Metric
- removed the SW2 at (265.9, 77.2)
- removed SW7: SW_Push, Button_Switch_SMD:SW_Push_1P1T_NO_6x6mm_H9.5mm
- removed U14: SN74LVC1T45DBV, Package_TO_SOT_SMD:SOT-23-6
- removed U21: PCF8574, Package_SO:SSOP-20_4.4x6.5mm_P0.65mm
- added C10: 100nF, Capacitor_SMD:C_0603_1608Metric, B.Cu at (147.2, 55.0)
- added C11: 100nF, Capacitor_SMD:C_0603_1608Metric, B.Cu at (147.2, 57.5)
- added C12: 10nF, Capacitor_SMD:C_0603_1608Metric, B.Cu at (130.2, 70.0)
- added C13: 10nF, Capacitor_SMD:C_0603_1608Metric, B.Cu at (130.2, 72.5)
- added C4: 100uF, Capacitor_SMD:CP_Elec_6.3x7.7, B.Cu at (126.3, 51.0)
- added C5: 47uF, Capacitor_SMD:C_1210_3225Metric, B.Cu at (108.0, 49.0)
- added C6: 4.7uF, Capacitor_SMD:C_1206_3216Metric, B.Cu at (82.4, 49.1)
- added C7: 4.7uF, Capacitor_SMD:C_1206_3216Metric, B.Cu at (82.4, 52.4)
- added C76: 4.7uF, Capacitor_SMD:C_0603_1608Metric, B.Cu at (142.2, 102.2)
- added C78: 4.7uF, Capacitor_SMD:C_0603_1608Metric, B.Cu at (142.2, 104.7)
- added C8: 4.7uF, Capacitor_SMD:C_1206_3216Metric, B.Cu at (82.4, 55.8)
- added C85: 1uF, Capacitor_SMD:C_0603_1608Metric, B.Cu at (196.1, 108.0)
- added C86: 100nF, Capacitor_SMD:C_0603_1608Metric, B.Cu at (193.5, 108.0)
- added C87: 100nF C0G, Capacitor_SMD:C_1206_3216Metric, B.Cu at (195.6, 112.8)
- added C88: 47uF, Capacitor_SMD:C_1210_3225Metric, B.Cu at (188.5, 112.8)
- added C89: 10uF, Capacitor_SMD:C_1206_3216Metric, B.Cu at (192.3, 112.8)
- added C9: 4.7uF, Capacitor_SMD:C_1206_3216Metric, B.Cu at (82.4, 59.1)
- added D18: SD05_SOD323, Diode_SMD:D_SOD-323, B.Cu at (162.0, 130.1)
- added D36: SD05_SOD323, Diode_SMD:D_SOD-323, B.Cu at (103.7, 130.1)
- added D50: LED, LED_THT:LED_D5.0mm, F.Cu at (202.0, 96.6)
- added D51: WS2812B, LED_SMD:LED_WS2812B_PLCC4_5.0x5.0mm_P3.2mm, F.Cu at (151.0, 85.0)
- added D52: WS2812B, LED_SMD:LED_WS2812B_PLCC4_5.0x5.0mm_P3.2mm, F.Cu at (151.0, 91.6)
- added D53: WS2812B, LED_SMD:LED_WS2812B_PLCC4_5.0x5.0mm_P3.2mm, F.Cu at (151.0, 98.2)
- added D54: LED, LED_THT:LED_D5.0mm, F.Cu at (209.7, 96.6)
- added D55: SD05_SOD323, Diode_SMD:D_SOD-323, B.Cu at (156.1, 113.0)
- added D56: 1N4148W, Diode_SMD:D_SOD-123, B.Cu at (95.0, 72.7)
- added D57: SD05_SOD323, Diode_SMD:D_SOD-323, B.Cu at (156.1, 116.0)
- added D58: 1N4148W, Diode_SMD:D_SOD-123, B.Cu at (95.0, 76.0)
- added D59: 1N4148W, Diode_SMD:D_SOD-123, B.Cu at (95.0, 79.3)
- added D61: SD05_SOD323, Diode_SMD:D_SOD-323, B.Cu at (156.1, 119.0)
- added D62: SD05_SOD323, Diode_SMD:D_SOD-323, B.Cu at (156.1, 121.9)
- added D63: 1N4148W, Diode_SMD:D_SOD-123, B.Cu at (95.0, 82.7)
- added D64: 1N4148W, Diode_SMD:D_SOD-123, B.Cu at (95.0, 86.0)
- added D65: SD05_SOD323, Diode_SMD:D_SOD-323, B.Cu at (161.0, 50.7)
- added D66: SD05_SOD323, Diode_SMD:D_SOD-323, B.Cu at (152.0, 50.9)
- added D67: SD05_SOD323, Diode_SMD:D_SOD-323, B.Cu at (152.0, 53.9)
- added D68: SD05_SOD323, Diode_SMD:D_SOD-323, B.Cu at (152.0, 56.8)
- added D69: SD05_SOD323, Diode_SMD:D_SOD-323, B.Cu at (152.0, 59.8)
- added D70: SD05_SOD323, Diode_SMD:D_SOD-323, B.Cu at (152.0, 62.7)
- added D71: SD05_SOD323, Diode_SMD:D_SOD-323, B.Cu at (152.0, 65.7)
- added H5: MountingHole, MountingHole:MountingHole_3.2mm_M3_ISO7380_Pad_TopBottom, F.Cu at (87.0, 86.0)
- added H5: MountingHole, MountingHole:MountingHole_3.2mm_M3_ISO7380_Pad_TopBottom, F.Cu at (71.1, 132.0)
- added H5: MountingHole, MountingHole:MountingHole_3.2mm_M3_ISO7380_Pad_TopBottom, F.Cu at (158.0, 92.0)
- added J11: Can, Connector_Phoenix_MSTB:PhoenixContact_MSTBA_2,5_3-G-5,08_1x03_P5.08mm_Horizontal, B.Cu at (100.0, 138.2)
- added J2: USB_C_Receptacle, Connector_USB:USB_C_Receptacle_G-Switch_GT-USB-7025, B.Cu at (70.6, 121.6)
- added J3: Conn_02x20_Odd_Even, Connector_PinHeader_2.54mm:PinHeader_2x20_P2.54mm_Horizontal, B.Cu at (117.4, 43.5)
- added J8: Conn_02x20_Odd_Even, Connector_PinHeader_2.54mm:PinHeader_2x20_P2.54mm_Horizontal, B.Cu at (169.5, 43.5)
- added R6: 330k, Resistor_SMD:R_0603_1608Metric, B.Cu at (133.0, 61.0)
- added R73: 1k, Resistor_SMD:R_0805_2012Metric, B.Cu at (200.4, 117.8)
- added R74: 68k, Resistor_SMD:R_0805_2012Metric, B.Cu at (197.5, 117.8)
- added R75: 100, Resistor_SMD:R_0805_2012Metric, B.Cu at (194.5, 117.8)
- added R76: 220k, Resistor_SMD:R_0805_2012Metric, B.Cu at (191.6, 117.8)
- added R77: 220k, Resistor_SMD:R_0805_2012Metric, B.Cu at (188.6, 117.8)
- added R78: 220k, Resistor_SMD:R_0805_2012Metric, B.Cu at (185.7, 117.8)
- added R79: 1k, Resistor_SMD:R_0805_2012Metric, B.Cu at (182.7, 117.8)
- added SW2: SW_Push, Button_Switch_SMD:SW_Push_1P1T_NO_CK_KMR2, F.Cu at (151.1, 72.8)
- added SW2: SW_Push, Button_Switch_SMD:SW_Push_1P1T_NO_CK_KMR2, F.Cu at (151.1, 78.8)
- added SW6: SW_Push, Button_Switch_SMD:SW_Push_1P1T_NO_6x6mm_H9.5mm, F.Cu at (209.2, 116.8)
- added U25: LMP2011, Package_TO_SOT_SMD:TSOT-23-5, B.Cu at (107.9, 112.7)
- added U26: LMP2011, Package_TO_SOT_SMD:TSOT-23-5, B.Cu at (101.0, 104.0)
- added U27: LMP2011, Package_TO_SOT_SMD:TSOT-23-5, B.Cu at (101.0, 108.6)
- BZ1, C27, C43, C79, D11, D12, D13, D15, D19, D20, D31, D32, D5, D8, F1, F2, J21, L2, L3, Q3, Q4, Q5, Q6, R15, R49, R51, R53, R54, R55, R61, R62, RV1, SW1, TH1, TP1, U22: moved to B.Cu
- C14: value 10uF -> 1nF; footprint Capacitor_SMD:C_1206_3216Metric -> Capacitor_SMD:C_0603_1608Metric; moved to B.Cu
- C15: value 100nF -> 4.7nF; footprint Capacitor_SMD:C_0805_2012Metric -> Capacitor_SMD:C_0603_1608Metric; moved to B.Cu
- C16: value 4.7uF -> 47pF; footprint Capacitor_SMD:C_1206_3216Metric -> Capacitor_SMD:C_0603_1608Metric; moved to B.Cu
- C17: value 22nF -> 39pF; moved to B.Cu
- C18: value 100uF -> 100nF; footprint Capacitor_SMD:CP_Elec_6.3x7.7 -> Capacitor_SMD:C_0603_1608Metric; moved to B.Cu
- C19: value 47uF -> 100nF; footprint Capacitor_SMD:C_1210_3225Metric -> Capacitor_SMD:C_0603_1608Metric; moved to B.Cu
- C2: value 10uF -> 4.7uF; footprint Capacitor_SMD:C_0805_2012Metric -> Capacitor_SMD:C_1206_3216Metric; moved to B.Cu
- C20, C21: value 4.7uF -> 47uF; footprint Capacitor_SMD:C_1206_3216Metric -> Capacitor_SMD:C_1210_3225Metric; moved to B.Cu
- C22, C23: value 4.7uF -> 47uF; footprint Capacitor_SMD:C_1206_3216Metric -> Capacitor_SMD:CP_Elec_6.3x5.8; moved to B.Cu
- C24: value 100nF -> 47uF; footprint Capacitor_SMD:C_0603_1608Metric -> Capacitor_SMD:C_1210_3225Metric; moved to B.Cu
- C25: value 10uF -> 47uF; footprint Capacitor_SMD:C_1206_3216Metric -> Capacitor_SMD:C_1210_3225Metric; moved to B.Cu
- C3: value 100nF -> 22nF; moved to B.Cu
- C33: value 100uF -> 47uF; footprint Capacitor_SMD:CP_Elec_6.3x7.7 -> Capacitor_SMD:CP_Elec_6.3x5.8; moved to B.Cu
- C42: value 4.7uF -> 10uF; footprint Capacitor_SMD:C_1206_3216Metric -> Capacitor_SMD:C_0805_2012Metric; moved to B.Cu
- C65: value 1uF -> 10uF; footprint Capacitor_SMD:C_0603_1608Metric -> Capacitor_SMD:C_1206_3216Metric; moved to B.Cu
- C66: footprint Capacitor_SMD:C_0603_1608Metric -> Capacitor_SMD:C_0805_2012Metric; moved to B.Cu
- D1, D9: value D_Schottky -> SD05_SOD323; footprint Diode_SMD:D_SMB -> Diode_SMD:D_SOD-323; moved to B.Cu
- D10: value D_Schottky -> 1N4148W; footprint Diode_SMD:D_SMB -> Diode_SMD:D_SOD-123; moved to B.Cu
- D14, D16, D17, D25, D26, D35, D4: value 1N4148W -> SD05_SOD323; footprint Diode_SMD:D_SOD-123 -> Diode_SMD:D_SOD-323; moved to B.Cu
- D2: value SD05_SOD323 -> 1N4148W; footprint Diode_SMD:D_SOD-323 -> Diode_SMD:D_SOD-123; moved to B.Cu
- D21, D22, D23, D24, D27, D28, D29, D30: value WS2812B -> SD05_SOD323; footprint LED_SMD:LED_WS2812B_PLCC4_5.0x5.0mm_P3.2mm -> Diode_SMD:D_SOD-323; moved to B.Cu
- D3, D6, D7: value SD05_SOD323 -> D_Schottky; footprint Diode_SMD:D_SOD-323 -> Diode_SMD:D_SMB; moved to B.Cu
- D33, D34, D37, D38: value LED -> SD05_SOD323; footprint LED_THT:LED_D5.0mm -> Diode_SMD:D_SOD-323; moved to B.Cu
- D42: value D_IR_EMITTER -> WS2812B; footprint LED_THT:LED_D5.0mm_Horizontal_O1.27mm_Z3.0mm_Clear -> LED_SMD:LED_WS2812B_PLCC4_5.0x5.0mm_P3.2mm
- D43: value SD05_SOD323 -> D_IR_EMITTER; footprint Diode_SMD:D_SOD-323 -> LED_THT:LED_D5.0mm_Horizontal_O1.27mm_Z3.0mm_Clear; moved to B.Cu
- D44, D45, D46, D47: value SD05_SOD323 -> WS2812B; footprint Diode_SMD:D_SOD-323 -> LED_SMD:LED_WS2812B_PLCC4_5.0x5.0mm_P3.2mm
- D48, D49: value SD05_SOD323 -> LED; footprint Diode_SMD:D_SOD-323 -> LED_THT:LED_D5.0mm
- J10: value I2C -> Neopixel; footprint Connector_JST:JST_XH_S4B-XH-A_1x04_P2.50mm_Horizontal -> Connector_Phoenix_MSTB:PhoenixContact_MSTBA_2,5_3-G-5,08_1x03_P5.08mm_Horizontal; moved to B.Cu
- J12: value Neopixel -> USB_A; footprint Connector_JST:JST_XH_S3B-XH-A_1x03_P2.50mm_Horizontal -> Connector_USB:USB_A_TE_292303-7_Horizontal; moved to B.Cu
- J13: value GPIO -> SPI_OUT; footprint Connector_JST:JST_XH_S3B-XH-A_1x03_P2.50mm_Horizontal -> Connector_Phoenix_MSTB:PhoenixContact_MSTBA_2,5_6-G-5,08_1x06_P5.08mm_Horizontal; moved to B.Cu
- J14: value CAN -> MOTOR; footprint Connector_JST:JST_XH_S4B-XH-A_1x04_P2.50mm_Horizontal -> Connector_Phoenix_MSTB:PhoenixContact_MSTBA_2,5_6-G-5,08_1x06_P5.08mm_Horizontal; moved to B.Cu
- J15: value MOTOR -> 12V OUT; footprint Connector_JST:JST_XH_S6B-XH-A_1x06_P2.50mm_Horizontal -> Connector_Phoenix_MSTB:PhoenixContact_MSTBA_2,5_2-G-5,08_1x02_P5.08mm_Horizontal; moved to B.Cu
- J16: value SERVO -> RTD_PT100; footprint Connector_JST:JST_XH_S3B-XH-A_1x03_P2.50mm_Horizontal -> Connector_Phoenix_MSTB:PhoenixContact_MSTBA_2,5_4-G-5,08_1x04_P5.08mm_Horizontal; moved to B.Cu
- J17: value GPIO -> SERIAL; footprint Connector_JST:JST_XH_S3B-XH-A_1x03_P2.50mm_Horizontal -> Connector_Phoenix_MSTB:PhoenixContact_MSTBA_2,5_4-G-5,08_1x04_P5.08mm_Horizontal; moved to B.Cu
- J18: value SERIAL -> I2C; footprint Connector_JST:JST_XH_S4B-XH-A_1x04_P2.50mm_Horizontal -> Connector_Phoenix_MSTB:PhoenixContact_MSTBA_2,5_4-G-5,08_1x04_P5.08mm_Horizontal; moved to B.Cu
- J19: value 12V OUT -> KEYPAD_MATRIX; footprint TerminalBlock_Phoenix:TerminalBlock_Phoenix_MKDS-1,5-2-5.08_1x02_P5.08mm_Horizontal -> Connector_PinHeader_2.54mm:PinHeader_1x08_P2.54mm_Vertical_SMD_Pin1Left
- J5: value A_OUT -> Barrel_Jack_MountingPin; footprint Connector_JST:JST_XH_S3B-XH-A_1x03_P2.50mm_Horizontal -> Connector_BarrelJack:BarrelJack_CUI_PJ-063AH_Horizontal; moved to B.Cu
- J6: value SPI_OUT -> USB_C_Receptacle; footprint Connector_JST:JST_XH_S6B-XH-A_1x06_P2.50mm_Horizontal -> Connector_USB:USB_C_Receptacle_G-Switch_GT-USB-7025; moved to B.Cu
- J9: value GPIO -> A_IN; footprint Connector_JST:JST_XH_S3B-XH-A_1x03_P2.50mm_Horizontal -> Connector_Phoenix_MSTB:PhoenixContact_MSTBA_2,5_2-G-5,08_1x02_P5.08mm_Horizontal; moved to B.Cu
- L4: value 6.8 -> L_Iron_Coupled_1324; footprint Inductor_SMD:L_Chilisin_BMRB00060624 -> Inductor_SMD:L_CommonModeChoke_TDK_ACM7060; moved to B.Cu
- Q1: value DMP2045U-7 -> BC850; moved to B.Cu
- Q2: value BC850 -> DMP2045U-7; moved to B.Cu
- R1, R2: value 5.1k -> 10k; moved to B.Cu
- R10: value DNP -> 29.4k; moved to B.Cu
- R11: value 10k -> 50k; moved to B.Cu
- R12: value 100 -> 10k 1%; moved to B.Cu
- R13: value 10k -> 2.2k 1%; moved to B.Cu
- R14: value 330k -> 1k 1%; moved to B.Cu
- R16: value 68k -> 1k 1%; moved to B.Cu
- R17: value 1k 1% -> 680 1%; moved to B.Cu
- R18: value 680 1% -> 220 1%; moved to B.Cu
- R19: value 50k -> 10k; moved to B.Cu
- R20: value 220 1% -> 10k; moved to B.Cu
- R21: value DNP -> 5.1k; moved to B.Cu
- R22: value 330k -> 5.1k; moved to B.Cu
- R23: value 68k -> 59; footprint Resistor_SMD:R_0603_1608Metric -> Resistor_SMD:R_1206_3216Metric; moved to B.Cu
- R24: value 10k 1% -> 59; footprint Resistor_SMD:R_0603_1608Metric -> Resistor_SMD:R_1206_3216Metric; moved to B.Cu
- R25: value 2.2k 1% -> 2; footprint Resistor_SMD:R_0603_1608Metric -> Resistor_SMD:R_2512_6332Metric; moved to B.Cu
- R3, R4: value 10k -> 5.1k; moved to B.Cu
- R32: value 5.1k -> 33k; moved to B.Cu
- R38, R41: value 100 -> 10k; footprint Resistor_SMD:R_0805_2012Metric -> Resistor_SMD:R_0603_1608Metric; moved to B.Cu
- R39: value 220k -> 10k; footprint Resistor_SMD:R_0805_2012Metric -> Resistor_SMD:R_0603_1608Metric; moved to B.Cu
- R40, R44: value 220k -> 100; footprint Resistor_SMD:R_0805_2012Metric -> Resistor_SMD:R_0603_1608Metric; moved to B.Cu
- R42: value 220k -> 4.7k; footprint Resistor_SMD:R_0805_2012Metric -> Resistor_SMD:R_0603_1608Metric; moved to B.Cu
- R43: value 68k -> 1k; footprint Resistor_SMD:R_0805_2012Metric -> Resistor_SMD:R_0603_1608Metric; moved to B.Cu
- R45: value 220k -> 39; footprint Resistor_SMD:R_0805_2012Metric -> Resistor_SMD:R_0603_1608Metric; moved to B.Cu
- R46, R47, R48: footprint Resistor_SMD:R_0805_2012Metric -> Resistor_SMD:R_0603_1608Metric; moved to B.Cu
- R5: value 33k -> DNP; moved to B.Cu
- R50: value 10k -> 100; moved to B.Cu
- R52: value 10k -> 22; footprint Resistor_SMD:R_0603_1608Metric -> Resistor_SMD:R_2512_6332Metric; moved to B.Cu
- R56, R60: value 10k -> 1k; moved to B.Cu
- R57, R58, R59, R63, R64: value 1k -> 10k; moved to B.Cu
- R7: value 10k -> 68k; moved to B.Cu
- R72: value 100 -> 1k; footprint Resistor_SMD:R_0603_1608Metric -> Resistor_SMD:R_0805_2012Metric; moved to B.Cu
- R8: value 10k -> 330k; moved to B.Cu
- R9: value 100 -> 68k; moved to B.Cu
- RN1, RN2: value 10k -> 4.7k; footprint Resistor_SMD:R_Array_Convex_5x0603 -> Resistor_SMD:R_Array_Convex_4x0603; moved to B.Cu
- RN3, RN4: value 4.7k -> 10k; footprint Resistor_SMD:R_Array_Convex_4x0603 -> Resistor_SMD:R_Array_Convex_5x0603; moved to B.Cu
- RV2: value 2k -> 100k; footprint Potentiometer_SMD:Potentiometer_Bourns_3314J_Vertical -> Potentiometer_THT:Potentiometer_Piher_PT-6-V_Vertical
- RV3: value 100k -> 10k; footprint Potentiometer_THT:Potentiometer_Piher_PT-6-V_Vertical -> potentiometer_2_axis_joystick:2-Axis-Joystick
- RV4: value 10k -> 2k; footprint potentiometer_2_axis_joystick:2-Axis-Joystick -> Potentiometer_SMD:Potentiometer_Bourns_3314J_Vertical; moved to B.Cu
- U1: value CC56-12YWA -> TPS22810DRV; footprint Display_7Segment:CC56-12YWA -> Package_SON:WSON-6-1EP_2x2mm_P0.65mm_EP1x1.6mm; moved to B.Cu
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Connections:
- C14 pad 1: /SPI/micro_SD/SD_VCC -> Net-(U2-COMP)
- C14 pad 2: GND -> Net-(C14-Pad2)
- C15 pad 1: /SPI/micro_SD/SD_VCC -> Net-(U3-COMP)
- C15 pad 2: GND -> Net-(C15-Pad2)
- C16 pad 1: +5V -> Net-(U2-COMP)
- C17 pad 1: Net-(U5-CT) -> Net-(U3-COMP)
- C18 pad 1: +12V -> Net-(U2-BOOT)
- C18 pad 2: GND -> Net-(D7-K)
- C19 pad 1: /OUTPUTS/BREAKOUT_USB_VBUS -> Net-(U3-BOOT)
- C19 pad 2: GND -> Net-(D8-K)
- C20 pad 1: +12V -> +3V3
- C22 pad 1: +12V -> +3V3
- C24 pad 1: +12V -> +3V3
- C25 pad 1: /SPI/micro_SD/SD_VCC -> +5V
- C27 pad 1: Net-(U5-BOOT) -> +3.3V
- C27 pad 2: Net-(D9-K) -> GND
- C3 pad 1: +5V -> Net-(U1-CT)
- C65 pad 1: /50Hz Filter/3.3VA_1 -> /SPI/micro_SD/SD_VCC
- C66 pad 1: /50Hz Filter/3.3VA_1 -> /SPI/micro_SD/SD_VCC
- D1 pad 1: +5V -> GND
- D1 pad 2: Net-(D1-A) -> Net-(D1-A2)
- D10 pad 1: Net-(D10-K) -> /esp32/ESP_BUTTON_RESET
- D10 pad 2: GND -> Net-(D10-A)
- D14 pad 1: /esp32/ESP_BUTTON_RESET -> GND
- D14 pad 2: Net-(D14-A) -> /CAN/CAN_H
- D15 pad 2: Net-(D14-A) -> /OUTPUTS/BREAKOUT_NEOPIXEL_IN
- D16 pad 1: Net-(D16-K) -> GND
- D16 pad 2: Net-(D16-A) -> /50Hz Filter/IN_P1+
- D17 pad 1: /MCU/DIGITAL_BUTTON_IN_1 -> GND
- D17 pad 2: Net-(D17-A) -> /CAN/CAN_L
- D19 pad 2: Net-(D16-A) -> /SPI/CS_BREAKOUT
- D2 pad 1: GND -> /MCU/MCU_RESET
- D2 pad 2: Net-(D2-A2) -> Net-(D1-A2)
- D20 pad 2: Net-(D17-A) -> /OUTPUTS/BREAKOUT_USB_VBUS
- D21 pad 1: +5V -> GND
- D21 pad 2: Net-(D21-DOUT) -> /MOTOR/MOTOR_OUT1_BREAKOUT_1
- D22 pad 1: +5V -> GND
- D22 pad 2: Net-(D22-DOUT) -> /SPI/CLK
- D23 pad 1: +5V -> GND
- D23 pad 2: Net-(D23-DOUT) -> /MCU/USB_HOST_OUT_P+
- D24 pad 1: +5V -> GND
- D24 pad 2: Net-(D24-DOUT) -> /MCU/MOTOR_CC_IN_1
- D25 pad 1: /MCU/DIGITAL_BUTTON_IN_2 -> GND
- D25 pad 2: Net-(D25-A) -> /SPI/MISO
- D26 pad 1: /MCU/DIGITAL_BUTTON_IN_3 -> GND
- D26 pad 2: Net-(D26-A) -> /MCU/USB_HOST_OUT_P-
- D27 pad 1: +5V -> GND
- D27 pad 2: Net-(D27-DOUT) -> /MCU/MOTOR_CC_IN_2
- D28 pad 1: +5V -> GND
- D28 pad 2: Net-(D28-DOUT) -> /SPI/MOSI
- D29 pad 1: +5V -> GND
- D29 pad 2: Net-(D29-DOUT) -> /MOTOR/MOTOR_OUT2_BREAKOUT_1
- D3 pad 1: GND -> +5V
- D30 pad 1: +5V -> GND
- D30 pad 2: /OUTPUTS/BREAKOUT_NEOPIXEL_IN -> /OUTPUTS/RTD_W1
- D31 pad 2: Net-(D25-A) -> +12V
- D32 pad 2: Net-(D26-A) -> /OUTPUTS/RTD_W2
- D33 pad 1: Net-(D33-K) -> GND
- D33 pad 2: /MCU/DIGITAL_LED_OUT_0 -> /OUTPUTS/RTD_W3
- D34 pad 1: Net-(D34-K) -> GND
- D34 pad 2: /digital/DIGITAL_LED_12V -> /OUTPUTS/RTD_W4
- D35 pad 1: +3V3 -> GND
- D35 pad 2: Net-(BZ1-+) -> Net-(D35-A2)
- D37 pad 1: Net-(D37-K) -> GND
- D37 pad 2: /MCU/DIGITAL_LED_OUT_1 -> /I2C/I2C_SDA_BREAKOUT
- D38 pad 1: Net-(D38-K) -> GND
- D38 pad 2: /digital/DIGITAL_LED_5V -> /I2C/I2C_SCL_BREAKOUT
- D39 pad 2: Net-(D39-A) -> +12V
- D4 pad 1: MCU_BUTTON_RESET -> GND
- D4 pad 2: Net-(D4-A) -> /MCU/USB_DP+
- D40 pad 2: /MCU/DIGITAL_LED_OUT_2 -> +5V
- D41 pad 2: /digital/DIGITAL_LED_3V3 -> +3V3
- D42 pad 1: Net-(D42-K) -> +5V
- D42 pad 2: Net-(D42-A) -> Net-(D42-DOUT)
- D43 pad 1: GND -> Net-(D43-K)
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Other:
- board outline added: 160 x 115 mm
