File: PRODIGY-MOTHERBOARD/filter.kicad_sch (KiCad schematic)
At the start: 0 parts

Commit message: SPI SD CARD circuit added.
Parts:
- added C32: 1uF, Capacitor_SMD:C_0603_1608Metric, symbol Device:C
- added C33: 100nF, Capacitor_SMD:C_0603_1608Metric, symbol Device:C
- added C34: 100nF C0G, Capacitor_SMD:C_1206_3216Metric, symbol Device:C
- added C35: 47uF, Capacitor_SMD:C_1210_3225Metric, symbol Device:C
- added C36: 10uF, Capacitor_SMD:C_1206_3216Metric, symbol Device:C
- added D24, D25: SD05_SOD323, Diode_SMD:D_SOD-323, symbol Diode:SD05_SOD323
- added R22, R23, R29: 1k, Resistor_SMD:R_0805_2012Metric, symbol Device:R
- added R24: 68k, Resistor_SMD:R_0805_2012Metric, symbol Device:R
- added R25: 100, Resistor_SMD:R_0805_2012Metric, symbol Device:R
- added R26, R27, R28: 220k, Resistor_SMD:R_0805_2012Metric, symbol Device:R
- added RV3: 2k, Potentiometer_SMD:Potentiometer_Bourns_3314J_Vertical, symbol Device:R_Potentiometer
- added TP1: A1, TestPoint:TestPoint_Pad_D3.0mm, symbol Connector:TestPoint
- added U23: MCP6021RT-E/OT, Package_TO_SOT_SMD:SOT-23-5, symbol Amplifier_Operational:MCP601-xOT
Connections:
- new net: R23.2, R24.1, R25.1
- new net: C34.1, C35.1, R25.2
- new net: C36.2, RV3.1
- new net: R29.1, RV3.2
- new net: C35.2, R26.2, R27.1, U23.3 (+)
- new net: C36.1, R28.2, U23.4 (-)
- new net +3.3VA: C32.1, C33.1, R26.1
- new net ANALOG_BREAKOUT_IN: R28.1, TP1.1, U23.1
- new net ANALOG_IN_P1+: D25.2 (A2), R23.1
- new net ANALOG_IN_P1-: D24.2 (A2), R22.1
- new net GND: C32.2, C33.2, C34.2, D24.1 (A1), D25.1 (A1), R22.2, R24.2, R27.2, R29.2
- new net R_VDD: U23.5 (V+)
- new net R_VSS: U23.2 (V-)
- no-connect marks 0 -> 1

Commit message: CAN schematic done
Parts:
- renumbered C32 to C39, C33 to C40, C34 to C41, C35 to C42, C36 to C43, D25 to D8, D24 to D9, R23 to R30, R22 to R31, R24 to R32, R25 to R33, R26 to R34, R27 to R35, R28 to R36, R29 to R37, RV3 to RV2, U23 to U21
Changed lines of the file:
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@@
 		(dnp no)
 		(fields_autoplaced yes)
-		(property "Reference" "#PWR076"
+		(property "Reference" "#PWR099"
 			(at 220.98 133.35 0)
 			(effects
@@
 			(project "PRODIGY-MOTHERBOARD"
 				(path "/f1c25860-8989-4190-bd24-2491d23ca7d9/d23a8b72-8742-4bfa-9594-8a2de80e1d70"
-					(reference "#PWR076")
+					(reference "#PWR099")
 					(unit 1)
 				)
@@
 		(dnp no)
 		(fields_autoplaced yes)
-		(property "Reference" "R25"
+		(property "Reference" "R33"
 			(at 152.4 75.565 0)
 			(effects
@@
 			(project "PRODIGY-MOTHERBOARD"
 				(path "/f1c25860-8989-4190-bd24-2491d23ca7d9/d23a8b72-8742-4bfa-9594-8a2de80e1d70"
-					(reference "R25")
+					(reference "R33")
 					(unit 1)
 				)
@@
 		(dnp no)
 		(fields_autoplaced yes)
-		(property "Reference" "RV3"
+		(property "Reference" "RV2"
 			(at 210.82 112.395 0)
 			(effects
@@
 			(project "PRODIGY-MOTHERBOARD"
 				(path "/f1c25860-8989-4190-bd24-2491d23ca7d9/d23a8b72-8742-4bfa-9594-8a2de80e1d70"
-					(reference "RV3")
+					(reference "RV2")
 					(unit 1)
 				)
@@
 		(dnp no)
 		(fields_autoplaced yes)
-		(property "Reference" "D25"
+		(property "Reference" "D8"
 			(at 74.93 105.4099 90)
 			(effects
@@
 			(project "PRODIGY-MOTHERBOARD"
 				(path "/f1c25860-8989-4190-bd24-2491d23ca7d9/d23a8b72-8742-4bfa-9594-8a2de80e1d70"
-					(reference "D25")
+					(reference "D8")
 					(unit 1)
 				)
@@
 		(dnp no)
 		(fields_autoplaced yes)
-		(property "Reference" "#PWR075"
+		(property "Reference" "#PWR098"
 			(at 138.43 107.95 0)
 			(effects
@@
 			(project "PRODIGY-MOTHERBOARD"
 				(path "/f1c25860-8989-4190-bd24-2491d23ca7d9/d23a8b72-8742-4bfa-9594-8a2de80e1d70"
-					(reference "#PWR075")
+					(reference "#PWR098")
 					(unit 1)
 				)
@@
 		(dnp no)
 		(fields_autoplaced yes)
-		(property "Reference" "#PWR077"
+		(property "Reference" "#PWR095"
 			(at 77.47 120.65 0)
 			(effects
@@
 			(project "PRODIGY-MOTHERBOARD"
 				(path "/f1c25860-8989-4190-bd24-2491d23ca7d9/d23a8b72-8742-4bfa-9594-8a2de80e1d70"
-					(reference "#PWR077")
+					(reference "#PWR095")
 					(unit 1)
 				)
@@
 		(on_board yes)
 		(dnp no)
-		(property "Reference" "R22"
+		(property "Reference" "R31"
 			(at 119.38 102.87 90)
 			(effects
@@
 			(project "PRODIGY-MOTHERBOARD"
 				(path "/f1c25860-8989-4190-bd24-2491d23ca7d9/d23a8b72-8742-4bfa-9594-8a2de80e1d70"
-					(reference "R22")
+					(reference "R31")
 					(unit 1)
 				)
@@
 		(on_board yes)
 		(dnp no)
-		(property "Reference" "U23"
+		(property "Reference" "U21"
 			(at 205.74 82.55 0)
 			(effects
@@
 			(project "PRODIGY-MOTHERBOARD"
 				(path "/f1c25860-8989-4190-bd24-2491d23ca7d9/d23a8b72-8742-4bfa-9594-8a2de80e1d70"
-					(reference "U23")
+					(reference "U21")
 					(unit 1)
 				)
@@
 		(dnp no)
 		(fields_autoplaced yes)
-		(property "Reference" "C35"
+		(property "Reference" "C42"
 			(at 163.83 77.47 90)
 			(effects
@@
 			(project "PRODIGY-MOTHERBOARD"
 				(path "/f1c25860-8989-4190-bd24-2491d23ca7d9/d23a8b72-8742-4bfa-9594-8a2de80e1d70"
-					(reference "C35")
+					(reference "C42")
 					(unit 1)
 				)
@@
 		(dnp no)
 		(fields_autoplaced yes)
-		(property "Reference" "R28"
+		(property "Reference" "R36"
 			(at 215.9 90.805 0)
 			(effects
@@
 			(project "PRODIGY-MOTHERBOARD"
 				(path "/f1c25860-8989-4190-bd24-2491d23ca7d9/d23a8b72-8742-4bfa-9594-8a2de80e1d70"
-					(reference "R28")
+					(reference "R36")
 					(unit 1)
 				)
@@
 		(dnp no)
 		(fields_autoplaced yes)
-		(property "Reference" "R29"
+		(property "Reference" "R37"
 			(at 223.52 120.015 0)
 			(effects
@@
 			(project "PRODIGY-MOTHERBOARD"
 				(path "/f1c25860-8989-4190-bd24-2491d23ca7d9/d23a8b72-8742-4bfa-9594-8a2de80e1d70"
-					(reference "R29")
+					(reference "R37")
 					(unit 1)
 				)
@@
 		(dnp no)
 		(fields_autoplaced yes)
-		(property "Reference" "R26"
+		(property "Reference" "R34"
 			(at 176.53 75.565 0)
 			(effects
@@
 			(project "PRODIGY-MOTHERBOARD"
 				(path "/f1c25860-8989-4190-bd24-2491d23ca7d9/d23a8b72-8742-4bfa-9594-8a2de80e1d70"
-					(reference "R26")
+					(reference "R34")
 					(unit 1)
 				)
@@
 		(dnp no)
 		(fields_autoplaced yes)
-		(property "Reference" "C32"
+		(property "Reference" "C39"
 			(at 101.6 71.755 0)
 			(effects
@@
 			(project "PRODIGY-MOTHERBOARD"
 				(path "/f1c25860-8989-4190-bd24-2491d23ca7d9/d23a8b72-8742-4bfa-9594-8a2de80e1d70"
-					(reference "C32")
+					(reference "C39")
 					(unit 1)
 				)
@@
 		(dnp no)
 		(fields_autoplaced yes)
-		(property "Reference" "R27"
+		(property "Reference" "R35"
 			(at 176.53 90.805 0)
 			(effects
@@
 			(project "PRODIGY-MOTHERBOARD"
 				(path "/f1c25860-8989-4190-bd24-2491d23ca7d9/d23a8b72-8742-4bfa-9594-8a2de80e1d70"
-					(reference "R27")
+					(reference "R35")
 					(unit 1)
 				)
@@
 		(dnp no)
 		(fields_autoplaced yes)
-		(property "Reference" "#PWR073"
+		(property "Reference" "#PWR097"
 			(at 97.79 85.09 0)
 			(effects
@@
 			(project "PRODIGY-MOTHERBOARD"
 				(path "/f1c25860-8989-4190-bd24-2491d23ca7d9/d23a8b72-8742-4bfa-9594-8a2de80e1d70"
-					(reference "#PWR073")
+					(reference "#PWR097")
 					(unit 1)
 				)
@@
 		(dnp no)
 		(fields_autoplaced yes)
-		(property "Reference" "D24"
+		(property "Reference" "D9"
 			(at 86.36 105.4099 90)
 			(effects
@@
 			(project "PRODIGY-MOTHERBOARD"
 				(path "/f1c25860-8989-4190-bd24-2491d23ca7d9/d23a8b72-8742-4bfa-9594-8a2de80e1d70"
-					(reference "D24")
+					(reference "D9")
 					(unit 1)
 				)
@@
 		(dnp no)
 		(fields_autoplaced yes)
-		(property "Reference" "C36"
+		(property "Reference" "C43"
 			(at 217.17 102.235 0)
 			(effects
@@
 			(project "PRODIGY-MOTHERBOARD"
 				(path "/f1c25860-8989-4190-bd24-2491d23ca7d9/d23a8b72-8742-4bfa-9594-8a2de80e1d70"
-					(reference "C36")
+					(reference "C43")
 					(unit 1)
 				)
@@
 		(dnp no)
 		(fields_autoplaced yes)
-		(property "Reference" "#PWR074"
+		(property "Reference" "#PWR096"
 			(at 83.82 120.65 0)
 			(effects
@@
 			(project "PRODIGY-MOTHERBOARD"
 				(path "/f1c25860-8989-4190-bd24-2491d23ca7d9/d23a8b72-8742-4bfa-9594-8a2de80e1d70"
-					(reference "#PWR074")
+					(reference "#PWR096")
 					(unit 1)
 				)
@@
 		(dnp no)
 		(fields_autoplaced yes)
-		(property "Reference" "C33"
+		(property "Reference" "C40"
 			(at 113.03 71.1199 0)
 			(effects
@@
 			(project "PRODIGY-MOTHERBOARD"
 				(path "/f1c25860-8989-4190-bd24-2491d23ca7d9/d23a8b72-8742-4bfa-9594-8a2de80e1d70"
-					(reference "C33")
+					(reference "C40")
 					(unit 1)
 				)
@@
 		(on_board yes)
 		(dnp no)
-		(property "Reference" "C34"
+		(property "Reference" "C41"
 			(at 153.67 90.805 0)
 			(effects
@@
 			(project "PRODIGY-MOTHERBOARD"
 				(path "/f1c25860-8989-4190-bd24-2491d23ca7d9/d23a8b72-8742-4bfa-9594-8a2de80e1d70"
-					(reference "C34")
+					(reference "C41")
 					(unit 1)
 				)
@@
 		(dnp no)
 		(fields_autoplaced yes)
-		(property "Reference" "R23"
+		(property "Reference" "R30"
 			(at 107.95 90.17 90)
 			(effects
@@
 			(project "PRODIGY-MOTHERBOARD"
 				(path "/f1c25860-8989-4190-bd24-2491d23ca7d9/d23a8b72-8742-4bfa-9594-8a2de80e1d70"
-					(reference "R23")
+					(reference "R30")
 					(unit 1)
 				)
@@
 		(dnp no)
 		(fields_autoplaced yes)
-		(property "Reference" "R24"
+		(property "Reference" "R32"
 			(at 140.97 83.185 0)
 			(effects
@@
 			(project "PRODIGY-MOTHERBOARD"
 				(path "/f1c25860-8989-4190-bd24-2491d23ca7d9/d23a8b72-8742-4bfa-9594-8a2de80e1d70"
-					(reference "R24")
+					(reference "R32")
 					(unit 1)
 				)
@@
 		(dnp no)
 		(fields_autoplaced yes)
-		(property "Reference" "#FLG02"
+		(property "Reference" "#FLG03"
 			(at 173.99 65.405 0)
 			(effects
@@
 			(project "PRODIGY-MOTHERBOARD"
 				(path "/f1c25860-8989-4190-bd24-2491d23ca7d9/d23a8b72-8742-4bfa-9594-8a2de80e1d70"
-					(reference "#FLG02")
+					(reference "#FLG03")
 					(unit 1)
 				)
@@
 		(dnp no)
 		(fields_autoplaced yes)
-		(property "Reference" "#FLG01"
+		(property "Reference" "#FLG02"
 			(at 104.14 62.865 0)
 			(effects
@@
 			(project "PRODIGY-MOTHERBOARD"
 				(path "/f1c25860-8989-4190-bd24-2491d23ca7d9/d23a8b72-8742-4bfa-9594-8a2de80e1d70"
-					(reference "#FLG01")
-					(unit 1)
-				)
+					(reference "#FLG02")
+					(unit 1)
+				)

Commit message: SPI NFC schematic done.
Parts:
- renumbered C39 to C56, C40 to C57, C41 to C58, C42 to C59, C43 to C60, D8 to D10, D9 to D11, R30 to R35, R31 to R36, R32 to R37, R33 to R38, R34 to R39, R35 to R40, R36 to R41, R37 to R42
Changed lines of the file:
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@@
 		(dnp no)
 		(fields_autoplaced yes)
-		(property "Reference" "#PWR099"
+		(property "Reference" "#PWR0118"
 			(at 220.98 133.35 0)
 			(effects
@@
 			(project "PRODIGY-MOTHERBOARD"
 				(path "/f1c25860-8989-4190-bd24-2491d23ca7d9/d23a8b72-8742-4bfa-9594-8a2de80e1d70"
-					(reference "#PWR099")
+					(reference "#PWR0118")
 					(unit 1)
 				)
@@
 		(dnp no)
 		(fields_autoplaced yes)
-		(property "Reference" "R33"
+		(property "Reference" "R38"
 			(at 152.4 75.565 0)
 			(effects
@@
 			(project "PRODIGY-MOTHERBOARD"
 				(path "/f1c25860-8989-4190-bd24-2491d23ca7d9/d23a8b72-8742-4bfa-9594-8a2de80e1d70"
-					(reference "R33")
+					(reference "R38")
 					(unit 1)
 				)
@@
 		(dnp no)
 		(fields_autoplaced yes)
-		(property "Reference" "D8"
+		(property "Reference" "D10"
 			(at 74.93 105.4099 90)
 			(effects
@@
 			(project "PRODIGY-MOTHERBOARD"
 				(path "/f1c25860-8989-4190-bd24-2491d23ca7d9/d23a8b72-8742-4bfa-9594-8a2de80e1d70"
-					(reference "D8")
+					(reference "D10")
 					(unit 1)
 				)
@@
 		(dnp no)
 		(fields_autoplaced yes)
-		(property "Reference" "#PWR098"
+		(property "Reference" "#PWR0117"
 			(at 138.43 107.95 0)
 			(effects
@@
 			(project "PRODIGY-MOTHERBOARD"
 				(path "/f1c25860-8989-4190-bd24-2491d23ca7d9/d23a8b72-8742-4bfa-9594-8a2de80e1d70"
-					(reference "#PWR098")
+					(reference "#PWR0117")
 					(unit 1)
 				)
@@
 		(dnp no)
 		(fields_autoplaced yes)
-		(property "Reference" "#PWR095"
+		(property "Reference" "#PWR0114"
 			(at 77.47 120.65 0)
 			(effects
@@
 			(project "PRODIGY-MOTHERBOARD"
 				(path "/f1c25860-8989-4190-bd24-2491d23ca7d9/d23a8b72-8742-4bfa-9594-8a2de80e1d70"
-					(reference "#PWR095")
+					(reference "#PWR0114")
 					(unit 1)
 				)
@@
 		(on_board yes)
 		(dnp no)
-		(property "Reference" "R31"
+		(property "Reference" "R36"
 			(at 119.38 102.87 90)
 			(effects
@@
 			(project "PRODIGY-MOTHERBOARD"
 				(path "/f1c25860-8989-4190-bd24-2491d23ca7d9/d23a8b72-8742-4bfa-9594-8a2de80e1d70"
-					(reference "R31")
+					(reference "R36")
 					(unit 1)
 				)
@@
 		(dnp no)
 		(fields_autoplaced yes)
-		(property "Reference" "C42"
+		(property "Reference" "C59"
 			(at 163.83 77.47 90)
 			(effects
@@
 			(project "PRODIGY-MOTHERBOARD"
 				(path "/f1c25860-8989-4190-bd24-2491d23ca7d9/d23a8b72-8742-4bfa-9594-8a2de80e1d70"
-					(reference "C42")
+					(reference "C59")
 					(unit 1)
 				)
@@
 		(dnp no)
 		(fields_autoplaced yes)
-		(property "Reference" "R36"
+		(property "Reference" "R41"
 			(at 215.9 90.805 0)
 			(effects
@@
 			(project "PRODIGY-MOTHERBOARD"
 				(path "/f1c25860-8989-4190-bd24-2491d23ca7d9/d23a8b72-8742-4bfa-9594-8a2de80e1d70"
-					(reference "R36")
+					(reference "R41")
 					(unit 1)
 				)
@@
 		(dnp no)
 		(fields_autoplaced yes)
-		(property "Reference" "R37"
+		(property "Reference" "R42"
 			(at 223.52 120.015 0)
 			(effects
@@
 			(project "PRODIGY-MOTHERBOARD"
 				(path "/f1c25860-8989-4190-bd24-2491d23ca7d9/d23a8b72-8742-4bfa-9594-8a2de80e1d70"
-					(reference "R37")
+					(reference "R42")
 					(unit 1)
 				)
@@
 		(dnp no)
 		(fields_autoplaced yes)
-		(property "Reference" "R34"
+		(property "Reference" "R39"
 			(at 176.53 75.565 0)
 			(effects
@@
 			(project "PRODIGY-MOTHERBOARD"
 				(path "/f1c25860-8989-4190-bd24-2491d23ca7d9/d23a8b72-8742-4bfa-9594-8a2de80e1d70"
-					(reference "R34")
+					(reference "R39")
 					(unit 1)
 				)
@@
 		(dnp no)
 		(fields_autoplaced yes)
-		(property "Reference" "C39"
+		(property "Reference" "C56"
 			(at 101.6 71.755 0)
 			(effects
@@
 			(project "PRODIGY-MOTHERBOARD"
 				(path "/f1c25860-8989-4190-bd24-2491d23ca7d9/d23a8b72-8742-4bfa-9594-8a2de80e1d70"
-					(reference "C39")
+					(reference "C56")
 					(unit 1)
 				)
@@
 		(dnp no)
 		(fields_autoplaced yes)
-		(property "Reference" "R35"
+		(property "Reference" "R40"
 			(at 176.53 90.805 0)
 			(effects
@@
 			(project "PRODIGY-MOTHERBOARD"
 				(path "/f1c25860-8989-4190-bd24-2491d23ca7d9/d23a8b72-8742-4bfa-9594-8a2de80e1d70"
-					(reference "R35")
+					(reference "R40")
 					(unit 1)
 				)
@@
 		(dnp no)
 		(fields_autoplaced yes)
-		(property "Reference" "#PWR097"
+		(property "Reference" "#PWR0116"
 			(at 97.79 85.09 0)
 			(effects
@@
 			(project "PRODIGY-MOTHERBOARD"
 				(path "/f1c25860-8989-4190-bd24-2491d23ca7d9/d23a8b72-8742-4bfa-9594-8a2de80e1d70"
-					(reference "#PWR097")
+					(reference "#PWR0116")
 					(unit 1)
 				)
@@
 		(dnp no)
 		(fields_autoplaced yes)
-		(property "Reference" "D9"
+		(property "Reference" "D11"
 			(at 86.36 105.4099 90)
 			(effects
@@
 			(project "PRODIGY-MOTHERBOARD"
 				(path "/f1c25860-8989-4190-bd24-2491d23ca7d9/d23a8b72-8742-4bfa-9594-8a2de80e1d70"
-					(reference "D9")
+					(reference "D11")
 					(unit 1)
 				)
@@
 		(dnp no)
 		(fields_autoplaced yes)
-		(property "Reference" "C43"
+		(property "Reference" "C60"
 			(at 217.17 102.235 0)
 			(effects
@@
 			(project "PRODIGY-MOTHERBOARD"
 				(path "/f1c25860-8989-4190-bd24-2491d23ca7d9/d23a8b72-8742-4bfa-9594-8a2de80e1d70"
-					(reference "C43")
+					(reference "C60")
 					(unit 1)
 				)
@@
 		(dnp no)
 		(fields_autoplaced yes)
-		(property "Reference" "#PWR096"
+		(property "Reference" "#PWR0115"
 			(at 83.82 120.65 0)
 			(effects
@@
 			(project "PRODIGY-MOTHERBOARD"
 				(path "/f1c25860-8989-4190-bd24-2491d23ca7d9/d23a8b72-8742-4bfa-9594-8a2de80e1d70"
-					(reference "#PWR096")
+					(reference "#PWR0115")
 					(unit 1)
 				)
@@
 		(dnp no)
 		(fields_autoplaced yes)
-		(property "Reference" "C40"
+		(property "Reference" "C57"
 			(at 113.03 71.1199 0)
 			(effects
@@
 			(project "PRODIGY-MOTHERBOARD"
 				(path "/f1c25860-8989-4190-bd24-2491d23ca7d9/d23a8b72-8742-4bfa-9594-8a2de80e1d70"
-					(reference "C40")
+					(reference "C57")
 					(unit 1)
 				)
@@
 		(on_board yes)
 		(dnp no)
-		(property "Reference" "C41"
+		(property "Reference" "C58"
 			(at 153.67 90.805 0)
 			(effects
@@
 			(project "PRODIGY-MOTHERBOARD"
 				(path "/f1c25860-8989-4190-bd24-2491d23ca7d9/d23a8b72-8742-4bfa-9594-8a2de80e1d70"
-					(reference "C41")
+					(reference "C58")
 					(unit 1)
 				)
@@
 		(dnp no)
 		(fields_autoplaced yes)
-		(property "Reference" "R30"
+		(property "Reference" "R35"
 			(at 107.95 90.17 90)
 			(effects
@@
 			(project "PRODIGY-MOTHERBOARD"
 				(path "/f1c25860-8989-4190-bd24-2491d23ca7d9/d23a8b72-8742-4bfa-9594-8a2de80e1d70"
-					(reference "R30")
+					(reference "R35")
 					(unit 1)
 				)
@@
 		(dnp no)
 		(fields_autoplaced yes)
-		(property "Reference" "R32"
+		(property "Reference" "R37"
 			(at 140.97 83.185 0)
 			(effects
@@
 			(project "PRODIGY-MOTHERBOARD"
 				(path "/f1c25860-8989-4190-bd24-2491d23ca7d9/d23a8b72-8742-4bfa-9594-8a2de80e1d70"
-					(reference "R32")
-					(unit 1)
-				)
+					(reference "R37")
+					(unit 1)
+				)

Commit message: Analog schematic finished, except the joystick part.
Parts:
- removed D10, D11: SD05_SOD323, Diode_SMD:D_SOD-323, symbol Diode:SD05_SOD323
Connections:
- net ANALOG_BREAKOUT_IN renamed ANALOG_BREAKOUT_OUT

Commit message: Added pins to MCU. Added Decoder for SPI SS-Multiplexing.
Other:
- moved on the sheet: C56, C57, C58, C59, C60, R35, R36, R37, R38, R39, R40, R41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
