File: PRODIGY-MOTHERBOARD/filter.kicad_sch (KiCad schematic)
At the start: 16 parts, among them U21 MCP6021RT-E/OT

Commit message: Added proper debounce filter elements to buttons.
Parts:
- renumbered C56 to C65, C57 to C66, C59 to C67, C58 to C68, C60 to C69, R38 to R41, R39 to R42, R37 to R43, R40 to R44, R41 to R45, R35 to R46, R36 to R47, R42 to R48, U21 to U22
Changed lines of the file:
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@@
 		(dnp no)
 		(fields_autoplaced yes)
-		(property "Reference" "#PWR0118"
+		(property "Reference" "#PWR0132"
 			(at 205.74 133.35 0)
 			(effects
@@
 			(project "PRODIGY-MOTHERBOARD"
 				(path "/f1c25860-8989-4190-bd24-2491d23ca7d9/d23a8b72-8742-4bfa-9594-8a2de80e1d70"
-					(reference "#PWR0118")
+					(reference "#PWR0132")
 					(unit 1)
 				)
@@
 		(dnp no)
 		(fields_autoplaced yes)
-		(property "Reference" "R38"
+		(property "Reference" "R41"
 			(at 137.16 75.565 0)
 			(effects
@@
 			(project "PRODIGY-MOTHERBOARD"
 				(path "/f1c25860-8989-4190-bd24-2491d23ca7d9/d23a8b72-8742-4bfa-9594-8a2de80e1d70"
-					(reference "R38")
+					(reference "R41")
 					(unit 1)
 				)
@@
 		(dnp no)
 		(fields_autoplaced yes)
-		(property "Reference" "#PWR0117"
+		(property "Reference" "#PWR0131"
 			(at 123.19 107.95 0)
 			(effects
@@
 			(project "PRODIGY-MOTHERBOARD"
 				(path "/f1c25860-8989-4190-bd24-2491d23ca7d9/d23a8b72-8742-4bfa-9594-8a2de80e1d70"
-					(reference "#PWR0117")
+					(reference "#PWR0131")
 					(unit 1)
 				)
@@
 		(on_board yes)
 		(dnp no)
-		(property "Reference" "R36"
+		(property "Reference" "R47"
 			(at 104.14 102.87 90)
 			(effects
@@
 			(project "PRODIGY-MOTHERBOARD"
 				(path "/f1c25860-8989-4190-bd24-2491d23ca7d9/d23a8b72-8742-4bfa-9594-8a2de80e1d70"
-					(reference "R36")
+					(reference "R47")
 					(unit 1)
 				)
@@
 		(on_board yes)
 		(dnp no)
-		(property "Reference" "U21"
+		(property "Reference" "U22"
 			(at 190.5 82.55 0)
 			(effects
@@
 			(project "PRODIGY-MOTHERBOARD"
 				(path "/f1c25860-8989-4190-bd24-2491d23ca7d9/d23a8b72-8742-4bfa-9594-8a2de80e1d70"
-					(reference "U21")
+					(reference "U22")
 					(unit 1)
 				)
@@
 		(dnp no)
 		(fields_autoplaced yes)
-		(property "Reference" "C59"
+		(property "Reference" "C67"
 			(at 148.59 77.47 90)
 			(effects
@@
 			(project "PRODIGY-MOTHERBOARD"
 				(path "/f1c25860-8989-4190-bd24-2491d23ca7d9/d23a8b72-8742-4bfa-9594-8a2de80e1d70"
-					(reference "C59")
+					(reference "C67")
 					(unit 1)
 				)
@@
 		(dnp no)
 		(fields_autoplaced yes)
-		(property "Reference" "R41"
+		(property "Reference" "R45"
 			(at 200.66 90.805 0)
 			(effects
@@
 			(project "PRODIGY-MOTHERBOARD"
 				(path "/f1c25860-8989-4190-bd24-2491d23ca7d9/d23a8b72-8742-4bfa-9594-8a2de80e1d70"
-					(reference "R41")
+					(reference "R45")
 					(unit 1)
 				)
@@
 		(dnp no)
 		(fields_autoplaced yes)
-		(property "Reference" "R42"
+		(property "Reference" "R48"
 			(at 208.28 120.015 0)
 			(effects
@@
 			(project "PRODIGY-MOTHERBOARD"
 				(path "/f1c25860-8989-4190-bd24-2491d23ca7d9/d23a8b72-8742-4bfa-9594-8a2de80e1d70"
-					(reference "R42")
+					(reference "R48")
 					(unit 1)
 				)
@@
 		(dnp no)
 		(fields_autoplaced yes)
-		(property "Reference" "R39"
+		(property "Reference" "R42"
 			(at 161.29 75.565 0)
 			(effects
@@
 			(project "PRODIGY-MOTHERBOARD"
 				(path "/f1c25860-8989-4190-bd24-2491d23ca7d9/d23a8b72-8742-4bfa-9594-8a2de80e1d70"
-					(reference "R39")
+					(reference "R42")
 					(unit 1)
 				)
@@
 		(dnp no)
 		(fields_autoplaced yes)
-		(property "Reference" "C56"
+		(property "Reference" "C65"
 			(at 86.36 71.755 0)
 			(effects
@@
 			(project "PRODIGY-MOTHERBOARD"
 				(path "/f1c25860-8989-4190-bd24-2491d23ca7d9/d23a8b72-8742-4bfa-9594-8a2de80e1d70"
-					(reference "C56")
+					(reference "C65")
 					(unit 1)
 				)
@@
 		(dnp no)
 		(fields_autoplaced yes)
-		(property "Reference" "R40"
+		(property "Reference" "R44"
 			(at 161.29 90.805 0)
 			(effects
@@
 			(project "PRODIGY-MOTHERBOARD"
 				(path "/f1c25860-8989-4190-bd24-2491d23ca7d9/d23a8b72-8742-4bfa-9594-8a2de80e1d70"
-					(reference "R40")
+					(reference "R44")
 					(unit 1)
 				)
@@
 		(dnp no)
 		(fields_autoplaced yes)
-		(property "Reference" "#PWR0116"
+		(property "Reference" "#PWR0130"
 			(at 82.55 85.09 0)
 			(effects
@@
 			(project "PRODIGY-MOTHERBOARD"
 				(path "/f1c25860-8989-4190-bd24-2491d23ca7d9/d23a8b72-8742-4bfa-9594-8a2de80e1d70"
-					(reference "#PWR0116")
+					(reference "#PWR0130")
 					(unit 1)
 				)
@@
 		(dnp no)
 		(fields_autoplaced yes)
-		(property "Reference" "C60"
+		(property "Reference" "C69"
 			(at 201.93 102.235 0)
 			(effects
@@
 			(project "PRODIGY-MOTHERBOARD"
 				(path "/f1c25860-8989-4190-bd24-2491d23ca7d9/d23a8b72-8742-4bfa-9594-8a2de80e1d70"
-					(reference "C60")
+					(reference "C69")
 					(unit 1)
 				)
@@
 		(dnp no)
 		(fields_autoplaced yes)
-		(property "Reference" "C57"
+		(property "Reference" "C66"
 			(at 97.79 71.1199 0)
 			(effects
@@
 			(project "PRODIGY-MOTHERBOARD"
 				(path "/f1c25860-8989-4190-bd24-2491d23ca7d9/d23a8b72-8742-4bfa-9594-8a2de80e1d70"
-					(reference "C57")
+					(reference "C66")
 					(unit 1)
 				)
@@
 		(on_board yes)
 		(dnp no)
-		(property "Reference" "C58"
+		(property "Reference" "C68"
 			(at 138.43 90.805 0)
 			(effects
@@
 			(project "PRODIGY-MOTHERBOARD"
 				(path "/f1c25860-8989-4190-bd24-2491d23ca7d9/d23a8b72-8742-4bfa-9594-8a2de80e1d70"
-					(reference "C58")
+					(reference "C68")
 					(unit 1)
 				)
@@
 		(dnp no)
 		(fields_autoplaced yes)
-		(property "Reference" "R35"
+		(property "Reference" "R46"
 			(at 92.71 90.17 90)
 			(effects
@@
 			(project "PRODIGY-MOTHERBOARD"
 				(path "/f1c25860-8989-4190-bd24-2491d23ca7d9/d23a8b72-8742-4bfa-9594-8a2de80e1d70"
-					(reference "R35")
+					(reference "R46")
 					(unit 1)
 				)
@@
 		(dnp no)
 		(fields_autoplaced yes)
-		(property "Reference" "R37"
+		(property "Reference" "R43"
 			(at 125.73 83.185 0)
 			(effects
@@
 			(project "PRODIGY-MOTHERBOARD"
 				(path "/f1c25860-8989-4190-bd24-2491d23ca7d9/d23a8b72-8742-4bfa-9594-8a2de80e1d70"
-					(reference "R37")
-					(unit 1)
-				)
+					(reference "R43")
+					(unit 1)
+				)

Commit message: Submitted V0 for evaluation. Avaiting feedback.
Parts:
- renumbered R41 to R42, R42 to R43, R43 to R44, R44 to R45, R45 to R46, R46 to R47, R47 to R48, R48 to R49, U22 to U23
Connections:
- net +3.3VA renamed +3V3
