File: PRODIGY-MOTHERBOARD/strain_gauge.kicad_sch (KiCad schematic)
At the start: 0 parts

Commit message: Finished v0.1 schematic.
Parts:
- added C90: 47uF, symbol Device:C
- added R88, R89, R90, R93, R94, R95: 10k, symbol Device:R
- added R91: 3.205k, symbol Device:R
- added R92: 2.5k, symbol Device:R
- added U28: LM4125AIM5-2.5, Package_TO_SOT_SMD:SOT-23-5, symbol Reference_Voltage:LM4125AIM5-2.5
- added U29, U30, U31, U32: LMP2011, Package_TO_SOT_SMD:TSOT-23-5, symbol Amplifier_Operational:AD8603
Connections:
- new net: R94.2, R95.1, U31.4 (-)
- new net: C90.1, U28.5 (Vout), U29.3 (+)
- new net: R90.2, R91.1, U30.4 (-)
- new net: R91.2, R93.1, U32.3 (+)
- new net: R88.1, R90.1, U30.1
- new net: R88.2, R89.1, U31.3 (+)
- new net: R93.2, R94.1, U32.1
- new net +3.3VA: U28.4 (Vin), U29.5 (V+), U30.5 (V+), U31.5 (V+), U32.5 (V+)
- new net GND: C90.2, R89.2, R92.2, U28.2 (GND), U29.2 (V-), U30.2 (V-), U31.2 (V-), U32.2 (V-)
- new net Loadcell_A_Excitation+: U29.1
- new net Loadcell_A_Excitation-: R92.1, U29.4 (-)
- new net Loadcell_A_Signal+: U30.3 (+)
- new net Loadcell_A_Signal-: U32.4 (-)
- new net Strain_Gauge_A_OUT: R95.2, U31.1
Other:
- note added: "Constant Current Source: 1mA 1mA = 2.5V / 2.5kOhm"
- note added: "Instrumentation Amplifier"
- note added: "Output voltage range: 0,1V - 0.34528V Gain: 2.5/0.34528 = 7.2405 R7 = 3.205k"
