File: PRODIGY-MOTHERBOARD/i2c_devices.kicad_sch (KiCad schematic)
At the start: 24 parts, among them J19 KEYPAD_MATRIX, J25 OLED, Q3 BC850, U12 PCF8574, U19 PCF8574, U20 LIS2DH12TR, U8 HDC1080

Commit message: CAN schematic done
Parts:
- renumbered C25 to C32, C26 to C33, C27 to C34, C29 to C35, C30 to C36, C28 to C37, C31 to C38, J19 to J26, J25 to J27, Q3 to Q2, RN1 to RN3, RN3 to RN4, RV2 to RV1, U12 to U17, U19 to U18, U8 to U19

Commit message: SPI NFC schematic done.
Parts:
- renumbered C32 to C49, C33 to C50, C34 to C51, C35 to C52, C36 to C53, C37 to C54, C38 to C55

Commit message: Added proper debounce filter elements to buttons.
Parts:
- renumbered C52 to C58, C53 to C59, C51 to C60, C49 to C61, C55 to C62, C54 to C63, C50 to C64, J27 to J26, J26 to J27, JP3 to JP2, JP5 to JP3, JP2 to JP4, JP4 to JP5, U20 to U18, U17 to U19, U19 to U20, U18 to U21

Commit message: Submitted V0 for evaluation. Avaiting feedback.
Parts:
- renumbered J26 to J18, J27 to J19, JP1 to JP4, JP2 to JP5, JP3 to JP6, JP4 to JP7, JP5 to JP8, JP6 to JP9, U18 to U19, U19 to U20, U20 to U21, U21 to U22
Connections:
- net GND: now also U19.5 (RES)
Other:
- note added: "Oled can be removed, but it expands the board's capabilities at minimal cost (More noise and I2C traffic)"

Commit message: Finished v0.1 schematic.
Parts:
- added FID11, FID12, FID13, FID14: Fiducial, symbol Mechanical:Fiducial
- renumbered C61 to C35, C64 to C36, C60 to C37, C58 to C38, C59 to C39, C63 to C40, C62 to C41, J18 to J20, JP4 to JP2, JP7 to JP3, JP5 to JP4, JP8 to JP5, JP9 to JP7, Q2 to Q1, RN3 to RN1, RN4 to RN2, U22 to U10, U21 to U11, U19 to U12, U20 to U9
Other:
- note removed: "Oled can be removed, but it expands the board's capabilities at minimal cost (More noise and I2C traffic)"

Commit message: MBT Schematic improved
Parts:
- J20: footprint (none) -> Connector_PinSocket_2.54mm:PinSocket_1x04_P2.54mm_Vertical
Changed lines of the file:
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@@
 			)
 		)
-		(property "Footprint" ""
+		(property "Footprint" "Connector_PinSocket_2.54mm:PinSocket_1x04_P2.54mm_Vertical"
 			(at 254 88.9 0)
 			(effects

Commit message: schematic v0.2 finalized
Parts:
- renumbered C35 to C34, C36 to C35, C37 to C36, C38 to C37, C39 to C38, C40 to C39, C41 to C40, FID11 to FID13, FID12 to FID14, FID13 to FID15, FID14 to FID16, JP2 to JP3, JP3 to JP4, JP4 to JP5, JP5 to JP6, JP6 to JP7, JP7 to JP8

Commit message: Motherboard footprints assigned.
Parts:
- C34, C35, C38, C39: footprint (none) -> Capacitor_SMD:C_0603_1608Metric
- C36, C37, C40: footprint (none) -> Capacitor_SMD:C_0805_2012Metric
- FID13, FID14, FID15, FID16: footprint (none) -> Fiducial:Fiducial_1mm_Mask3mm
- JP3, JP4, JP5, JP6, JP7, JP8: footprint (none) -> Jumper:SolderJumper-2_P1.3mm_Open_Pad1.0x1.5mm
- RN1, RN2: footprint Resistor_SMD:R_Array_Convex_4x0603 -> Resistor_SMD:R_0603_1608Metric
- RV1: footprint Potentiometer_SMD:Potentiometer_Bourns_3224J_Horizontal -> Potentiometer_SMD:Potentiometer_Bourns_3314J_Vertical
