File: PRODIGY-MOTHERBOARD/i2c_devices.kicad_sch (KiCad schematic)
At the start: 28 parts, among them J19 KEYPAD_MATRIX, J20 OLED, Q1 BC850, U10 PCF8574, U11 HDC1080, U12 LIS2DH12TR, U9 PCF8574

Commit message: finished motherboard bom and updated footprints
Parts:
- C34, C35, C38, C39: TME (none) -> CL10B104KB8NNNC
- C36, C37, C40: TME (none) -> CL21A106KOQNNNE
- DS1: TME (none) -> RC1602B-BIW-ESV
- FID13, FID14, FID15, FID16: now not fitted
- J19: TME (none) -> M20-8770842
- J20: TME (none) -> ZL262-4SG
- JP3, JP4, JP5, JP6, JP7, JP8: now not fitted; now left out of the parts list
- Q1: TME (none) -> BC850B-DIO
- RN1, RN2: value 4.7k -> 10k; TME (none) -> DR1206-10K-4/8
- RV1: TME (none) -> 3314J-1-103E
- U10, U9: TME (none) -> PCF8574TS/3.118
- U11: MOUSER (none) -> 595-HDC1080DMBR
- U12: MOUSER (none) -> 511-LIS2DH12TR

Commit message: Motherboard PCB layout started
Parts:
- removed FID13, FID15, FID16: Fiducial, Fiducial:Fiducial_1mm_Mask3mm, symbol Mechanical:Fiducial
- RN1, RN2: footprint Resistor_SMD:R_0603_1608Metric -> Resistor_SMD:R_Array_Concave_4x0603

Commit message: Resistor array fixed, layout main components locked, high speed routing done
Parts:
- removed RN2: 10k, Resistor_SMD:R_Array_Concave_4x0603, symbol Device:R_Network04
- added RN2: R_Pack04, Resistor_SMD:R_Array_Convex_4x0603, symbol Device:R_Pack04
Connections:
- net +5V: now also RN2.5 (R4.2), RN2.6 (R3.2), RN2.7 (R2.2), RN2.8 (R1.2)
- net INTERRUPT_KEYPAD: now also RN2.1 (R1.1)
- net at JP4.2 (B), U10.3 (A2): now also RN2.2 (R2.1)
- net at JP8.2 (B), U10.1 (A0): now also RN2.4 (R4.1)
- net at JP6.2 (B), U10.2 (A1): now also RN2.3 (R3.1)
Changed lines of the file:
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@@
+	)
+	(junction
+		(at 74.93 123.19)
+		(diameter 0)
+		(color 0 0 0 0)
 	)
 	(junction
@@
 	)
 	(junction
+		(at 72.39 123.19)
+		(diameter 0)
+		(color 0 0 0 0)
+	)
+	(junction
 		(at 151.13 27.94)
 		(diameter 0)
@@
 		(color 0 0 0 0)
 	)
+	(junction
+		(at 69.85 123.19)
+		(diameter 0)
+		(color 0 0 0 0)
+	)
 	(no_connect
 		(at 243.84 41.91)
@@
 	(wire
 		(pts
+			(xy 72.39 123.19) (xy 74.93 123.19)
+		)
+		(stroke
+			(width 0)
+			(type default)
+		)
+	)
+	(wire
+		(pts
 			(xy 158.75 27.94) (xy 151.13 27.94)
 		)
@@
 	(wire
 		(pts
+			(xy 67.31 123.19) (xy 69.85 123.19)
+		)
+		(stroke
+			(width 0)
+			(type default)
+		)
+	)
+	(wire
+		(pts
 			(xy 147.32 44.45) (xy 151.13 44.45)
 		)
@@
 		(pts
 			(xy 53.34 181.61) (xy 67.31 181.61)
+		)
+		(stroke
+			(width 0)
+			(type default)
+		)
+	)
+	(wire
+		(pts
+			(xy 69.85 123.19) (xy 72.39 123.19)
 		)
 		(stroke
@@
 	)
 	(symbol
+		(lib_id "Device:R_Pack04")
+		(at 72.39 128.27 0)
+		(unit 1)
+		(exclude_from_sim no)
+		(in_bom yes)
+		(on_board yes)
+		(dnp no)
+		(fields_autoplaced yes)
+		(property "Reference" "RN2"
+			(at 77.47 126.9999 0)
+			(effects
+				(font
+					(size 1.27 1.27)
+				)
+				(justify left)
+			)
+		)
+		(property "Value" "R_Pack04"
+			(at 77.47 129.5399 0)
+			(effects
+				(font
+					(size 1.27 1.27)
+				)
+				(justify left)
+			)
+		)
+		(property "Footprint" "Resistor_SMD:R_Array_Convex_4x0603"
+			(at 79.375 128.27 90)
+			(effects
+				(font
+					(size 1.27 1.27)
+				)
+				(hide yes)
+			)
+		)
+		(property "Datasheet" "~"
+			(at 72.39 128.27 0)
+			(effects
+				(font
+					(size 1.27 1.27)
+				)
+				(hide yes)
+			)
+		)
+		(property "Description" "4 resistor network, parallel topology"
+			(at 72.39 128.27 0)
+			(effects
+				(font
+					(size 1.27 1.27)
+				)
+				(hide yes)
+			)
+		)
+		(pin "8"
+		)
+		(pin "4"
+		)
+		(pin "5"
+		)
+		(pin "2"
+		)
+		(pin "7"
+		)
+		(pin "6"
+		)
+		(pin "1"
+		)
+		(pin "3"
+		)
+		(instances
+			(project "PRODIGY-MOTHERBOARD"
+				(path "/f1c25860-8989-4190-bd24-2491d23ca7d9/68745e9f-546d-4e12-ac2b-ba23aeab0093/94efb13e-f47a-4ad5-a80b-985c2164e820"
+					(reference "RN2")
+					(unit 1)
+				)
+			)
+		)
+	)
+	(symbol
 		(lib_id "power:GND")
 		(at 25.4 78.74 0)
@@
 					(unit 1)
 				)
-			)
-		)
-	)
-	(symbol
-		(lib_id "Device:R_Network04")
-		(at 69.85 128.27 0)
-		(mirror y)
-		(unit 1)
-		(exclude_from_sim no)
-		(in_bom yes)
-		(on_board yes)
-		(dnp no)
-		(property "Reference" "RN2"
-			(at 77.47 127.2539 0)
-			(effects
-				(font
-					(size 1.27 1.27)
-				)
-				(justify right)
-			)
-		)
-		(property "Value" "10k"
-			(at 77.47 129.7939 0)
-			(effects
-				(font
-					(size 1.27 1.27)
-				)
-				(justify right)
-			)
-		)
-		(property "Footprint" "Resistor_SMD:R_Array_Concave_4x0603"
-			(at 62.865 128.27 90)
-			(effects
-				(font
-					(size 1.27 1.27)
-				)
-				(hide yes)
-			)
-		)
-		(property "Datasheet" "http://www.vishay.com/docs/31509/csc.pdf"
-			(at 69.85 128.27 0)
-			(effects
-				(font
-					(size 1.27 1.27)
-				)
-				(hide yes)
-			)
-		)
-		(property "Description" "4 resistor network, star topology, bussed resistors, small symbol"
-			(at 69.85 128.27 0)
-			(effects
-				(font
-					(size 1.27 1.27)
-				)
-				(hide yes)
-			)
-		)
-		(property "MOUSER" ""
-			(at 69.85 128.27 0)
-			(effects
-				(font
-					(size 1.27 1.27)
-				)
-				(hide yes)
-			)
-		)
-		(property "Sim.Type" ""
-			(at 69.85 128.27 0)
-			(effects
-				(font
-					(size 1.27 1.27)
-				)
-				(hide yes)
-			)
-		)
-		(property "TME" "DR1206-10K-4/8"
-			(at 69.85 128.27 0)
-			(effects
-				(font
-					(size 1.27 1.27)
-				)
-				(hide yes)
-			)
-		)
-		(pin "2"
-		)
-		(pin "4"
-		)
-		(pin "3"
-		)
-		(pin "1"
-		)
-		(pin "5"
-		)
-		(instances
-			(project "PRODIGY-MOTHERBOARD"
-				(path "/f1c25860-8989-4190-bd24-2491d23ca7d9/68745e9f-546d-4e12-ac2b-ba23aeab0093/94efb13e-f47a-4ad5-a80b-985c2164e820"
-					(reference "RN2")
-					(unit 1)
-				)

Commit message: lot more routing on the motherboard
Parts:
- removed RN1: 10k, Resistor_SMD:R_Array_Concave_4x0603, symbol Device:R_Network04
- added RN1: R_Pack04, Resistor_SMD:R_Array_Convex_4x0603, symbol Device:R_Pack04
Connections:
- net +5V: now also RN1.5 (R4.2), RN1.6 (R3.2), RN1.7 (R2.2), RN1.8 (R1.2)
- net at JP7.2 (B), U9.1 (A0): now also RN1.4 (R4.1)
- net at JP3.2 (B), U9.3 (A2): now also RN1.2 (R2.1)
- net at JP5.2 (B), U9.2 (A1): now also RN1.3 (R3.1)
- net at Q1.1 (B), U9.7 (P3): now also RN1.1 (R1.1)
- net +3.3V renamed +3V3
