File: PRODIGY-MOTHERBOARD/nfc.kicad_sch (KiCad schematic)
At the start: 33 parts, among them U16 PN5321A3HN_C1xx, Y1 27.12MHz

Commit message: Motherboard footprints assigned.
Parts:
- C43, C46, C47, C48, C49, C50, C51, C52, C53, C54, C55, C56, C57, C58, C59, C60, C61, C62, C63: footprint (none) -> Capacitor_SMD:C_0603_1608Metric
- C44, C45: footprint (none) -> Capacitor_SMD:C_0805_2012Metric
- FID17, FID18: footprint (none) -> Fiducial:Fiducial_1mm_Mask3mm
- L5, L6: footprint (none) -> Inductor_SMD:L_0603_1608Metric
- R33, R34, R35, R36, R37: footprint (none) -> Resistor_SMD:R_0603_1608Metric
- Y1: footprint (none) -> Crystal:Crystal_SMD_EuroQuartz_MJ-4Pin_5.0x3.2mm

Commit message: finished motherboard bom and updated footprints
Parts:
- AE1, FID17, FID18: now not fitted
- C43, C46, C47, C48, C49, C52: TME (none) -> CL10B104KB8NNNC
- C44, C45: TME (none) -> CL21A475KAQNNNG
- C50, C51, C57, C58: TME (none) -> 0603N220J500CT
- C53: TME (none) -> 0603B102K500CT
- C54, C55: TME (none) -> CL10C221JB8NNNC
- C56, C59, C62, C63: value 5pF -> 4.7pF; TME (none) -> CC0603BRNPO9BN4R7
- C60, C61: TME (none) -> 0603N101J500CT
- L5, L6: TME (none) -> MLF1608DR56JT
- R33: TME (none) -> WR06X1002FTL
- R34: TME (none) -> RC0603JR-071K
- R35: TME (none) -> ERA3AEB272V
- R36, R37: TME (none) -> WF06P-3R3-5%
- U16: MOUSER (none) -> 771-PN5321A3HNC10
- Y1: footprint Crystal:Crystal_SMD_EuroQuartz_MJ-4Pin_5.0x3.2mm -> Crystal:Crystal_SMD_SeikoEpson_FA128-4Pin_2.0x1.6mm; TME (none) -> XRCGB27M120F3M00R0
Changed lines of the file:
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@@
 			)
 		)
-		(property "Value" "5pF"
+		(property "Value" "4.7pF"
 			(at 227.33 31.75 90)
 			(effects
@@
 			)
 		)
-		(property "TME" ""
+		(property "TME" "CC0603BRNPO9BN4R7 "
 			(at 227.33 36.83 0)
 			(effects
@@
 		(in_bom yes)
 		(on_board yes)
-		(dnp no)
+		(dnp yes)
 		(property "Reference" "AE1"
 			(at 276.352 63.246 90)
@@
 			)
 		)
-		(property "TME" ""
+		(property "TME" "CL10C221JB8NNNC"
 			(at 199.39 62.23 0)
 			(effects
@@
 			)
 		)
-		(property "TME" ""
+		(property "TME" "CL10B104KB8NNNC  "
 			(at 20.32 74.93 0)
 			(effects
@@
 			)
 		)
-		(property "TME" ""
+		(property "TME" "CL10B104KB8NNNC  "
 			(at 36.83 54.61 0)
 			(effects
@@
 			)
 		)
-		(property "Value" "5pF"
+		(property "Value" "4.7pF"
 			(at 227.33 78.74 90)
 			(effects
@@
 			)
 		)
-		(property "TME" ""
+		(property "TME" "CC0603BRNPO9BN4R7 "
 			(at 227.33 73.66 0)
 			(effects
@@
 			)
 		)
-		(property "TME" ""
+		(property "TME" "CL21A475KAQNNNG"
 			(at 22.86 54.61 0)
 			(effects
@@
 			)
 		)
-		(property "TME" ""
+		(property "TME" "CL10B104KB8NNNC  "
 			(at 151.13 67.31 0)
 			(effects
@@
 			)
 		)
-		(property "TME" ""
+		(property "TME" "WF06P-3R3-5%"
 			(at 264.16 48.26 0)
 			(effects
@@
 			)
 		)
-		(property "TME" ""
+		(property "TME" "0603B102K500CT"
 			(at 165.1 57.15 0)
 			(effects
@@
 			)
 		)
-		(property "TME" ""
+		(property "TME" "MLF1608DR56JT"
 			(at 187.96 66.04 0)
 			(effects
@@
 			)
 		)
-		(property "TME" ""
+		(property "TME" "MLF1608DR56JT"
 			(at 187.96 48.26 0)
 			(effects
@@
 			)
 		)
-		(property "TME" ""
+		(property "TME" "ERA3AEB272V"
 			(at 165.1 67.31 0)
 			(effects
@@
 			)
 		)
-		(property "TME" ""
+		(property "TME" "CL10B104KB8NNNC  "
 			(at 35.56 36.83 0)
 			(effects
@@
 			)
 		)
-		(property "TME" ""
+		(property "TME" "WR06X1002FTL "
 			(at 100.33 41.91 0)
 			(effects
@@
 			)
 		)
-		(property "TME" ""
+		(property "TME" "CL10C221JB8NNNC"
 			(at 199.39 52.07 0)
 			(effects
@@
 			)
 		)
-		(property "TME" ""
+		(property "TME" "0603N220J500CT"
 			(at 87.63 81.28 0)
 			(effects
@@
 			)
 		)
-		(property "TME" ""
+		(property "TME" "0603N220J500CT"
 			(at 71.12 81.28 0)
 			(effects
@@
 			)
 		)
-		(property "TME" ""
+		(property "TME" "CL10B104KB8NNNC  "
 			(at 46.99 74.93 0)
 			(effects
@@
 			)
 		)
-		(property "TME" ""
+		(property "TME" "0603N101J500CT"
 			(at 240.03 62.23 0)
 			(effects
@@
 			)
 		)
-		(property "Value" "5pF"
+		(property "Value" "4.7pF"
 			(at 256.54 63.4999 0)
 			(effects
@@
 			)
 		)
-		(property "TME" ""
+		(property "TME" "CC0603BRNPO9BN4R7 "
 			(at 252.73 62.23 0)
 			(effects
@@
 			)
 		)
-		(property "TME" ""
+		(property "TME" "0603N220J500CT"
 			(at 227.33 66.04 0)
 			(effects
@@
 			)
 		)
-		(property "TME" ""
+		(property "TME" "RC0603JR-071K "
 			(at 151.13 57.15 0)
 			(effects
@@
 			)
 		)
-		(property "TME" ""
+		(property "TME" "CL10B104KB8NNNC  "
 			(at 34.29 74.93 0)
 			(effects
@@
 		(in_bom yes)
 		(on_board yes)
-		(dnp no)
+		(dnp yes)
 		(fields_autoplaced yes)
 		(property "Reference" "FID17"
@@
 			)
 		)
-		(property "TME" ""
+		(property "TME" "0603N101J500CT"
 			(at 240.03 52.07 0)
 			(effects
@@
 			)
 		)
-		(property "TME" ""
+		(property "TME" "0603N220J500CT"
 			(at 227.33 48.26 0)
 			(effects
@@
 			)
 		)
-		(property "Footprint" "Crystal:Crystal_SMD_EuroQuartz_MJ-4Pin_5.0x3.2mm"
+		(property "Footprint" "Crystal:Crystal_SMD_SeikoEpson_FA128-4Pin_2.0x1.6mm"
 			(at 78.74 77.47 0)
 			(effects
@@
 			)
 		)
-		(property "TME" ""
+		(property "TME" "XRCGB27M120F3M00R0"
 			(at 78.74 77.47 0)
 			(effects
@@
 			)
 		)
-		(property "Value" "5pF"
+		(property "Value" "4.7pF"
 			(at 256.54 53.3399 0)
 			(effects
@@
 			)
 		)
-		(property "TME" ""
+		(property "TME" "CC0603BRNPO9BN4R7 "
 			(at 252.73 52.07 0)
 			(effects
@@
 			)
 		)
-		(property "MOUSER" ""
+		(property "MOUSER" " 771-PN5321A3HNC10 "
 			(at 123.19 71.12 0)
 			(effects
@@
 		(in_bom yes)
 		(on_board yes)
-		(dnp no)
+		(dnp yes)
 		(fields_autoplaced yes)
 		(property "Reference" "FID18"
@@
 			)
 		)
-		(property "TME" ""
+		(property "TME" "CL21A475KAQNNNG"
 			(at 22.86 36.83 0)
 			(effects
@@
 			)
 		)
-		(property "TME" ""
+		(property "TME" "WF06P-3R3-5%"
 			(at 264.16 66.04 0)
 			(effects

Commit message: Motherboard PCB layout started
Parts:
- removed FID17, FID18: Fiducial, Fiducial:Fiducial_1mm_Mask3mm, symbol Mechanical:Fiducial
Changed lines of the file:
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@@
-	)
-	(symbol
-		(lib_id "Mechanical:Fiducial")
-		(at 113.03 123.19 0)
-		(unit 1)
-		(exclude_from_sim no)
-		(in_bom yes)
-		(on_board yes)
-		(dnp yes)
-		(fields_autoplaced yes)
-		(property "Reference" "FID17"
-			(at 115.57 121.9199 0)
-			(effects
-				(font
-					(size 1.27 1.27)
-				)
-				(justify left)
-			)
-		)
-		(property "Value" "Fiducial"
-			(at 115.57 124.4599 0)
-			(effects
-				(font
-					(size 1.27 1.27)
-				)
-				(justify left)
-			)
-		)
-		(property "Footprint" "Fiducial:Fiducial_1mm_Mask3mm"
-			(at 113.03 123.19 0)
-			(effects
-				(font
-					(size 1.27 1.27)
-				)
-				(hide yes)
-			)
-		)
-		(property "Datasheet" "~"
-			(at 113.03 123.19 0)
-			(effects
-				(font
-					(size 1.27 1.27)
-				)
-				(hide yes)
-			)
-		)
-		(property "Description" "Fiducial Marker"
-			(at 113.03 123.19 0)
-			(effects
-				(font
-					(size 1.27 1.27)
-				)
-				(hide yes)
-			)
-		)
-		(property "MOUSER" ""
-			(at 113.03 123.19 0)
-			(effects
-				(font
-					(size 1.27 1.27)
-				)
-				(hide yes)
-			)
-		)
-		(property "Sim.Type" ""
-			(at 113.03 123.19 0)
-			(effects
-				(font
-					(size 1.27 1.27)
-				)
-				(hide yes)
-			)
-		)
-		(property "TME" ""
-			(at 113.03 123.19 0)
-			(effects
-				(font
-					(size 1.27 1.27)
-				)
-				(hide yes)
-			)
-		)
-		(instances
-			(project "PRODIGY-MOTHERBOARD"
-				(path "/f1c25860-8989-4190-bd24-2491d23ca7d9/e2913798-f444-47a6-8b64-53020d7d816b/d8aab2a1-25b6-4fb2-8368-6cdabd5442db"
-					(reference "FID17")
-					(unit 1)
-				)
-			)
-		)
 	)
 	(symbol
@@
 					(unit 1)
 				)
-			)
-		)
-	)
-	(symbol
-		(lib_id "Mechanical:Fiducial")
-		(at 128.27 123.19 0)
-		(unit 1)
-		(exclude_from_sim no)
-		(in_bom yes)
-		(on_board yes)
-		(dnp yes)
-		(fields_autoplaced yes)
-		(property "Reference" "FID18"
-			(at 130.81 121.9199 0)
-			(effects
-				(font
-					(size 1.27 1.27)
-				)
-				(justify left)
-			)
-		)
-		(property "Value" "Fiducial"
-			(at 130.81 124.4599 0)
-			(effects
-				(font
-					(size 1.27 1.27)
-				)
-				(justify left)
-			)
-		)
-		(property "Footprint" "Fiducial:Fiducial_1mm_Mask3mm"
-			(at 128.27 123.19 0)
-			(effects
-				(font
-					(size 1.27 1.27)
-				)
-				(hide yes)
-			)
-		)
-		(property "Datasheet" "~"
-			(at 128.27 123.19 0)
-			(effects
-				(font
-					(size 1.27 1.27)
-				)
-				(hide yes)
-			)
-		)
-		(property "Description" "Fiducial Marker"
-			(at 128.27 123.19 0)
-			(effects
-				(font
-					(size 1.27 1.27)
-				)
-				(hide yes)
-			)
-		)
-		(property "MOUSER" ""
-			(at 128.27 123.19 0)
-			(effects
-				(font
-					(size 1.27 1.27)
-				)
-				(hide yes)
-			)
-		)
-		(property "Sim.Type" ""
-			(at 128.27 123.19 0)
-			(effects
-				(font
-					(size 1.27 1.27)
-				)
-				(hide yes)
-			)
-		)
-		(property "TME" ""
-			(at 128.27 123.19 0)
-			(effects
-				(font
-					(size 1.27 1.27)
-				)
-				(hide yes)
-			)
-		)
-		(instances
-			(project "PRODIGY-MOTHERBOARD"
-				(path "/f1c25860-8989-4190-bd24-2491d23ca7d9/e2913798-f444-47a6-8b64-53020d7d816b/d8aab2a1-25b6-4fb2-8368-6cdabd5442db"
-					(reference "FID18")
-					(unit 1)
-				)

Commit message: nice routing done. nfc antenna close to done
Parts:
- AE1: footprint (none) -> NFC_antenna_v1:40x40 antenna
Changed lines of the file:
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@@
 			)
 		)
-		(property "Footprint" ""
+		(property "Footprint" "NFC_antenna_v1:40x40 antenna"
 			(at 278.13 55.88 0)
 			(effects
