File: PRODIGY-MOTHERBOARD/sevenseg.kicad_sch (KiCad schematic)
At the start: 5 parts, among them U14 MAX7219 / tm1637, U15 CC56-12YWA

Commit message: Motherboard PCB layout started
Parts:
- U15: footprint Display_7Segment:CA56-12SRWA -> seven_segment_four_digit:4_digit_7_segment_display
Changed lines of the file:
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@@
 			)
 		)
-		(property "Footprint" "Display_7Segment:CA56-12SRWA"
+		(property "Footprint" "seven_segment_four_digit:4_digit_7_segment_display"
 			(at 180.34 96.52 0)
 			(effects
