File: PRODIGY-ATMEGA2560/conLeft.kicad_sch (KiCad schematic)
At the start: 1 part, among them J1 DF40C-100DS-0.4V(51)

Commit message: ESP32 and ATMEGA bom done.
Parts:
- J1: value DF40C-100DS-0.4V(51) -> DF40C-100DP-04V-51; TME (none) -> DF40C-100DP-04V-51
Changed lines of the file:
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@@
 			)
 		)
-		(property "Value" "DF40C-100DS-0.4V(51)"
+		(property "Value" "DF40C-100DP-04V-51 "
 			(at 135.89 25.654 0)
 			(effects
@@
 			(effects
 				(font
+					(size 1.27 1.27)
+				)
+				(hide yes)
+			)
+		)
+		(property "TME" "DF40C-100DP-04V-51 "
+			(at 135.89 25.4 0)
+			(effects
+				(font

Commit message: Atmega layout done. orientation and alignment testing done. routing started.
Parts:
- J1: footprint DF40C:HIROSE_DF40C-100DS-0.4V_51_ -> DF40C-100DP-0:DF40C100DP04V51
Connections:
- net USB_DM is gone; now on net GND: J1.3
- net ANALOG_BREAKOUT_PIEZO: now also J1.2; no longer J1.100
- net ANALOG_BREAKOUT_PT100: now also J1.8; no longer J1.94
- net ANALOG_HEATER_TEMPERATURE: now also J1.14; no longer J1.88
- net ANALOG_JOYSTICK_X: now also J1.13; no longer J1.87
- net ANALOG_JOYSTICK_Y: now also J1.7; no longer J1.93
- net ANALOG_MICROPHONE: now also J1.1; no longer J1.99
- net ANALOG_PHOTOTRANSISTOR: now also J1.19; no longer J1.81
- net ANALOG_POTENTIOMETER: now also J1.20; no longer J1.82
- net CAN_EN: now also J1.86; no longer J1.16
- net CAN_OUT_RX1: now also J1.83; no longer J1.17
- net CAN_OUT_TX1: now also J1.85; no longer J1.15
- net CAN_SILENT: now also J1.84; no longer J1.18
- net DIGITAL_BUTTON_IN_0: now also J1.53; no longer J1.47
- net DIGITAL_BUTTON_IN_1: now also J1.51; no longer J1.49
- net DIGITAL_BUTTON_IN_2: now also J1.49; no longer J1.51
- net DIGITAL_BUTTON_IN_3: now also J1.47; no longer J1.53
- net DIGITAL_BUZZER_OUT: now also J1.42; no longer J1.60
- net DIGITAL_HEATER_OUT: now also J1.48; no longer J1.54
- net DIGITAL_IR_EMITTER: now also J1.67; no longer J1.33
- net DIGITAL_IR_RECEIVER: now also J1.65; no longer J1.35
- net DIGITAL_LED_OUT_0: now also J1.43; no longer J1.57
- net DIGITAL_LED_OUT_1: now also J1.41; no longer J1.59
- net DIGITAL_LED_OUT_2: now also J1.44; no longer J1.58
- net DIGITAL_NEOPIXEL_OUT: now also J1.61; no longer J1.39
- net DIGITAL_RGB_B: now also J1.55; no longer J1.45
- net DIGITAL_RGB_G: now also J1.57; no longer J1.43
- net DIGITAL_RGB_R: now also J1.59; no longer J1.41
- net GND: now also J1.10, J1.15, J1.16, J1.21, J1.22, J1.27, J1.28, J1.33, J1.34, J1.39, J1.4, J1.40, J1.45, J1.46, J1.52, J1.58, J1.63, J1.64, J1.69, J1.70, J1.75, J1.76, J1.81, J1.82, J1.87, J1.88, J1.9, J1.93, J1.94; no longer J1.13, J1.14, J1.19, J1.20, J1.25, J1.26, J1.31, J1.32, J1.37, J1.38, J1.44, J1.50, J1.55, J1.56, J1.61, J1.62, J1.67, J1.68, J1.7, J1.73, J1.74, J1.79, J1.8, J1.80, J1.85, J1.86, J1.91, J1.92, J1.97, J1.98
- net I2C_INTERRUPT_ACCEL: now also J1.73; no longer J1.27
- net I2C_INTERRUPT_KEYPAD: now also J1.71; no longer J1.29
- net I2C_SCL: now also J1.77; no longer J1.23
- net I2C_SDA: now also J1.79; no longer J1.21
- net MOTOR_CC_IN_1: now also J1.35; no longer J1.65
- net MOTOR_CC_IN_2: now also J1.36; no longer J1.66
- net MOTOR_PWM_OUT_1: now also J1.37; no longer J1.63
- net MOTOR_PWM_OUT_2: now also J1.38; no longer J1.64
- net SERIAL_OUT_RX1: now also J1.91; no longer J1.9
- net SERIAL_OUT_RX2: now also J1.90; no longer J1.12
- net SERIAL_OUT_TX1: now also J1.89; no longer J1.11
- net SERIAL_OUT_TX2: now also J1.92; no longer J1.10
- net SPI_CS_BREAKOUT: now also J1.72; no longer J1.30
- net SPI_CS_NFC: now also J1.56; no longer J1.46
- net SPI_CS_SEVENSEG: now also J1.68; no longer J1.34
- net SPI_CS_TFT: now also J1.66; no longer J1.36
- net SPI_IRQ_NFC: now also J1.54; no longer J1.48
- net SPI_MISO: now also J1.78; no longer J1.24
- net SPI_MOSI: now also J1.80; no longer J1.22
- net SPI_RST_NFC: now also J1.50; no longer J1.52
- net SPI_SCK: now also J1.74; no longer J1.28
- net SPI_TFT_DC: now also J1.62; no longer J1.40
- net SPI_TFT_RESET: now also J1.60; no longer J1.42
- net USB_HOST_ENABLE: now also J1.100; no longer J1.2
- net USB_HOST_FAULT: now also J1.99; no longer J1.1
- net USB_HOST_OUT_P+: now also J1.96; no longer J1.6
- net USB_HOST_OUT_P-: now also J1.98; no longer J1.4
- net USB+: now reaches J1.95
- net USB_DP: no longer names the net of J1.5
- new net USB-: J1.97
Changed lines of the file:
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@@
 		)
 	)
-	(hierarchical_label "USB_DP"
+	(hierarchical_label "USB+"
 		(shape bidirectional)
 		(at 147.32 34.29 0)
@@
 		)
 	)
-	(hierarchical_label "USB_DM"
+	(hierarchical_label "USB-"
 		(shape bidirectional)
 		(at 147.32 31.75 0)
@@
 	(symbol
 		(lib_id "2x50_generic_connector:2x50_Odd-Even")
-		(at 135.89 25.4 0)
+		(at 135.89 157.48 0)
+		(mirror x)
 		(unit 1)
 		(exclude_from_sim no)
@@
 		(dnp no)
 		(property "Reference" "J1"
-			(at 135.89 23.114 0)
+			(at 135.89 159.766 0)
 			(effects
 				(font
@@
 		)
 		(property "Value" "DF40C-100DP-04V-51 "
-			(at 135.89 25.654 0)
-			(effects
-				(font
-					(size 1.27 1.27)
-				)
-			)
-		)
-		(property "Footprint" "DF40C:HIROSE_DF40C-100DS-0.4V_51_"
-			(at 135.636 23.876 0)
+			(at 135.89 157.226 0)
+			(effects
+				(font
+					(size 1.27 1.27)
+				)
+			)
+		)
+		(property "Footprint" "DF40C-100DP-0:DF40C100DP04V51"
+			(at 135.636 159.004 0)
 			(effects
 				(font
@@
 		)
 		(property "Datasheet" ""
-			(at 135.636 23.876 0)
+			(at 135.636 159.004 0)
 			(effects
 				(font
@@
 		)
 		(property "Description" ""
-			(at 135.636 23.876 0)
+			(at 135.636 159.004 0)
 			(effects
 				(font
@@
 		)
 		(property "TME" "DF40C-100DP-04V-51 "
-			(at 135.89 25.4 0)
-			(effects
-				(font
+			(at 135.89 157.48 0)
+			(effects
+				(font
