File: PRODIGY-ATMEGA2560/usbBridge.kicad_sch (KiCad schematic)
At the start: 9 parts, among them Q1 BC850, Q2 BC850, U3 FT231XQ

Commit message: All footprint assosiations have been made across all schematics.
Parts:
- C10: footprint (none) -> Capacitor_SMD:C_0603_1608Metric
- C9: footprint (none) -> Capacitor_SMD:C_0805_2012Metric
Changed lines of the file:
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@@
 			)
 		)
-		(property "Footprint" ""
+		(property "Footprint" "Capacitor_SMD:C_0805_2012Metric"
 			(at 147.6248 125.73 0)
 			(effects
@@
 			)
 		)
-		(property "Footprint" ""
+		(property "Footprint" "Capacitor_SMD:C_0603_1608Metric"
 			(at 161.5948 125.73 0)
 			(effects

Commit message: ESP32 and ATMEGA bom done.
Parts:
- C10: TME (none) -> CL10B104KB8NNNC
- C9: TME (none) -> 0603N100J500CT
- Q1, Q2: TME (none) -> BC850B-DIO
- R1, R2: TME (none) -> SMD0603-0R
- R3, R4: TME (none) -> WR06X1002FTL
- U3: TME (none) -> FT231XQ-R
Changed lines of the file:
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@@
+			)
+		)
+		(property "TME" "BC850B-DIO "
+			(at 204.47 113.03 0)
+			(effects
+				(font
+					(size 1.27 1.27)
+				)
+				(hide yes)
 			)
 		)
@@
 			)
 		)
+		(property "TME" "SMD0603-0R"
+			(at 121.92 100.33 0)
+			(effects
+				(font
+					(size 1.27 1.27)
+				)
+				(hide yes)
+			)
+		)
 		(pin "1"
 		)
@@
 			)
 		)
+		(property "TME" "FT231XQ-R"
+			(at 92.71 115.57 0)
+			(effects
+				(font
+					(size 1.27 1.27)
+				)
+				(hide yes)
+			)
+		)
 		(pin "1"
 		)
@@
 			)
 		)
+		(property "TME" "BC850B-DIO "
+			(at 204.47 129.54 0)
+			(effects
+				(font
+					(size 1.27 1.27)
+				)
+				(hide yes)
+			)
+		)
 		(pin "2"
 		)
@@
 			)
 		)
+		(property "TME" "0603N100J500CT "
+			(at 148.59 121.92 0)
+			(effects
+				(font
+					(size 1.27 1.27)
+				)
+				(hide yes)
+			)
+		)
 		(pin "2"
 		)
@@
 			)
 		)
+		(property "TME" "CL10B104KB8NNNC "
+			(at 162.56 121.92 0)
+			(effects
+				(font
+					(size 1.27 1.27)
+				)
+				(hide yes)
+			)
+		)
 		(pin "2"
 		)
@@
 			)
 		)
+		(property "TME" "WR06X1002FTL "
+			(at 194.31 129.54 0)
+			(effects
+				(font
+					(size 1.27 1.27)
+				)
+				(hide yes)
+			)
+		)
 		(pin "1"
 		)
@@
 			)
 		)
+		(property "TME" "SMD0603-0R"
+			(at 121.92 102.87 0)
+			(effects
+				(font
+					(size 1.27 1.27)
+				)
+				(hide yes)
+			)
+		)
 		(pin "1"
 		)
@@
 			(at 194.31 113.03 0)
 			(effects
+				(font
+					(size 1.27 1.27)
+				)
+				(hide yes)
+			)
+		)
+		(property "TME" "WR06X1002FTL "
+			(at 194.31 113.03 0)
+			(effects

Commit message: Atmega layout done. orientation and alignment testing done. routing started.
Connections:
- net USB_DM renamed USB-
- net USB_DP renamed USB+
Changed lines of the file:
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@@
 		)
 	)
-	(hierarchical_label "USB_DM"
+	(hierarchical_label "USB-"
 		(shape bidirectional)
 		(at 71.12 107.95 180)
@@
 		)
 	)
-	(hierarchical_label "USB_DP"
+	(hierarchical_label "USB+"
 		(shape bidirectional)
 		(at 71.12 110.49 180)
@@
 		)
 		(instances
-			(project ""
+			(project "PRODIGY-ATMEGA2560"
 				(path "/58f705c8-87df-406b-b9b9-efbb33b15a7f/c0859e15-ccd4-4bc9-9657-4794b2548a11"
 					(reference "#PWR015")
