File: PRODIGY-ATMEGA2560/PRODIGY-ATMEGA2560.kicad_pcb (KiCad board)
At the start: 4 copper layers, 55 x 40 mm, 29 parts, among them J1 DF40C-100DP-04V-51, J2 DF40C-100DP-04V-51, Q1 BC850, Q2 BC850, U1 ATmega2560-8A, U2 TXS0108EPW, U3 FT231XQ, Y1 8MHz

Commit message: atmega board done, labeling done, gerber export done,
Parts:
- added G***: LOGO, LOGO, F.Cu at (109.8, 128.1)
Routing:
- net GND: vias 112 -> 179
Other:
- board text added: "Desgined by Kovács Márk"
- board text added: "JLCJLCJLC WAYWAYWAY 30092024 v0.1"
- board text added: "PRODIGY-ATMEGA"
- board text added: "V0.1"
